File: ProProject_X1 Expander_2024-05-26_15-16-51_2024-05-26.kicad_pcb (KiCad board)
At the start: 4 copper layers, 145 x 57 mm, 107 parts, among them U1 LAN9514, U2 FT2232HL, U3 TPS54202DDCR, U4 LM1084S-3.3/TR, X1 25MHz, X2 12MHz

Commit message: initial full placement and routing
Parts:
- C19: moved to B.Cu
- C32, C38, C39, C40: footprint Capacitor_SMD:C_0603_1608Metric -> Capacitor_SMD:C_0402_1005Metric
- C33, C34, C35, C36, C37, C42, C44: footprint Capacitor_SMD:C_0603_1608Metric -> Capacitor_SMD:C_0402_1005Metric; moved to F.Cu
- C41, C43, FB3, FB4: moved to F.Cu
- moved R17 26.6 mm to (175.6, 105.4), turned to 0 degrees
- moved R16 26.4 mm to (175.6, 106.9), turned to 0 degrees
- moved C39 26.2 mm to (181.0, 104.8), turned to 90 degrees
- moved C40 23.9 mm to (183.1, 111.9), turned to 0 degrees
- moved R14 23.7 mm to (179.2, 107.8)
- moved R15 23.1 mm to (178.9, 103.4), turned to 0 degrees
- moved R8 21.4 mm to (91.9, 119.9)
- moved C33 20.5 mm to (191.5, 109.1), turned to -90 degrees
- moved C32 18.1 mm to (192.6, 113.1)
- moved R21 17.3 mm to (149.5, 119.4), turned to -90 degrees
- moved C31 17.2 mm to (193.9, 111.9)
- moved R30 16.7 mm to (148.0, 119.4), turned to 90 degrees
- moved R18 16.5 mm to (86.9, 89.6), turned to 90 degrees
- moved C42 15.6 mm to (185.4, 108.4)
- moved FB4 14.1 mm to (184.9, 112.4), turned to 90 degrees
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Connections:
- AP_HARNESS1 pad 1: 5V -> GND
- AP_HARNESS1 pad 10: GND -> CAMO_DP
- AP_HARNESS1 pad 11: Net-(AP_HARNESS1-Pad11) -> CAMO_DN
- AP_HARNESS1 pad 12: GND -> 5V
- AP_HARNESS1 pad 2: CAMO_DN -> Net-(AP_HARNESS1-Pad2)
- AP_HARNESS1 pad 3: CAMO_DP -> GND
- AP_HARNESS1 pad 4: GND -> UARTTX
- AP_HARNESS1 pad 5: MBDN -> UARTRX
- AP_HARNESS1 pad 6: MBDP -> UART3V3
- AP_HARNESS1 pad 7: UART3V3 -> MBDP
- AP_HARNESS1 pad 8: UARTRX -> MBDN
- AP_HARNESS1 pad 9: UARTTX -> GND
- C34 pad 2: VIO -> 3V3
- C35 pad 2: VIO -> 3V3
- C36 pad 2: VIO -> 3V3
- C37 pad 2: VIO -> 3V3
- D2 pad 1: ACBUS0 -> ACBUS1
- D2 pad 3: ACBUS1 -> ACBUS0
- D3 pad 1: ACBUS4 -> ACBUS5
- D3 pad 3: ACBUS5 -> ACBUS4
- D4 pad 1: ADBUS0 -> ADBUS1
- D4 pad 3: ADBUS1 -> ADBUS0
- D5 pad 1: ADBUS4 -> ADBUS5
- D5 pad 3: ADBUS5 -> ADBUS4
- D6 pad 1: BCBUS0 -> BCBUS1
- D6 pad 3: BCBUS1 -> BCBUS0
- D7 pad 1: BCBUS4 -> BCBUS5
- D7 pad 3: BCBUS5 -> BCBUS4
- D8 pad 1: BDBUS0 -> BDBUS1
- D8 pad 3: BDBUS1 -> BDBUS0
- D9 pad 1: BDBUS4 -> BDBUS5
- D9 pad 3: BDBUS5 -> BDBUS4
- F1 pad 2: Net-(AP_HARNESS1-Pad11) -> Net-(AP_HARNESS1-Pad2)
- U2 pad 20: VIO -> 3V3
- U2 pad 31: VIO -> 3V3
- U2 pad 42: VIO -> 3V3
- U2 pad 56: VIO -> 3V3
Routing:
- net BDBUS0: track 0.00 -> 164.0 mm
- net BDBUS1: track 0.00 -> 154.7 mm, vias 0 -> 2
- net BDBUS2: track 0.00 -> 137.5 mm, vias 0 -> 2
- net FTDI_DN: track 7.21 -> 136.6 mm, vias 1 -> 3
- net FTDI_DP: track 7.21 -> 136.6 mm, vias 1 -> 3
- net BDBUS3: track 0.00 -> 126.7 mm
- net BDBUS4: track 0.00 -> 122.3 mm
- net BDBUS5: track 0.00 -> 116.4 mm
- net UARTTX: track 0.00 -> 115.0 mm, vias 0 -> 2
- net BDBUS6: track 0.00 -> 112.5 mm
- net BDBUS7: track 0.00 -> 111.6 mm
- net UARTRX: track 0.00 -> 111.4 mm, vias 0 -> 2
- net UART3V3: track 0.00 -> 107.5 mm, vias 0 -> 2
- net BCBUS0: track 0.00 -> 101.7 mm
- net BCBUS1: track 0.00 -> 89.4 mm
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Other:
- outline, holes or cut-outs redrawn
- board text removed: "THE IMPEDANCE IS BULLSHIT FIGURE OUT THE NET WIDTH NEXT TIME"

Commit message: clean up DRC and silkscreen
Parts:
- added R2: 0, Resistor_SMD:R_0603_1608Metric, F.Cu at (157.2, 127.0)
- R18: value 10kΩ -> 330
- moved C8 0.38 mm to (203.0, 125.4)
Connections:
- C4 pad 2: 5V -> /MAIN/5V_INT
- C5 pad 2: 5V -> /MAIN/5V_INT
- L1 pad 2: 5V -> /MAIN/5V_INT
- R3 pad 2: 5V -> /MAIN/5V_INT
Routing:
- net 5V: track 42.7 -> 44.2 mm, vias 24 -> 23
- net GND: track 82.8 -> 81.9 mm, vias 108 -> 171
- net VDD3A: vias 13 -> 12
- net 3V3: vias 45 -> 43
- added copper zone on F.Cu, net /MAIN/5V_INT
- added copper zone on B.Cu, net 5V
Other:
- board text added: "3.3"
- board text added: "3V3"
- board text added: "5V"
- board text added: "AC0"
- board text added: "AC1"
- board text added: "AC2"
- board text added: "AC3"
- board text added: "AC4"
- board text added: "AC5"
- board text added: "AC6"
- board text added: "AC7"
- board text added: "AD0"
- board text added: "AD1"
- board text added: "AD2"
- board text added: "AD3"
- board text added: "AD4"
- board text added: "AD5"
- board text added: "AD6"
- board text added: "AD7"
- board text added: "BC0"
- board text added: "BC1"
- board text added: "BC2"
- board text added: "BC3"
- board text added: "BC4"
- board text added: "BC5"
- board text added: "BC6"
- board text added: "BC7"
- board text added: "BD0"
- board text added: "BD1"
- board text added: "BD2"
- board text added: "BD3"
- board text added: "BD4"
- board text added: "BD5"
- board text added: "BD6"
- board text added: "BD7"
- board text added: "DBG AP"
- board text added: "Gnd"
- board text added: "I²C"
- board text added: "RX"
- board text added: "SCL"
- board text added: "SDA"
- board text added: "TX"
- board text added: "port B"

Commit message: add LCSC part tags, silkscreen
Parts:
- added G***: LOGO, X1 Expande-easyedapro:emarhavil, F.Cu at (171.0, 135.0)
- added G***: LOGO, X1 Expande-easyedapro:x1plus, F.Cu at (138.5, 111.5)
- added REF**: OSHW-Symbol_6.7x6mm_SilkScreen, Symbol:OSHW-Symbol_6.7x6mm_SilkScreen, F.Cu at (179.0, 135.0)
Other:
- board text added: "X1P-002-A01"

Commit message: LCSC part updates
Parts:
- renumbered STEMMA-I2C1 to I2C1
Changed lines of the file:
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@@
 			)
 		)
-		(property "Supplier Part" "C19190478"
+		(property "Supplier Part" "C2935929"
 			(at 0 0 0)
 			(unlocked yes)
@@
 			)
 		)
-		(property "LCSC Part" "C19190478"
+		(property "LCSC Part" "C2935929"
 			(at 0 0 0)
 			(unlocked yes)
@@
 			)
 		)
-		(property "LCSC" "C19190478"
+		(property "LCSC" "C2935929"
 			(at 0 0 0)
 			(unlocked yes)
@@
 		(layer "F.Cu")
 		(at 73.425 87.01 -90)
-		(property "Reference" "STEMMA-I2C1"
+		(property "Reference" "I2C1"
 			(at 0 0 -90)
 			(unlocked yes)
