File: 3_GPIO.kicad_sch (KiCad schematic)
At the start: 17 parts, among them P3 A_A4

Commit message: rename to x1-expander
Parts:
- ACBUS1, ADBUS1, BCBUS1, BDBUS1: footprint X1 Expande-easyedapro:HDR-TH_16P-P2.54-H-F-R2-C8-W9.0 -> x1-expander:HDR-TH_16P-P2.54-H-F-R2-C8-W9.0; symbol X1 Expande-easyedapro:HC-JN254-2-08-W -> x1-expander:HC-JN254-2-08-W
- D2, D3, D4, D5, D6, D7, D8, D9: footprint X1 Expande-easyedapro:SOT-23-6_L2.9-W1.6-P0.95-LS2.8-BL -> x1-expander:SOT-23-6_L2.9-W1.6-P0.95-LS2.8-BL; symbol X1 Expande-easyedapro:SRV05-4.TCT_C2687126 -> x1-expander:SRV05-4.TCT_C2687126
- I2C1: footprint X1 Expande-easyedapro:CONN-TH_S4B-PH-KL-LF-SN -> x1-expander:CONN-TH_S4B-PH-KL-LF-SN; symbol X1 Expande-easyedapro:S4B-PH-KL(LF)(SN) -> x1-expander:S4B-PH-KL(LF)(SN)
- P3: footprint X1 Expande-easyedapro: -> x1-expander:; symbol X1 Expande-easyedapro:A_A4 -> x1-expander:A_A4
- R18: symbol X1 Expande-easyedapro:10kΩ -> x1-expander:10kΩ
- R19, R20: symbol X1 Expande-easyedapro:4.7k -> x1-expander:4.7k
Changed lines of the file:
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@@
 	)
 	(symbol
-		(lib_id "X1 Expande-easyedapro:HC-JN254-2-08-W")
+		(lib_id "x1-expander:HC-JN254-2-08-W")
 		(at 187.96 132.08 0)
 		(unit 1)
@@
 			)
 		)
-		(property "Footprint" "X1 Expande-easyedapro:HDR-TH_16P-P2.54-H-F-R2-C8-W9.0"
+		(property "Footprint" "x1-expander:HDR-TH_16P-P2.54-H-F-R2-C8-W9.0"
 			(at 187.96 132.08 0)
 			(effects
@@
 		)
 		(instances
-			(project "ProProject_X1 Expander_2024-05-26_15-16-51_2024-05-26"
+			(project "x1-expander"
 				(path "/5c4052f8-31d6-4de3-b862-4d09b0660e26/52713671-aa4b-4412-b159-5876c2aaf3b7"
 					(reference "BDBUS1")
@@
 	)
 	(symbol
-		(lib_id "X1 Expande-easyedapro:SRV05-4.TCT_C2687126")
+		(lib_id "x1-expander:SRV05-4.TCT_C2687126")
 		(at 48.26 83.82 270)
 		(unit 1)
@@
 			)
 		)
-		(property "Footprint" "X1 Expande-easyedapro:SOT-23-6_L2.9-W1.6-P0.95-LS2.8-BL"
+		(property "Footprint" "x1-expander:SOT-23-6_L2.9-W1.6-P0.95-LS2.8-BL"
 			(at 48.26 83.82 0)
 			(effects
@@
 		)
 		(instances
-			(project "ProProject_X1 Expander_2024-05-26_15-16-51_2024-05-26"
+			(project "x1-expander"
 				(path "/5c4052f8-31d6-4de3-b862-4d09b0660e26/52713671-aa4b-4412-b159-5876c2aaf3b7"
 					(reference "D3")
@@
 	)
 	(symbol
-		(lib_id "X1 Expande-easyedapro:A_A4")
+		(lib_id "x1-expander:A_A4")
 		(at 0 -0.254 0)
 		(unit 1)
@@
 			)
 		)
-		(property "Footprint" "X1 Expande-easyedapro:"
+		(property "Footprint" "x1-expander:"
 			(at 0 -0.254 0)
 			(effects
@@
 		)
 		(instances
-			(project "ProProject_X1 Expander_2024-05-26_15-16-51_2024-05-26"
+			(project "x1-expander"
 				(path "/5c4052f8-31d6-4de3-b862-4d09b0660e26/52713671-aa4b-4412-b159-5876c2aaf3b7"
 					(reference "P3")
@@
 	)
 	(symbol
-		(lib_id "X1 Expande-easyedapro:HC-JN254-2-08-W")
+		(lib_id "x1-expander:HC-JN254-2-08-W")
 		(at 187.96 73.66 0)
 		(unit 1)
@@
 			)
 		)
-		(property "Footprint" "X1 Expande-easyedapro:HDR-TH_16P-P2.54-H-F-R2-C8-W9.0"
+		(property "Footprint" "x1-expander:HDR-TH_16P-P2.54-H-F-R2-C8-W9.0"
 			(at 187.96 73.66 0)
 			(effects
@@
 		)
 		(instances
-			(project "ProProject_X1 Expander_2024-05-26_15-16-51_2024-05-26"
+			(project "x1-expander"
 				(path "/5c4052f8-31d6-4de3-b862-4d09b0660e26/52713671-aa4b-4412-b159-5876c2aaf3b7"
 					(reference "ADBUS1")
@@
 	)
 	(symbol
-		(lib_id "X1 Expande-easyedapro:SRV05-4.TCT_C2687126")
+		(lib_id "x1-expander:SRV05-4.TCT_C2687126")
 		(at 121.92 83.82 270)
 		(unit 1)
@@
 			)
 		)
-		(property "Footprint" "X1 Expande-easyedapro:SOT-23-6_L2.9-W1.6-P0.95-LS2.8-BL"
+		(property "Footprint" "x1-expander:SOT-23-6_L2.9-W1.6-P0.95-LS2.8-BL"
 			(at 121.92 83.82 0)
 			(effects
@@
 		)
 		(instances
-			(project "ProProject_X1 Expander_2024-05-26_15-16-51_2024-05-26"
+			(project "x1-expander"
 				(path "/5c4052f8-31d6-4de3-b862-4d09b0660e26/52713671-aa4b-4412-b159-5876c2aaf3b7"
 					(reference "D5")
@@
 	)
 	(symbol
-		(lib_id "X1 Expande-easyedapro:HC-JN254-2-08-W")
+		(lib_id "x1-expander:HC-JN254-2-08-W")
 		(at 187.96 102.87 0)
 		(unit 1)
@@
 			)
 		)
-		(property "Footprint" "X1 Expande-easyedapro:HDR-TH_16P-P2.54-H-F-R2-C8-W9.0"
+		(property "Footprint" "x1-expander:HDR-TH_16P-P2.54-H-F-R2-C8-W9.0"
 			(at 187.96 102.87 0)
 			(effects
@@
 		)
 		(instances
-			(project "ProProject_X1 Expander_2024-05-26_15-16-51_2024-05-26"
+			(project "x1-expander"
 				(path "/5c4052f8-31d6-4de3-b862-4d09b0660e26/52713671-aa4b-4412-b159-5876c2aaf3b7"
 					(reference "BCBUS1")
@@
 	)
 	(symbol
-		(lib_id "X1 Expande-easyedapro:SRV05-4.TCT_C2687126")
+		(lib_id "x1-expander:SRV05-4.TCT_C2687126")
 		(at 48.26 128.27 270)
 		(unit 1)
@@
 			)
 		)
-		(property "Footprint" "X1 Expande-easyedapro:SOT-23-6_L2.9-W1.6-P0.95-LS2.8-BL"
+		(property "Footprint" "x1-expander:SOT-23-6_L2.9-W1.6-P0.95-LS2.8-BL"
 			(at 48.26 128.27 0)
 			(effects
@@
 		)
 		(instances
-			(project "ProProject_X1 Expander_2024-05-26_15-16-51_2024-05-26"
+			(project "x1-expander"
 				(path "/5c4052f8-31d6-4de3-b862-4d09b0660e26/52713671-aa4b-4412-b159-5876c2aaf3b7"
 					(reference "D6")
@@
 	)
 	(symbol
-		(lib_id "X1 Expande-easyedapro:SRV05-4.TCT_C2687126")
+		(lib_id "x1-expander:SRV05-4.TCT_C2687126")
 		(at 121.92 128.27 270)
 		(unit 1)
@@
 			)
 		)
-		(property "Footprint" "X1 Expande-easyedapro:SOT-23-6_L2.9-W1.6-P0.95-LS2.8-BL"
+		(property "Footprint" "x1-expander:SOT-23-6_L2.9-W1.6-P0.95-LS2.8-BL"
 			(at 121.92 128.27 0)
 			(effects
@@
 		)
 		(instances
-			(project "ProProject_X1 Expander_2024-05-26_15-16-51_2024-05-26"
+			(project "x1-expander"
 				(path "/5c4052f8-31d6-4de3-b862-4d09b0660e26/52713671-aa4b-4412-b159-5876c2aaf3b7"
 					(reference "D8")
@@
 	)
 	(symbol
-		(lib_id "X1 Expande-easyedapro:SRV05-4.TCT_C2687126")
+		(lib_id "x1-expander:SRV05-4.TCT_C2687126")
 		(at 48.26 168.91 270)
 		(unit 1)
@@
 			)
 		)
-		(property "Footprint" "X1 Expande-easyedapro:SOT-23-6_L2.9-W1.6-P0.95-LS2.8-BL"
+		(property "Footprint" "x1-expander:SOT-23-6_L2.9-W1.6-P0.95-LS2.8-BL"
 			(at 48.26 168.91 0)
 			(effects
@@
 		)
 		(instances
-			(project "ProProject_X1 Expander_2024-05-26_15-16-51_2024-05-26"
+			(project "x1-expander"
 				(path "/5c4052f8-31d6-4de3-b862-4d09b0660e26/52713671-aa4b-4412-b159-5876c2aaf3b7"
 					(reference "D7")
@@
 	)
 	(symbol
-		(lib_id "X1 Expande-easyedapro:SRV05-4.TCT_C2687126")
+		(lib_id "x1-expander:SRV05-4.TCT_C2687126")
 		(at 121.92 168.91 270)
 		(unit 1)
@@
 			)
 		)
-		(property "Footprint" "X1 Expande-easyedapro:SOT-23-6_L2.9-W1.6-P0.95-LS2.8-BL"
+		(property "Footprint" "x1-expander:SOT-23-6_L2.9-W1.6-P0.95-LS2.8-BL"
 			(at 121.92 168.91 0)
 			(effects
@@
 		)
 		(instances
-			(project "ProProject_X1 Expander_2024-05-26_15-16-51_2024-05-26"
+			(project "x1-expander"
 				(path "/5c4052f8-31d6-4de3-b862-4d09b0660e26/52713671-aa4b-4412-b159-5876c2aaf3b7"
 					(reference "D9")
@@
 	)
 	(symbol
-		(lib_id "X1 Expande-easyedapro:SRV05-4.TCT_C2687126")
+		(lib_id "x1-expander:SRV05-4.TCT_C2687126")
 		(at 121.92 43.18 270)
 		(unit 1)
@@
 			)
 		)
-		(property "Footprint" "X1 Expande-easyedapro:SOT-23-6_L2.9-W1.6-P0.95-LS2.8-BL"
+		(property "Footprint" "x1-expander:SOT-23-6_L2.9-W1.6-P0.95-LS2.8-BL"
 			(at 121.92 43.18 0)
 			(effects
@@
 		)
 		(instances
-			(project "ProProject_X1 Expander_2024-05-26_15-16-51_2024-05-26"
+			(project "x1-expander"
 				(path "/5c4052f8-31d6-4de3-b862-4d09b0660e26/52713671-aa4b-4412-b159-5876c2aaf3b7"
 					(reference "D4")
@@
 	)
 	(symbol
-		(lib_id "X1 Expande-easyedapro:S4B-PH-KL(LF)(SN)")
+		(lib_id "x1-expander:S4B-PH-KL(LF)(SN)")
 		(at 262.89 157.48 0)
 		(unit 1)
@@
 			)
 		)
-		(property "Footprint" "X1 Expande-easyedapro:CONN-TH_S4B-PH-KL-LF-SN"
+		(property "Footprint" "x1-expander:CONN-TH_S4B-PH-KL-LF-SN"
 			(at 262.89 157.48 0)
 			(effects
@@
 		)
 		(instances
-			(project "ProProject_X1 Expander_2024-05-26_15-16-51_2024-05-26"
+			(project "x1-expander"
 				(path "/5c4052f8-31d6-4de3-b862-4d09b0660e26/52713671-aa4b-4412-b159-5876c2aaf3b7"
 					(reference "I2C1")
@@
 	)
 	(symbol
-		(lib_id "X1 Expande-easyedapro:4.7k")
+		(lib_id "x1-expander:4.7k")
 		(at 237.49 151.13 90)
 		(unit 1)
@@
 		)
 		(instances
-			(project "ProProject_X1 Expander_2024-05-26_15-16-51_2024-05-26"
+			(project "x1-expander"
 				(path "/5c4052f8-31d6-4de3-b862-4d09b0660e26/52713671-aa4b-4412-b159-5876c2aaf3b7"
 					(reference "R19")
@@
 	)
 	(symbol
-		(lib_id "X1 Expande-easyedapro:10kΩ")
+		(lib_id "x1-expander:10kΩ")
 		(at 233.68 161.29 90)
 		(unit 1)
@@
 		)
 		(instances
-			(project "ProProject_X1 Expander_2024-05-26_15-16-51_2024-05-26"
+			(project "x1-expander"
 				(path "/5c4052f8-31d6-4de3-b862-4d09b0660e26/52713671-aa4b-4412-b159-5876c2aaf3b7"
 					(reference "R18")
@@
 	)
 	(symbol
-		(lib_id "X1 Expande-easyedapro:4.7k")
+		(lib_id "x1-expander:4.7k")
 		(at 243.84 163.83 90)
 		(unit 1)
@@
 		)
 		(instances
-			(project "ProProject_X1 Expander_2024-05-26_15-16-51_2024-05-26"
+			(project "x1-expander"
 				(path "/5c4052f8-31d6-4de3-b862-4d09b0660e26/52713671-aa4b-4412-b159-5876c2aaf3b7"
 					(reference "R20")
@@
 	)
 	(symbol
-		(lib_id "X1 Expande-easyedapro:HC-JN254-2-08-W")
+		(lib_id "x1-expander:HC-JN254-2-08-W")
 		(at 187.96 44.45 0)
 		(unit 1)
@@
 			)
 		)
-		(property "Footprint" "X1 Expande-easyedapro:HDR-TH_16P-P2.54-H-F-R2-C8-W9.0"
+		(property "Footprint" "x1-expander:HDR-TH_16P-P2.54-H-F-R2-C8-W9.0"
 			(at 187.96 44.45 0)
 			(effects
@@
 		)
 		(instances
-			(project "ProProject_X1 Expander_2024-05-26_15-16-51_2024-05-26"
+			(project "x1-expander"
 				(path "/5c4052f8-31d6-4de3-b862-4d09b0660e26/52713671-aa4b-4412-b159-5876c2aaf3b7"
 					(reference "ACBUS1")
@@
 	)
 	(symbol
-		(lib_id "X1 Expande-easyedapro:SRV05-4.TCT_C2687126")
+		(lib_id "x1-expander:SRV05-4.TCT_C2687126")
 		(at 48.26 43.18 270)
 		(unit 1)
@@
 			)
 		)
-		(property "Footprint" "X1 Expande-easyedapro:SOT-23-6_L2.9-W1.6-P0.95-LS2.8-BL"
+		(property "Footprint" "x1-expander:SOT-23-6_L2.9-W1.6-P0.95-LS2.8-BL"
 			(at 48.26 43.18 0)
 			(effects
@@
 		)
 		(instances
-			(project "ProProject_X1 Expander_2024-05-26_15-16-51_2024-05-26"
+			(project "x1-expander"
 				(path "/5c4052f8-31d6-4de3-b862-4d09b0660e26/52713671-aa4b-4412-b159-5876c2aaf3b7"
 					(reference "D2")
