File: x1-expander.kicad_pcb (KiCad board)
At the start: 4 copper layers, 145 x 57 mm, 111 parts, among them U1 LAN9514, U2 FT2232HL, U3 TPS54202DDCR, U4 LM1084S-3.3/TR, X1 25MHz, X2 12MHz

Commit message: rename to x1-expander
Parts:
- ACBUS1, ADBUS1, BCBUS1, BDBUS1: footprint X1 Expande-easyedapro:HDR-TH_16P-P2.54-H-F-R2-C8-W9.0 -> x1-expander:HDR-TH_16P-P2.54-H-F-R2-C8-W9.0
- AP_HARNESS1: footprint X1 Expande-easyedapro:CONN-SMD_12P-P1.25_HCTL_HC-1.25-12PWT -> x1-expander:CONN-SMD_12P-P1.25_HCTL_HC-1.25-12PWT
- D1, D2, D3, D4, D5, D6, D7, D8, D9: footprint X1 Expande-easyedapro:SOT-23-6_L2.9-W1.6-P0.95-LS2.8-BL -> x1-expander:SOT-23-6_L2.9-W1.6-P0.95-LS2.8-BL
- G***: footprint X1 Expande-easyedapro:emarhavil -> x1-expander:emarhavil
- G***: footprint X1 Expande-easyedapro:x1plus -> x1-expander:x1plus
- I2C1: footprint X1 Expande-easyedapro:CONN-TH_S4B-PH-KL-LF-SN -> x1-expander:CONN-TH_S4B-PH-KL-LF-SN
- L1: footprint X1 Expande-easyedapro:IND-SMD_L7.2-W6.6_GPSR07X0 -> x1-expander:IND-SMD_L7.2-W6.6_GPSR07X0
- LAN1: footprint X1 Expande-easyedapro:RJ45-TH_HC913550A-M899-A -> x1-expander:RJ45-TH_HC913550A-M899-A
- RN1: footprint X1 Expande-easyedapro:RES-ARRAY-SMD_0402-8P-L2.0-W1.0-BL -> x1-expander:RES-ARRAY-SMD_0402-8P-L2.0-W1.0-BL
- U1: footprint X1 Expande-easyedapro:QFN64G-0.5-9X9MM -> x1-expander:QFN64G-0.5-9X9MM
- U2: footprint X1 Expande-easyedapro:LQFP-64_L10.0-W10.0-P0.50-LS12.0-TL -> x1-expander:LQFP-64_L10.0-W10.0-P0.50-LS12.0-TL
- U3: footprint X1 Expande-easyedapro:SOT-23-6_L2.9-W1.6-P0.95-LS2.8-BL-2 -> x1-expander:SOT-23-6_L2.9-W1.6-P0.95-LS2.8-BL-2
- U4: footprint X1 Expande-easyedapro:TO-263-3_L8.6-W10.2-P2.54-LS14.4-TL -> x1-expander:TO-263-3_L8.6-W10.2-P2.54-LS14.4-TL
- UART1: footprint X1 Expande-easyedapro:HDR-TH_4P-P2.54-H-M-W10.3 -> x1-expander:HDR-TH_4P-P2.54-H-M-W10.3
- USB1, USB2: footprint X1 Expande-easyedapro:USB-TH_10.0-4C6.3-ZB -> x1-expander:USB-TH_10.0-4C6.3-ZB
- X1, X2: footprint X1 Expande-easyedapro:OSC-SMD_4P-L3.2-W2.5-BL -> x1-expander:OSC-SMD_4P-L3.2-W2.5-BL

Commit message: replace LAN1 with C375844
Parts:
- LAN1: value HC913550A-M899-A -> HR911103A; footprint x1-expander:RJ45-TH_HC913550A-M899-A -> x1-expander:RJ45-TH_HR911103A
- moved C19 9.30 mm to (82.7, 99.5)
Connections:
- LAN1 pad 10: GND -> LNKA
- LAN1 pad 11: 3V3 -> SPD
- LAN1 pad 12: LNKA -> 3V3
- LAN1 pad 13: SPD -> unconnected-(LAN1-EH-Pad13)
- LAN1 pad 3: RXP -> Net-(LAN1-RCT)
- LAN1 pad 4: Net-(LAN1-RCT) -> GND
- LAN1 pad 5: Net-(LAN1-RCT) -> GND
- LAN1 pad 6: RXN -> Net-(LAN1-RCT)
- LAN1 pad 7: unconnected-(LAN1-NC-Pad7) -> RXP
- LAN1 pad 8: GND -> RXN
- LAN1 pad 9: GND -> 3V3
Routing:
- net TXP: track 37.2 -> 42.6 mm
- net TXN: track 37.4 -> 42.8 mm
- net RXN: track 39.5 -> 36.4 mm
- net RXP: track 39.5 -> 36.6 mm
- net Net-(LAN1-RCT): track 30.8 -> 33.0 mm
- net GND: track 81.9 -> 83.2 mm, vias 171 -> 170
- net 3V3: track 103.4 -> 102.4 mm

Commit message: rotate C41 for lower impedance, replace LAN1 PTH mechanicals with NPTH
Parts:
- moved C47 1.09 mm to (141.2, 126.7), turned to 0 degrees
Routing:
- net GND: vias 170 -> 173
Changed lines of the file:
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@@
 		(at 80.105 100.635 -90)
 		(property "Reference" "LAN1"
-			(at 0 -10.9 -90)
+			(at 0 -10.9 90)
 			(layer "F.SilkS")
 			(hide yes)
@@
 		)
 		(property "Value" "HR911103A"
-			(at 0 10.9 -90)
+			(at 0 10.9 90)
 			(layer "F.Fab")
 			(effects
@@
 		)
 		(fp_text user "${REFERENCE}"
-			(at 0 0 -90)
+			(at 0 0 90)
 			(layer "F.Fab")
 			(effects
@@
 			)
 		)
-		(pad "" thru_hole circle
+		(pad "" np_thru_hole circle
 			(at -5.71 1.99 270)
 			(size 3.4 3.4)
 			(drill 3.4)
-			(layers "*.Cu" "*.Mask")
-			(remove_unused_layers no)
+			(layers "F&B.Cu" "*.Mask")
 		)
-		(pad "" thru_hole circle
+		(pad "" np_thru_hole circle
 			(at 5.75 1.99 270)
 			(size 3.4 3.4)
 			(drill 3.4)
-			(layers "*.Cu" "*.Mask")
-			(remove_unused_layers no)
+			(layers "F&B.Cu" "*.Mask")
 		)
 		(pad "1" thru_hole circle
@@
 	(footprint "Capacitor_SMD:C_1210_3225Metric"
 		(layer "F.Cu")
-		(at 141.875 125.85 90)
+		(at 141.2 126.7)
 		(descr "Capacitor SMD 1210 (3225 Metric), square (rectangular) end terminal, IPC_7351 nominal, (Body size source: IPC-SM-782 page 76, https://www.pcb-3d.com/wordpress/wp-content/uploads/ipc-sm-782a_amendment_1_and_2.pdf), generated with kicad-footprint-generator")
 		(tags "capacitor")
 		(property "Reference" "C47"
-			(at -0.775 -2.375 -90)
+			(at -0.775 -2.375 360)
 			(layer "F.SilkS")
 			(effects
@@
 		)
 		(property "Value" "100µF"
-			(at 0 2.3 -90)
+			(at 0 2.3 360)
 			(layer "F.Fab")
 			(effects
@@
 		)
 		(property "Footprint" "Capacitor_SMD:C_1210_3225Metric"
-			(at 0 0 90)
+			(at 0 0 0)
 			(unlocked yes)
 			(layer "F.Fab")
@@
 		)
 		(property "Datasheet" ""
-			(at 0 0 90)
+			(at 0 0 0)
 			(unlocked yes)
 			(layer "F.Fab")
@@
 		)
 		(property "Description" ""
-			(at 0 0 90)
+			(at 0 0 0)
 			(unlocked yes)
 			(layer "F.Fab")
@@
 		)
 		(property "Add into BOM" "yes"
-			(at 0 0 90)
+			(at 0 0 0)
 			(unlocked yes)
 			(layer "F.Fab")
@@
 		)
 		(property "Convert to PCB" "yes"
-			(at 0 0 90)
+			(at 0 0 0)
 			(unlocked yes)
 			(layer "F.Fab")
@@
 		)
 		(property "Origin Footprint" "C0603"
-			(at 0 0 90)
+			(at 0 0 0)
 			(unlocked yes)
 			(layer "F.Fab")
@@
 		)
 		(property "LCSC" "C23742"
-			(at 0 0 90)
+			(at 0 0 0)
 			(unlocked yes)
 			(layer "F.Fab")
@@
 		)
 		(fp_line
-			(start 2.3 -1.6)
-			(end 2.3 1.6)
+			(start -2.3 -1.6)
+			(end 2.3 -1.6)
 			(stroke
 				(width 0.05)
@@
 		)
 		(fp_line
-			(start -2.3 -1.6)
-			(end 2.3 -1.6)
+			(start -2.3 1.6)
+			(end -2.3 -1.6)
 			(stroke
 				(width 0.05)
@@
 		)
 		(fp_line
-			(start 2.3 1.6)
-			(end -2.3 1.6)
+			(start 2.3 -1.6)
+			(end 2.3 1.6)
 			(stroke
 				(width 0.05)
@@
 		)
 		(fp_line
-			(start -2.3 1.6)
-			(end -2.3 -1.6)
+			(start 2.3 1.6)
+			(end -2.3 1.6)
 			(stroke
 				(width 0.05)
@@
 		)
 		(fp_line
-			(start 1.6 -1.25)
-			(end 1.6 1.25)
+			(start -1.6 -1.25)
+			(end 1.6 -1.25)
 			(stroke
 				(width 0.1)
@@
 		)
 		(fp_line
-			(start -1.6 -1.25)
-			(end 1.6 -1.25)
+			(start -1.6 1.25)
+			(end -1.6 -1.25)
 			(stroke
 				(width 0.1)
@@
 		)
 		(fp_line
-			(start 1.6 1.25)
-			(end -1.6 1.25)
+			(start 1.6 -1.25)
+			(end 1.6 1.25)
 			(stroke
 				(width 0.1)
@@
 		)
 		(fp_line
-			(start -1.6 1.25)
-			(end -1.6 -1.25)
+			(start 1.6 1.25)
+			(end -1.6 1.25)
 			(stroke
 				(width 0.1)
@@
 		)
 		(fp_text user "${REFERENCE}"
-			(at 0 0 -90)
+			(at 0 0 360)
 			(layer "F.Fab")
 			(effects
@@
 		)
 		(pad "1" smd roundrect
-			(at -1.475 0 90)
+			(at -1.475 0)
 			(size 1.15 2.7)
 			(layers "F.Cu" "F.Paste" "F.Mask")
@@
 		)
 		(pad "2" smd roundrect
-			(at 1.475 0 90)
+			(at 1.475 0)
 			(size 1.15 2.7)
 			(layers "F.Cu" "F.Paste" "F.Mask")
@@
 	)
 	(via
+		(at 139.875 128.75)
+		(size 0.6096)
+		(drill 0.3048)
+		(layers "F.Cu" "B.Cu")
+		(free yes)
+		(net 3)
+	)
+	(via
 		(at 99.25 127.625)
 		(size 0.6096)
@@
 	)
 	(via
-		(at 139.875 127)
-		(size 0.6096)
-		(drill 0.3048)
-		(layers "F.Cu" "B.Cu")
-		(free yes)
-		(net 3)
-	)
-	(via
 		(at 103.875 124.125)
 		(size 0.6096)
@@
 	)
 	(via
+		(at 138.625 127.125)
+		(size 0.6096)
+		(drill 0.3048)
+		(layers "F.Cu" "B.Cu")
+		(free yes)
+		(net 3)
+	)
+	(via
 		(at 107.875 130.625)
 		(size 0.6096)
@@
 	)
 	(via
+		(at 138.625 126.25)
+		(size 0.6096)
+		(drill 0.3048)
+		(layers "F.Cu" "B.Cu")
+		(free yes)
+		(net 3)
+	)
+	(via
 		(at 87 109.5)
 		(size 0.6)
@@
 	)
 	(via
+		(at 138 125.625)
+		(size 0.6096)
+		(drill 0.3048)
+		(layers "F.Cu" "B.Cu")
+		(free yes)
+		(net 3)
+	)
+	(via
 		(at 190.75 106.25)
 		(size 0.6)
@@
 	)
 	(via
+		(at 139 128.75)
+		(size 0.6096)
+		(drill 0.3048)
+		(layers "F.Cu" "B.Cu")
+		(free yes)
+		(net 3)
+	)
+	(via
 		(at 96.875 118)
 		(size 0.6096)
@@
 	)
 	(via
+		(at 138.625 128)
+		(size 0.6096)
+		(drill 0.3048)
+		(layers "F.Cu" "B.Cu")
+		(free yes)
+		(net 3)
+	)
+	(via
 		(at 140.625 137.375)
 		(size 0.6096)
@@
 	)
 	(via
-		(at 139.875 127.875)
-		(size 0.6096)
-		(drill 0.3048)
-		(layers "F.Cu" "B.Cu")
-		(free yes)
-		(net 3)
-	)
-	(via
 		(at 101.625 125.125)
 		(size 0.6096)
@@
 	)
 	(via
-		(at 139.875 128.75)
-		(size 0.6096)
-		(drill 0.3048)
-		(layers "F.Cu" "B.Cu")
-		(free yes)
-		(net 3)
-	)
-	(via
 		(at 188.5 107.875)
 		(size 0.6)
@@
 	)
 	(segment
+		(start 93.529531 125)
+		(end 93.375 125)
+		(width 0.2)
+		(layer "B.Cu")
+		(net 72)
+	)
+	(segment
 		(start 99.625 132.458522)
 		(end 97.5202 130.353722)
@@
 	)
 	(segment
-		(start 97.5202 130.353722)
-		(end 97.5202 128.990669)
+		(start 82.973 114.598)
+		(end 82.973 105.75)
 		(width 0.2)
 		(layer "B.Cu")
@@
 	)
 	(segment
-		(start 97.5202 128.990669)
-		(end 93.529531 125)
+		(start 82.973 105.75)
+		(end 82.925 105.75)
 		(width 0.2)
 		(layer "B.Cu")
@@
 	)
 	(segment
-		(start 93.529531 125)
-		(end 93.375 125)
+		(start 93.375 125)
+		(end 82.973 114.598)
 		(width 0.2)
 		(layer "B.Cu")
@@
 	)
 	(segment
-		(start 82.585 105.41)
-		(end 75.375 98.2)
+		(start 97.5202 130.353722)
+		(end 97.5202 128.990669)
 		(width 0.2)
 		(layer "B.Cu")
@@
 	)
 	(segment
-		(start 99.625 133.025)
-		(end 99.625 132.458522)
+		(start 97.5202 128.990669)
+		(end 93.529531 125)
 		(width 0.2)
 		(layer "B.Cu")
@@
 	)
 	(segment
-		(start 93.375 125)
-		(end 82.585 114.21)
+		(start 99.625 133.025)
+		(end 99.625 132.458522)
 		(width 0.2)
 		(layer "B.Cu")
@@
 	)
 	(segment
-		(start 82.585 114.21)
-		(end 82.585 105.41)
+		(start 82.925 105.75)
+		(end 75.375 98.2)
 		(width 0.2)
 		(layer "B.Cu")

Commit message: 5V switcher routing improvements
Routing:
- net 5V: track 44.2 -> 47.2 mm
- net GND: vias 173 -> 172
Changed lines of the file:
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@@
 	)
 	(via
-		(at 150.125 129.25)
+		(at 150.25 129.25)
 		(size 0.6)
 		(drill 0.3)
@@
 	)
 	(via
-		(at 150.125 131)
+		(at 150.25 131)
 		(size 0.6)
 		(drill 0.3)
@@
 	)
 	(via
-		(at 150.125 128.375)
-		(size 0.6)
-		(drill 0.3)
-		(layers "F.Cu" "B.Cu")
-		(free yes)
-		(net 3)
-	)
-	(via
 		(at 103.875 126.2588)
 		(size 0.6096)
@@
 	)
 	(via
-		(at 150.125 130.125)
+		(at 150.25 130.125)
 		(size 0.6)
 		(drill 0.3)
@@
 	)
 	(via
+		(at 150.625 119.375)
+		(size 0.6096)
+		(drill 0.3048)
+		(layers "F.Cu" "B.Cu")
+		(free yes)
+		(net 3)
+	)
+	(via
 		(at 100.375 124.125)
 		(size 0.6096)
@@
 	)
 	(via
-		(at 150.875 128.75)
-		(size 0.6)
-		(drill 0.3)
-		(layers "F.Cu" "B.Cu")
-		(free yes)
-		(net 3)
-	)
-	(via
 		(at 174.125 118.875)
 		(size 0.6096)
@@
 	)
 	(via
-		(at 150.875 129.625)
+		(at 151 129.625)
 		(size 0.6)
 		(drill 0.3)
@@
 	)
 	(segment
-		(start 154.37 119.37)
-		(end 160.125 125.125)
-		(width 0.8)
-		(layer "B.Cu")
-		(net 4)
-	)
-	(segment
 		(start 70.625 112.875)
 		(end 70.625 114.125)
@@
 	)
 	(segment
-		(start 154.37 116.8)
-		(end 154.37 119.37)
-		(width 0.8)
-		(layer "B.Cu")
-		(net 4)
-	)
-	(segment
 		(start 101.24175 91.91675)
 		(end 98.70175 91.91675)
@@
 	)
 	(segment
+		(start 154.37 116.8)
+		(end 158.05 116.8)
+		(width 0.8)
+		(layer "B.Cu")
+		(net 4)
+	)
+	(segment
 		(start 72.75 125.149)
 		(end 72.75 125.875)
@@
 	)
 	(segment
+		(start 158.05 116.8)
+		(end 160.125 118.875)
+		(width 0.8)
+		(layer "B.Cu")
+		(net 4)
+	)
+	(segment
 		(start 159.24175 91.91675)
 		(end 156.70175 91.91675)
@@
 	)
 	(segment
+		(start 160.125 118.875)
+		(end 160.125 125.975)
+		(width 0.8)
+		(layer "B.Cu")
+		(net 4)
+	)
+	(segment
 		(start 70.625 113.5)
 		(end 71.6 113.5)
@@
 	(segment
 		(start 71.8 127.172)
-		(end 71.8 125.149)
-		(width 0.2)
+		(end 77.103 132.475)
+		(width 0.3)
 		(layer "B.Cu")
 		(net 11)
 	)
 	(segment
-		(start 77.103 132.475)
+		(start 71.8 125.149)
 		(end 71.8 127.172)
-		(width 0.2)
+		(width 0.3)
 		(layer "B.Cu")
 		(net 11)
@@
 		(layer "F.Cu")
 		(hatch edge 0.5)
-		(priority 4)
+		(priority 5)
 		(connect_pads yes
-			(clearance 0.127)
+			(clearance 0.3)
 		)
 		(min_thickness 0.25)
@@
 		(polygon
 			(pts
-				(xy 145.625 128.475) (xy 149.625 128.475) (xy 149.625 131.1) (xy 148 131.1) (xy 148 132.85) (xy 147.25 132.85)
+				(xy 145.625 128.225) (xy 149.625 128.225) (xy 149.625 131.1) (xy 148 131.1) (xy 148 132.85) (xy 147.25 132.85)
 				(xy 147.25 131.1) (xy 145.625 131.1)
 			)

Commit message: repair ADBUS0 and ADBUS1 routing
Routing:
- net ADBUS1: track 41.9 -> 42.6 mm
Changed lines of the file:
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@@
+	)
+	(segment
+		(start 181.125 102.375)
+		(end 178.347 99.597)
+		(width 0.127)
+		(layer "B.Cu")
+		(net 23)
 	)
 	(segment
@@
 	)
 	(segment
-		(start 182.7 102.375)
-		(end 179.922 99.597)
+		(start 178.347 99.597)
+		(end 178 99.597)
 		(width 0.127)
 		(layer "B.Cu")
@@
 	)
 	(segment
+		(start 182.7 102.375)
+		(end 181.125 102.375)
+		(width 0.127)
+		(layer "B.Cu")
+		(net 23)
+	)
+	(segment
 		(start 151.55275 87.06325)
 		(end 147.91825 90.69775)
@@
 	)
 	(segment
-		(start 179.922 99.597)
+		(start 178 99.597)
 		(end 165.393909 99.597)
 		(width 0.127)
@@
 	)
 	(segment
+		(start 150.45825 93.29325)
+		(end 151.62175 94.45675)
+		(width 0.127)
+		(layer "B.Cu")
+		(net 27)
+	)
+	(segment
+		(start 151.82275 88.96325)
+		(end 150.45825 90.32775)
+		(width 0.127)
+		(layer "B.Cu")
+		(net 27)
+	)
+	(segment
+		(start 184.5 100.575)
+		(end 184.5 99.5)
+		(width 0.127)
+		(layer "B.Cu")
+		(net 27)
+	)
+	(segment
+		(start 156.316 99.1095)
+		(end 151.65 94.4435)
+		(width 0.127)
+		(layer "B.Cu")
+		(net 27)
+	)
+	(segment
+		(start 165.529357 99.27)
+		(end 165.368857 99.1095)
+		(width 0.127)
+		(layer "B.Cu")
+		(net 27)
+	)
+	(segment
+		(start 184.5 99.5)
+		(end 184.27 99.27)
+		(width 0.127)
+		(layer "B.Cu")
+		(net 27)
+	)
+	(segment
 		(start 165.368857 99.1095)
 		(end 156.316 99.1095)
@@
 	)
 	(segment
-		(start 183.195 99.27)
-		(end 165.529357 99.27)
-		(width 0.127)
-		(layer "B.Cu")
-		(net 27)
-	)
-	(segment
-		(start 165.529357 99.27)
-		(end 165.368857 99.1095)
-		(width 0.127)
-		(layer "B.Cu")
-		(net 27)
-	)
-	(segment
-		(start 150.45825 93.29325)
-		(end 151.62175 94.45675)
-		(width 0.127)
-		(layer "B.Cu")
-		(net 27)
-	)
-	(segment
-		(start 184.5 100.575)
-		(end 183.195 99.27)
-		(width 0.127)
-		(layer "B.Cu")
-		(net 27)
-	)
-	(segment
-		(start 156.316 99.1095)
-		(end 151.65 94.4435)
-		(width 0.127)
-		(layer "B.Cu")
-		(net 27)
-	)
-	(segment
-		(start 151.82275 88.96325)
-		(end 150.45825 90.32775)
-		(width 0.127)
-		(layer "B.Cu")
-		(net 27)
-	)
-	(segment
 		(start 150.45825 90.32775)
 		(end 150.45825 93.29325)
 		(width 0.127)
 		(layer "B.Cu")
+		(net 27)
+	)
+	(segment
+		(start 184.27 99.27)
+		(end 165.529357 99.27)
+		(width 0.127)
+		(layer "B.Cu")

Commit message: put FTDI VCORE on In2.Cu
Routing:
- net VCORE: track 37.2 -> 11.4 mm
- added copper zone on In2.Cu, net VCORE
Changed lines of the file:
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@@
 	)
 	(segment
-		(start 183.625 112.625)
-		(end 191.971646 112.625)
-		(width 0.3)
-		(layer "F.Cu")
-		(net 60)
-	)
-	(segment
-		(start 192.070904 112.724258)
-		(end 193.025 111.770162)
-		(width 0.3)
-		(layer "F.Cu")
-		(net 60)
-	)
-	(segment
 		(start 192.375 104.5)
 		(end 192.375 104.375)
@@
 		(net 60)
 	)
-	(segment
-		(start 183.475 104.9)
-		(end 184 104.375)
-		(width 0.3)
-		(layer "F.Cu")
-		(net 60)
-	)
-	(segment
-		(start 183.475 112.475)
-		(end 183.475 104.9)
-		(width 0.3)
-		(layer "F.Cu")
-		(net 60)
-	)
-	(segment
-		(start 183.625 112.625)
-		(end 183.475 112.475)
-		(width 0.3)
-		(layer "F.Cu")
-		(net 60)
-	)
-	(segment
-		(start 193.025 105.15)
-		(end 192.375 104.5)
-		(width 0.3)
-		(layer "F.Cu")
-		(net 60)
-	)
-	(segment
-		(start 193.025 111.770162)
-		(end 193.025 105.15)
-		(width 0.3)
-		(layer "F.Cu")
-		(net 60)
-	)
 	(via
 		(at 192.375 104.375)
@@
 			)
 		)
+	)
+	(zone
+		(net 60)
+		(net_name "VCORE")
+		(layer "In2.Cu")
+		(hatch edge 0.5)
+		(priority 4)
+		(connect_pads yes
+			(clearance 0.3)
+		)
+		(min_thickness 0.25)
+		(filled_areas_thickness no)
+		(fill yes
+			(thermal_gap 0.5)
+			(thermal_bridge_width 0.5)
+			(smoothing fillet)
+			(radius 0.2)
+		)
+		(polygon
+			(pts
+				(xy 181.125 103.25) (xy 193.625 103.25) (xy 193.625 106.125) (xy 193.625 106.125) (xy 193.625 111.5)
+				(xy 193.625 111.5) (xy 193.625 113.875) (xy 181.125 113.875)
+			)
+		)
