File: x1-expander.kicad_pcb (KiCad board)
At the start: 4 copper layers, 145 x 57 mm, 111 parts, among them U1 LAN9514, U2 FT2232HL, U3 TPS54202DDCR, U4 LM1084S-3.3/TR, X1 25MHz, X2 12MHz

Commit message: move vdd18core to inner layer
Routing:
- net /LAN/VDD18CORE: track 33.1 -> 7.11 mm, vias 0 -> 2
- added copper zone on In2.Cu, net /LAN/VDD18CORE
Changed lines of the file:
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@@
 	)
 	(segment
-		(start 110.7798 131.249781)
-		(end 105.029581 137)
-		(width 0.8)
+		(start 107.625 128.35)
+		(end 106.725 128.35)
+		(width 0.2)
 		(layer "F.Cu")
 		(net 53)
 	)
 	(segment
-		(start 94.775 130.908)
-		(end 94.775 129.875)
-		(width 0.8)
+		(start 94.775 129.875)
+		(end 94.775 130.15)
+		(width 0.3)
 		(layer "F.Cu")
 		(net 53)
@@
 	(segment
 		(start 105.5465 128.2445)
+		(end 106.6195 128.2445)
+		(width 0.2)
+		(layer "F.Cu")
+		(net 53)
+	)
+	(segment
+		(start 107.3805 128.2445)
 		(end 107.5195 128.2445)
 		(width 0.2)
@@
 	)
 	(segment
-		(start 96.4535 130.251)
-		(end 95.151 130.251)
+		(start 95.624 130.251)
+		(end 95.25 130.625)
 		(width 0.3)
 		(layer "F.Cu")
@@
 	)
 	(segment
-		(start 96.7798 132.9128)
-		(end 94.775 130.908)
-		(width 0.8)
+		(start 96.4535 130.251)
+		(end 95.624 130.251)
+		(width 0.3)
 		(layer "F.Cu")
 		(net 53)
@@
 	)
 	(segment
-		(start 105.029581 137)
-		(end 98 137)
-		(width 0.8)
-		(layer "F.Cu")
-		(net 53)
-	)
-	(segment
-		(start 109.40901 128.175)
-		(end 110.7798 129.54579)
-		(width 0.8)
+		(start 106.725 128.35)
+		(end 106.6195 128.2445)
+		(width 0.2)
 		(layer "F.Cu")
 		(net 53)
 	)
 	(segment
-		(start 96.7798 135.7798)
-		(end 96.7798 132.9128)
-		(width 0.8)
+		(start 94.775 130.15)
+		(end 95.25 130.625)
+		(width 0.3)
 		(layer "F.Cu")
 		(net 53)
 	)
 	(segment
-		(start 98 137)
-		(end 96.7798 135.7798)
-		(width 0.8)
+		(start 107 128.625)
+		(end 107.3805 128.2445)
+		(width 0.2)
 		(layer "F.Cu")
 		(net 53)
 	)
-	(segment
-		(start 110.7798 129.54579)
-		(end 110.7798 131.249781)
-		(width 0.8)
-		(layer "F.Cu")
+	(via
+		(at 95.25 130.625)
+		(size 0.6096)
+		(drill 0.3048)
+		(layers "F.Cu" "B.Cu")
 		(net 53)
 	)
-	(segment
-		(start 95.151 130.251)
-		(end 94.775 129.875)
-		(width 0.3)
-		(layer "F.Cu")
+	(via
+		(at 107 128.625)
+		(size 0.6096)
+		(drill 0.3048)
+		(layers "F.Cu" "B.Cu")
 		(net 53)
 	)
@@
 		(polygon
 			(pts
-				(xy 97.25 135) (xy 92.625 135) (xy 92.625 127.125) (xy 94.125 127.125) (xy 94.125 120.375) (xy 98 120.375)
+				(xy 97.25 135) (xy 91 135) (xy 91 127.125) (xy 94.125 127.125) (xy 94.125 120.375) (xy 98 120.375)
 				(xy 98 112.875) (xy 106.75 112.875) (xy 106.75 123.25) (xy 97.375 123.125)
 			)
@@
 			)
 		)
+	)
+	(zone
+		(net 53)
+		(net_name "/LAN/VDD18CORE")
+		(layer "In2.Cu")
+		(hatch edge 0.5)
+		(priority 14)
+		(connect_pads yes
+			(clearance 0.3)
+		)
+		(min_thickness 0.25)
+		(filled_areas_thickness no)
+		(fill yes
+			(thermal_gap 0.5)
+			(thermal_bridge_width 0.5)
+			(smoothing fillet)
+			(radius 0.2)
+		)
+		(polygon
+			(pts
+				(xy 94.25 129.125) (xy 94.25 132.125) (xy 106.125 132.217637) (xy 106.125 129.125) (xy 107.25 129.125)
+				(xy 107.25 127.5) (xy 97.375 127.5) (xy 97.375 129.125)
+			)
+		)

Commit message: staple ground planes with 5mm via grid
Routing:
- net GND: vias 172 -> 303

Commit message: remove a few strange off-grid vias
Routing:
- net GND: vias 303 -> 292
Changed lines of the file:
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@@
 	)
 	(via
-		(at 139 120.625)
+		(at 139.25 120.125)
 		(size 0.6096)
 		(drill 0.3048)
@@
 	)
 	(via
-		(at 192.875 118.875)
-		(size 0.6096)
-		(drill 0.3048)
-		(layers "F.Cu" "B.Cu")
-		(free yes)
-		(net 3)
-	)
-	(via
 		(at 130 85)
 		(size 0.6096)
@@
 	)
 	(via
-		(at 87 109.5)
-		(size 0.6)
-		(drill 0.3)
-		(layers "F.Cu" "B.Cu")
-		(net 3)
-	)
-	(via
 		(at 70 130)
 		(size 0.6096)
@@
 	)
 	(via
-		(at 126 133.25)
-		(size 0.6096)
-		(drill 0.3048)
-		(layers "F.Cu" "B.Cu")
-		(free yes)
-		(net 3)
-	)
-	(via
 		(at 72.75 122)
 		(size 0.6096)
@@
 	)
 	(via
+		(at 160 115)
+		(size 0.6096)
+		(drill 0.3048)
+		(layers "F.Cu" "B.Cu")
+		(free yes)
+		(net 3)
+	)
+	(via
 		(at 109 130.875)
 		(size 0.6096)
@@
 	)
 	(via
-		(at 138 125.625)
-		(size 0.6096)
-		(drill 0.3048)
-		(layers "F.Cu" "B.Cu")
-		(free yes)
-		(net 3)
-	)
-	(via
 		(at 190.75 106.25)
 		(size 0.6)
@@
 	)
 	(via
-		(at 109.25 116.25)
-		(size 0.6096)
-		(drill 0.3048)
-		(layers "F.Cu" "B.Cu")
-		(free yes)
-		(net 3)
-	)
-	(via
 		(at 108.375 135.25)
 		(size 0.6096)
@@
 	)
 	(via
-		(at 102 109.25)
+		(at 101.75 109)
 		(size 0.6096)
 		(drill 0.3048)
@@
 	)
 	(via
-		(at 113.875 120.625)
-		(size 0.6096)
-		(drill 0.3048)
-		(layers "F.Cu" "B.Cu")
-		(free yes)
-		(net 3)
-	)
-	(via
 		(at 200 95)
 		(size 0.6096)
@@
 	)
 	(via
-		(at 126 120.625)
-		(size 0.6096)
-		(drill 0.3048)
-		(layers "F.Cu" "B.Cu")
-		(free yes)
-		(net 3)
-	)
-	(via
 		(at 139 128.75)
 		(size 0.6096)
@@
 	)
 	(via
-		(at 131.25 132.25)
-		(size 0.6096)
-		(drill 0.3048)
-		(layers "F.Cu" "B.Cu")
-		(free yes)
-		(net 3)
-	)
-	(via
 		(at 110.125 126.7588)
 		(size 0.6096)
@@
 	)
 	(via
-		(at 126 122.5)
-		(size 0.6096)
-		(drill 0.3048)
-		(layers "F.Cu" "B.Cu")
-		(free yes)
-		(net 3)
-	)
-	(via
 		(at 149.25 131.85)
 		(size 0.6)
@@
 	)
 	(via
-		(at 168 118.875)
-		(size 0.6096)
-		(drill 0.3048)
-		(layers "F.Cu" "B.Cu")
-		(free yes)
-		(net 3)
-	)
-	(via
-		(at 174.125 118.875)
-		(size 0.6096)
-		(drill 0.3048)
-		(layers "F.Cu" "B.Cu")
-		(free yes)
-		(net 3)
-	)
-	(via
 		(at 102.75 128.75)
 		(size 0.6096)
@@
 	)
 	(via
-		(at 136.25 124.5)
-		(size 0.6096)
-		(drill 0.3048)
-		(layers "F.Cu" "B.Cu")
-		(free yes)
-		(net 3)
-	)
-	(via
 		(at 199.625 132)
 		(size 0.6)
@@
 	)
 	(via
-		(at 139 122.5)
+		(at 139.25 123)
 		(size 0.6096)
 		(drill 0.3048)
@@
 	)
 	(via
-		(at 90.75 107.125)
-		(size 0.6096)
-		(drill 0.3048)
+		(at 90.5 105.5)
+		(size 0.6096)
+		(drill 0.3048)

Commit message: add esd protection to uart
Parts:
- added D10: SRV05-4.TCT_C2687126, x1-expander:SOT-23-6_L2.9-W1.6-P0.95-LS2.8-BL, B.Cu at (207.0, 87.8)
Connections:
- AP_HARNESS1 pad 6: UART3V3 -> unconnected-(AP_HARNESS1-Pad6)
- UART1 pad 1: UART3V3 -> 3V3
Routing:
- net UART3V3: track 107.5 -> 0.00 mm, vias 2 -> 0
- net 3V3: track 102.4 -> 117.5 mm, vias 43 -> 44
- net UARTRX: track 111.4 -> 111.9 mm
- net GND: vias 292 -> 293

Commit message: pcb: gpio 5v from inner layer, fatten ap dbg 3v3
Routing:
- net 5V: track 47.2 -> 20.0 mm, vias 23 -> 19
- net BDBUS1: track 154.7 -> 153.6 mm
- net BDBUS2: track 137.5 -> 138.3 mm
- net GND: vias 293 -> 292
