File: x1-expander.kicad_pcb (KiCad board)
At the start: 4 copper layers, 145 x 57 mm, 120 parts, among them U1 LAN9514, U2 FT2232HL, U3 TPS54202DDCR, U4 LM1084S-3.3/TR, U5 M93C86-WMN6TP, X1 25MHz, X2 12MHz

Commit message: place eeprom, move LAN9514 north, route ethernet
Parts:
- moved R33 28.9 mm to (96.5, 130.8), turned to -90 degrees
- moved C48 28.2 mm to (96.5, 133.4), turned to -90 degrees
- moved U5 20.6 mm to (101.0, 132.0), turned to 180 degrees
- moved R34 19.9 mm to (103.0, 135.3), turned to 0 degrees
- moved X1 4.02 mm to (95.5, 113.4)
- moved C10 4.02 mm to (93.3, 114.3)
- moved C11 4.02 mm to (107.6, 125.5)
- moved C12 4.02 mm to (96.5, 126.2)
- moved C13 4.02 mm to (105.2, 124.6)
- moved C14 4.02 mm to (104.9, 126.7)
- moved C15 4.02 mm to (105.0, 120.2)
- moved C16 4.02 mm to (98.0, 127.2)
- moved C17 4.02 mm to (102.0, 127.2)
- moved C18 4.02 mm to (105.5, 123.6)
- moved C21 4.02 mm to (96.4, 121.2)
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Routing:
- net TXN: track 8.76 -> 37.2 mm
- net TXP: track 9.87 -> 34.1 mm
- net /LAN/EECS: track 0.00 -> 11.9 mm
- net RXP: track 26.3 -> 34.5 mm
- net RXN: track 26.2 -> 34.2 mm
- net /LAN/EECLK: track 0.00 -> 7.11 mm
- net /LAN/EEMOSI: track 0.00 -> 5.42 mm
- net /LAN/EEMISO: track 0.00 -> 3.97 mm
- net 3V3: track 120.4 -> 123.3 mm, vias 40 -> 41
- net GND: track 77.6 -> 79.7 mm, vias 264 -> 263
- net Net-(U5-ORG): track 0.00 -> 2.01 mm

Commit message: Bani6809/power led (#20)
* add power led

* fix crlf
Parts:
- added LED1: KT-0603R, x1-expander:LED0603-RD, F.Cu at (70.0, 131.7)
- added R35: 330, Resistor_SMD:R_0603_1608Metric, F.Cu at (73.3, 131.6)
Routing:
- net 5V: track 18.4 -> 27.1 mm
- net Net-(LED1-K): track 0.00 -> 1.70 mm

Commit message: swap USB connectors
Parts:
- USB1, USB2: value AF 14.0 CC-T -> USB-226-BRW; footprint x1-expander:USB-A-TH_AF14.0CC-T -> x1-expander:USB-A-TH_USB-226-BRW
- moved D1 7.78 mm to (82.4, 120.6)
- moved R23 7.52 mm to (89.5, 119.4)
- moved R22 6.89 mm to (89.5, 118.0)
- moved USB2 6.33 mm to (82.3, 125.6)
- moved USB1 6.26 mm to (82.3, 116.5)
Routing:
- net GND: vias 263 -> 242

Commit message: route USB ports
Parts:
- removed R22, R23, R24, R25: 0, Resistor_SMD:R_0603_1608Metric
- C45, C46: moved to B.Cu
- moved C45 8.86 mm to (75.4, 118.0), turned to 90 degrees
- moved C46 8.41 mm to (75.4, 124.1), turned to -90 degrees
- moved F2 2.21 mm to (71.5, 115.1), turned to -90 degrees
- moved LED1 0.25 mm to (70.2, 131.6)
- moved R35 0.20 mm to (73.5, 131.6)
Connections:
- D1 pad 4: USB2_DN -> USB2_DP
- D1 pad 5: 5V -> Net-(USB1-VBUS)
- D1 pad 6: USB2_DP -> USB2_DN
- U1 pad 1: /LAN/USB1R_DN -> USB1_DN
- U1 pad 2: /LAN/USB1R_DP -> USB1_DP
- U1 pad 3: /LAN/USB2R_DN -> USB2_DN
- U1 pad 4: /LAN/USB2R_DP -> USB2_DP
Routing:
- net USB1_DP: track 0.00 -> 31.0 mm
- net Net-(USB1-VBUS): track 2.71 -> 31.3 mm
- net USB1_DN: track 0.00 -> 28.1 mm
- net USB2_DN: track 0.00 -> 23.3 mm
- net USB2_DP: track 0.00 -> 23.3 mm
- net Net-(LAN1-RCT): track 23.9 -> 13.3 mm
- net Net-(U1-nLNKA_LED/GPIO1): track 19.6 -> 10.7 mm
- net 5V: track 27.1 -> 25.3 mm

Commit message: escape other USB diff pairs
Routing:
- net FTDI_DN: track 118.3 -> 132.6 mm
- net FTDI_DP: track 117.9 -> 131.5 mm
- net /LAN/CAMOR_DN: track 62.8 -> 75.1 mm
- net /LAN/CAMOR_DP: track 63.9 -> 75.6 mm
Changed lines of the file:
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@@
 	)
 	(segment
+		(start 88.8043 123.44927)
+		(end 88.8043 129.125)
+		(width 0.1554)
+		(layer "F.Cu")
+		(net 11)
+	)
+	(segment
+		(start 94.720161 122.16725)
+		(end 90.08632 122.16725)
+		(width 0.1554)
+		(layer "F.Cu")
+		(net 11)
+	)
+	(segment
+		(start 90.08632 122.16725)
+		(end 88.8043 123.44927)
+		(width 0.1554)
+		(layer "F.Cu")
+		(net 11)
+	)
+	(segment
 		(start 170.8207 122.5229)
 		(end 170.5936 122.75)
@@
 	)
 	(segment
+		(start 94.735192 122.18228)
+		(end 94.720161 122.16725)
+		(width 0.1554)
+		(layer "F.Cu")
+		(net 11)
+	)
+	(segment
 		(start 170.8207 107.3521)
 		(end 170.8207 122.5229)
@@
 	)
 	(segment
+		(start 95.405829 122.18228)
+		(end 94.735192 122.18228)
+		(width 0.1554)
+		(layer "F.Cu")
+		(net 11)
+	)
+	(segment
+		(start 96.2035 122.2292)
+		(end 95.452749 122.2292)
+		(width 0.1554)
+		(layer "F.Cu")
+		(net 11)
+	)
+	(segment
+		(start 95.452749 122.2292)
+		(end 95.405829 122.18228)
+		(width 0.1554)
+		(layer "F.Cu")
+		(net 11)
+	)
+	(segment
 		(start 170.5936 107.125)
 		(end 170.8207 107.3521)
@@
 	)
 	(segment
+		(start 88.4457 123.30073)
+		(end 88.4457 129.125)
+		(width 0.1554)
+		(layer "F.Cu")
+		(net 114)
+	)
+	(segment
 		(start 171.1793 122.5229)
 		(end 171.4064 122.75)
@@
 	)
 	(segment
+		(start 94.88372 121.8237)
+		(end 94.86867 121.80865)
+		(width 0.1554)
+		(layer "F.Cu")
+		(net 114)
+	)
+	(segment
 		(start 171.1793 107.3521)
 		(end 171.1793 122.5229)
@@
 	)
 	(segment
+		(start 94.86867 121.80865)
+		(end 89.93778 121.80865)
+		(width 0.1554)
+		(layer "F.Cu")
+		(net 114)
+	)
+	(segment
+		(start 95.375749 121.8237)
+		(end 94.88372 121.8237)
+		(width 0.1554)
+		(layer "F.Cu")
+		(net 114)
+	)
+	(segment
 		(start 171.4064 107.125)
 		(end 171.1793 107.3521)
@@
 		(net 114)
 	)
+	(segment
+		(start 96.2035 121.7467)
+		(end 95.452749 121.7467)
+		(width 0.1554)
+		(layer "F.Cu")
+		(net 114)
+	)
+	(segment
+		(start 89.93778 121.80865)
+		(end 88.4457 123.30073)
+		(width 0.1554)
+		(layer "F.Cu")
+		(net 114)
+	)
+	(segment
+		(start 95.452749 121.7467)
+		(end 95.375749 121.8237)
+		(width 0.1554)
+		(layer "F.Cu")
+		(net 114)
+	)
 	(via
 		(at 171.4064 122.75)
@@
 	)
 	(segment
+		(start 92.25308 123.1705)
+		(end 92.24128 123.1587)
+		(width 0.1554)
+		(layer "F.Cu")
+		(net 116)
+	)
+	(segment
+		(start 90.3043 123.69927)
+		(end 90.3043 129.25)
+		(width 0.1554)
+		(layer "F.Cu")
+		(net 116)
+	)
+	(segment
+		(start 91.75872 123.1587)
+		(end 91.74692 123.1705)
+		(width 0.1554)
+		(layer "F.Cu")
+		(net 116)
+	)
+	(segment
+		(start 95.378049 123.1705)
+		(end 92.25308 123.1705)
+		(width 0.1554)
+		(layer "F.Cu")
+		(net 116)
+	)
+	(segment
+		(start 95.452749 123.2452)
+		(end 95.378049 123.1705)
+		(width 0.1554)
+		(layer "F.Cu")
+		(net 116)
+	)
+	(segment
+		(start 91.74692 123.1705)
+		(end 90.83307 123.1705)
+		(width 0.1554)
+		(layer "F.Cu")
+		(net 116)
+	)
+	(segment
+		(start 92.24128 123.1587)
+		(end 91.75872 123.1587)
+		(width 0.1554)
+		(layer "F.Cu")
+		(net 116)
+	)
+	(segment
+		(start 90.83307 123.1705)
+		(end 90.3043 123.69927)
+		(width 0.1554)
+		(layer "F.Cu")
+		(net 116)
+	)
+	(segment
+		(start 96.2035 123.2452)
+		(end 95.452749 123.2452)
+		(width 0.1554)
+		(layer "F.Cu")
+		(net 116)
+	)
+	(segment
 		(start 97.57427 134.0707)
 		(end 106.75572 134.0707)
@@
 	)
 	(segment
+		(start 90.68453 122.8119)
+		(end 89.9457 123.55073)
+		(width 0.1554)
+		(layer "F.Cu")
+		(net 117)
+	)
+	(segment
+		(start 89.9457 123.55073)
+		(end 89.9457 129.25)
+		(width 0.1554)
+		(layer "F.Cu")
+		(net 117)
+	)
+	(segment
+		(start 91.610192 122.80012)
+		(end 91.598411 122.8119)
+		(width 0.1554)
+		(layer "F.Cu")
+		(net 117)
+	)
+	(segment
+		(start 91.598411 122.8119)
+		(end 90.68453 122.8119)
+		(width 0.1554)
+		(layer "F.Cu")
+		(net 117)
+	)
+	(segment
+		(start 95.378049 122.8119)
+		(end 92.401588 122.8119)
+		(width 0.1554)
+		(layer "F.Cu")
+		(net 117)
+	)
+	(segment
+		(start 95.452749 122.7372)
+		(end 95.378049 122.8119)
+		(width 0.1554)
+		(layer "F.Cu")
+		(net 117)
+	)
+	(segment
+		(start 96.2035 122.7372)
+		(end 95.452749 122.7372)
+		(width 0.1554)
+		(layer "F.Cu")
+		(net 117)
+	)
+	(segment
+		(start 92.389808 122.80012)
+		(end 91.610192 122.80012)
+		(width 0.1554)
+		(layer "F.Cu")
+		(net 117)
+	)
+	(segment
+		(start 92.401588 122.8119)
+		(end 92.389808 122.80012)
+		(width 0.1554)
+		(layer "F.Cu")
+		(net 117)
+	)
+	(segment
