File: 1_MAIN.kicad_sch (KiCad schematic)
At the start: 44 parts, among them P1 A_A4, U2 FT2232HL, U3 TPS54202DDCR, U4 LM1084S-3.3/TR, X2 12MHz

Commit message: initial full placement and routing
Parts:
- C32, C33, C34, C35, C36, C37, C38, C39, C40, C42, C44: footprint Capacitor_SMD:C_0603_1608Metric -> Capacitor_SMD:C_0402_1005Metric
Connections:
- net VIO is gone; now on net 3V3: C34.2, C35.2, C36.2, C37.2, U2.20 (VCCIO), U2.31 (VCCIO), U2.42 (VCCIO), U2.56 (VCCIO)
- net 5V: now also AP_HARNESS1.12; no longer AP_HARNESS1.1
- net CAMO_DN: now also AP_HARNESS1.11; no longer AP_HARNESS1.2
- net CAMO_DP: now also AP_HARNESS1.10; no longer AP_HARNESS1.3
- net GND: now also AP_HARNESS1.1, AP_HARNESS1.3, AP_HARNESS1.9; no longer AP_HARNESS1.10, AP_HARNESS1.12, AP_HARNESS1.4
- net MBDN: now also AP_HARNESS1.8; no longer AP_HARNESS1.5
- net MBDP: now also AP_HARNESS1.7; no longer AP_HARNESS1.6
- net UART3V3: now also AP_HARNESS1.6; no longer AP_HARNESS1.7
- net UARTRX: now also AP_HARNESS1.5; no longer AP_HARNESS1.8
- net UARTTX: now also AP_HARNESS1.4; no longer AP_HARNESS1.9
- net at F1.2: now also AP_HARNESS1.2; no longer AP_HARNESS1.11

Commit message: clean up DRC and silkscreen
Parts:
- added R2: 0, Resistor_SMD:R_0603_1608Metric, symbol Device:R_Small
Connections:
- net 5V: now also R2.2; no longer C4.2, C5.2, L1.2, R3.2
- new net 5V_INT: C4.2, C5.2, L1.2, R2.1, R3.2
Changed lines of the file:
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@@
 	)
 	(junction
-		(at 175.26 16.51)
-		(diameter 0)
-		(color 0 0 0 0)
-	)
-	(junction
 		(at 203.2 147.32)
 		(diameter 0)
@@
 	)
 	(junction
+		(at 175.26 16.51)
+		(diameter 0)
+		(color 0 0 0 0)
+	)
+	(junction
 		(at 90.17 26.67)
 		(diameter 0)
@@
 	(wire
 		(pts
-			(xy 177.8 16.51) (xy 175.26 16.51)
-		)
-		(stroke
-			(width 0)
-			(type default)
-		)
-	)
-	(wire
-		(pts
 			(xy 52.07 15.24) (xy 55.88 15.24)
 		)
@@
 	(wire
 		(pts
+			(xy 182.88 16.51) (xy 189.23 16.51)
+		)
+		(stroke
+			(width 0)
+			(type default)
+		)
+	)
+	(wire
+		(pts
+			(xy 175.26 16.51) (xy 177.8 16.51)
+		)
+		(stroke
+			(width 0)
+			(type default)
+		)
+	)
+	(wire
+		(pts
 			(xy 227.33 135.89) (xy 203.2 135.89)
 		)
@@
 		)
 	)
+	(label "5V_INT"
+		(at 160.02 16.51 0)
+		(fields_autoplaced yes)
+		(effects
+			(font
+				(size 1.27 1.27)
+			)
+			(justify left bottom)
+		)
+	)
 	(global_label "ADBUS7"
 		(shape bidirectional)
@@
 	(global_label "5V"
 		(shape bidirectional)
-		(at 177.8 16.51 0)
+		(at 189.23 16.51 0)
 		(effects
 			(font
@@
 		)
 		(property "Intersheetrefs" "${INTERSHEET_REFS}"
-			(at 177.8 16.51 0)
+			(at 189.23 16.51 0)
 			(effects
 				(font
@@
 					(unit 1)
 				)
+			)
+		)
+	)
+	(symbol
+		(lib_id "Device:R_Small")
+		(at 180.34 16.51 90)
+		(unit 1)
+		(exclude_from_sim no)
+		(in_bom yes)
+		(on_board yes)
+		(dnp no)
+		(fields_autoplaced yes)
+		(property "Reference" "R2"
+			(at 180.34 11.6289 90)
+			(effects
+				(font
+					(size 1.27 1.27)
+				)
+			)
+		)
+		(property "Value" "0"
+			(at 180.34 14.0532 90)
+			(effects
+				(font
+					(size 1.27 1.27)
+				)
+			)
+		)
+		(property "Footprint" "Resistor_SMD:R_0603_1608Metric"
+			(at 180.34 16.51 0)
+			(effects
+				(font
+					(size 1.27 1.27)
+				)
+				(hide yes)
+			)
+		)
+		(property "Datasheet" "~"
+			(at 180.34 16.51 0)
+			(effects
+				(font
+					(size 1.27 1.27)
+				)
+				(hide yes)
+			)
+		)
+		(property "Description" "Resistor, small symbol"
+			(at 180.34 16.51 0)
+			(effects
+				(font
+					(size 1.27 1.27)
+				)
+				(hide yes)
+			)
+		)
+		(pin "2"
+		)
+		(pin "1"
+		)
+		(instances
+			(project "ProProject_X1 Expander_2024-05-26_15-16-51_2024-05-26"
+				(path "/5c4052f8-31d6-4de3-b862-4d09b0660e26/1898a0d3-3c33-4600-8778-eef1e2c48cfc"
+					(reference "R2")
+					(unit 1)
+				)

Commit message: add LCSC part tags, silkscreen
Parts:
- AP_HARNESS1: LCSC (none) -> C2937184
- C1: LCSC (none) -> C361063
- C2, C3: LCSC (none) -> C14663
- C20, C30: LCSC (none) -> C1663
- C31, C41, C43: LCSC (none) -> C1705
- C32, C33, C34, C35, C36, C37, C38, C39, C40, C42, C44: LCSC (none) -> C1525
- C4, C5: LCSC (none) -> C59461
- C47: LCSC (none) -> C23742
- C6: LCSC (none) -> C1681
- C7, C8: LCSC (none) -> C15850
- F1: LCSC (none) -> C2830246
- FB3, FB4: LCSC (none) -> C1017
- L1: LCSC (none) -> C5189959
- R1: LCSC (none) -> C25804
- R14: LCSC (none) -> C22790
- R15: LCSC (none) -> C21190
- R16, R17: LCSC (none) -> C22859
- R2: LCSC (none) -> C21189
- R3: LCSC (none) -> C23185
- R4: LCSC (none) -> C25803
- R5: LCSC (none) -> C25952
- U2: LCSC (none) -> C27882
- U3: LCSC (none) -> C191884
- U4: LCSC (none) -> C259972
- UART1: LCSC (none) -> C19190478; LCSC Part (none) -> C19190478
- X2: LCSC (none) -> C9002

Commit message: LCSC part updates
Parts:
- UART1: LCSC C19190478 -> C2935929; LCSC Part C19190478 -> C2935929; Supplier Part C19190478 -> C2935929
Changed lines of the file:
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@@
 		(at 279.4 173.99 0)
 		(unit 1)
-		(exclude_from_sim no)
+		(exclude_from_sim yes)
 		(in_bom no)
 		(on_board yes)
@@
 		)
 		(property "Description" "Open Hardware logo, small"
-			(at 279.4 173.99 0)
-			(effects
-				(font
-					(size 1.27 1.27)
-				)
-				(hide yes)
-			)
-		)
-		(property "Sim.Enable" "0"
 			(at 279.4 173.99 0)
 			(effects
@@
 			)
 		)
-		(property "Supplier Part" "C19190478"
+		(property "Supplier Part" "C2935929"
 			(at 270.51 63.5 0)
 			(effects
@@
 			)
 		)
-		(property "LCSC Part" "C19190478"
+		(property "LCSC Part" "C2935929"
 			(at 270.51 63.5 0)
 			(effects
@@
 			)
 		)
-		(property "LCSC" "C19190478"
+		(property "LCSC" "C2935929"
 			(at 270.51 63.5 0)
 			(effects

Commit message: rename to x1-expander
Parts:
- AP_HARNESS1: footprint X1 Expande-easyedapro:CONN-SMD_12P-P1.25_HCTL_HC-1.25-12PWT -> x1-expander:CONN-SMD_12P-P1.25_HCTL_HC-1.25-12PWT; symbol X1 Expande-easyedapro:HC-1.25-12PWT -> x1-expander:HC-1.25-12PWT
- C1, C2, C3, C32, C33, C34, C35, C36, C37, C38, C39, C40, C42, C44, C47: symbol X1 Expande-easyedapro:100nF -> x1-expander:100nF
- C20, C30: symbol X1 Expande-easyedapro:30pF -> x1-expander:30pF
- C31, C41, C43: symbol X1 Expande-easyedapro:4.7uF -> x1-expander:4.7uF
- C4, C5: symbol X1 Expande-easyedapro:22uF -> x1-expander:22uF
- C6: symbol X1 Expande-easyedapro:75pF -> x1-expander:75pF
- C7, C8: symbol X1 Expande-easyedapro:10uF -> x1-expander:10uF
- F1: symbol X1 Expande-easyedapro:JK-NSMD100-16V -> x1-expander:JK-NSMD100-16V
- FB3, FB4: symbol X1 Expande-easyedapro:600Ω -> x1-expander:600Ω
- L1: footprint X1 Expande-easyedapro:IND-SMD_L7.2-W6.6_GPSR07X0 -> x1-expander:IND-SMD_L7.2-W6.6_GPSR07X0; symbol X1 Expande-easyedapro:15uH -> x1-expander:15uH
- P1: footprint X1 Expande-easyedapro: -> x1-expander:; symbol X1 Expande-easyedapro:A_A4 -> x1-expander:A_A4
- R1: symbol X1 Expande-easyedapro:511k -> x1-expander:511k
- R14: symbol X1 Expande-easyedapro:12k/1% -> x1-expander:12k/1%
- R15: symbol X1 Expande-easyedapro:1k -> x1-expander:1k
- R16, R17: symbol X1 Expande-easyedapro:10 -> x1-expander:10
- R3: symbol X1 Expande-easyedapro:49.9 -> x1-expander:49.9
- R4: symbol X1 Expande-easyedapro:100k -> x1-expander:100k
- R5: symbol X1 Expande-easyedapro:13.3k -> x1-expander:13.3k
- U2: footprint X1 Expande-easyedapro:LQFP-64_L10.0-W10.0-P0.50-LS12.0-TL -> x1-expander:LQFP-64_L10.0-W10.0-P0.50-LS12.0-TL; symbol X1 Expande-easyedapro:FT2232HL -> x1-expander:FT2232HL
- U3: footprint X1 Expande-easyedapro:SOT-23-6_L2.9-W1.6-P0.95-LS2.8-BL-2 -> x1-expander:SOT-23-6_L2.9-W1.6-P0.95-LS2.8-BL-2; symbol X1 Expande-easyedapro:TPS54202DDCR -> x1-expander:TPS54202DDCR
- U4: footprint X1 Expande-easyedapro:TO-263-3_L8.6-W10.2-P2.54-LS14.4-TL -> x1-expander:TO-263-3_L8.6-W10.2-P2.54-LS14.4-TL; symbol X1 Expande-easyedapro:LM1084S-3.3/TR -> x1-expander:LM1084S-3.3/TR
- UART1: footprint X1 Expande-easyedapro:HDR-TH_4P-P2.54-H-M-W10.3 -> x1-expander:HDR-TH_4P-P2.54-H-M-W10.3; symbol X1 Expande-easyedapro:P125-1104A0BR138A1 -> x1-expander:P125-1104A0BR138A1
- X2: footprint X1 Expande-easyedapro:OSC-SMD_4P-L3.2-W2.5-BL -> x1-expander:OSC-SMD_4P-L3.2-W2.5-BL; symbol X1 Expande-easyedapro:12MHz -> x1-expander:12MHz

Commit message: add esd protection to uart
Parts:
- added D10: SRV05-4.TCT_C2687126, x1-expander:SOT-23-6_L2.9-W1.6-P0.95-LS2.8-BL, symbol x1-expander:SRV05-4.TCT_C2687126
Connections:
- net 3V3: now also UART1.1, D10.5
- net GND: now also D10.2
- net UARTRX: now also D10.1, D10.6
- net UARTTX: now also D10.3, D10.4
- net UART3V3: no longer names the net of AP_HARNESS1.6
- net UART3V3: no longer UART1.1
- no-connect marks 7 -> 8
Other:
- note added: "UART ESD"
- moved on the sheet: C34, C35, C36, C37, C38, C39, C40

Commit message: 35v caps
Parts:
- added C48, C49, C50, C51: 22µF, Capacitor_SMD:C_0805_2012Metric, symbol x1-expander:100nF
- C47: value 100µF -> 22µF; footprint Capacitor_SMD:C_1210_3225Metric -> Capacitor_SMD:C_0805_2012Metric; LCSC C23742 -> C6119901
Connections:
- net 24V: now also C48.2, C49.2, C50.2, C51.2
- net GND: now also C48.1, C49.1, C50.1, C51.1
Other:
- moved on the sheet: C47
