File: 1_MAIN.kicad_sch (KiCad schematic)
At the start: 46 parts, among them P1 A_A4, U2 FT2232HL, U3 TPS54202DDCR, U4 LM1084S-3.3/TR, X2 12MHz

Commit message: add power led
Parts:
- added LED1: KT-0603R, x1-expander:LED0603-RD, symbol x1-expander:KT-0603R
- added R35: 330, Resistor_SMD:R_0603_1608Metric, symbol x1-expander:10kΩ
Connections:
- net 5V: now also LED1.2 (A)
- net GND: now also R35.1
- new net: LED1.1 (K), R35.2
