File: 1_MAIN.kicad_sch (KiCad schematic)
At the start: 46 parts, among them P1 A_A4, U2 FT2232HL, U3 TPS54202DDCR, U4 LM1084S-3.3/TR, X2 12MHz

Commit message: Bani6809/power led (#20)
* add power led

* fix crlf
Parts:
- added LED1: KT-0603R, x1-expander:LED0603-RD, symbol x1-expander:KT-0603R
- added R35: 330, Resistor_SMD:R_0603_1608Metric, symbol x1-expander:10kΩ
Connections:
- net 5V: now also LED1.2 (A)
- net GND: now also R35.1
- new net: LED1.1 (K), R35.2

Commit message: add power leds, ground lan1 EH (#22)
Parts:
- added LED2, LED3: KT-0603R, x1-expander:LED0603-RD, symbol x1-expander:KT-0603R
- added R22: 680, Resistor_SMD:R_0603_1608Metric, symbol x1-expander:10kΩ
- added R23: 4.7k, Resistor_SMD:R_1206_3216Metric, symbol x1-expander:10kΩ
- R35: value 330 -> 1k; LCSC C23138 -> C21190; Manufacturer Part 0402WGF1002TCE -> 0603WAF1001T5E; Origin Footprint R0402 -> R0603; Supplier Part C25744 -> C21190
Connections:
- net 24V: now also LED3.2 (A)
- net 3V3: now also LED2.2 (A)
- net GND: now also R22.1, R23.1
- new net: LED3.1 (K), R23.2
- new net: LED2.1 (K), R22.2
Other:
- moved on the sheet: C41, C42, C43, C44, FB3, FB4, LED1, R35
