File: 2_LAN.kicad_sch (KiCad schematic)
At the start: 56 parts, among them U1 LAN9514, U5 M93C86-WMN6TP, X1 25MHz

Commit message: WIP: move passives around for U1
Connections:
- net CAMOR_DN: now also U1.8 (USBDM5); no longer U1.6 (USBDM4)
- net CAMOR_DP: now also U1.9 (USBDP5); no longer U1.7 (USBDP4)
- net FTDI_DN: now also U1.6 (USBDM4); no longer U1.8 (USBDM5)
- net FTDI_DP: now also U1.7 (USBDP4); no longer U1.9 (USBDP5)
Other:
- moved on the sheet: R26, R27
Changed lines of the file:
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@@
 	(wire
 		(pts
-			(xy 147.32 93.98) (xy 162.56 93.98)
+			(xy 184.15 27.94) (xy 191.77 27.94)
 		)
 		(stroke
@@
 	(wire
 		(pts
-			(xy 184.15 27.94) (xy 191.77 27.94)
+			(xy 157.48 58.42) (xy 162.56 58.42)
 		)
 		(stroke
@@
 	(wire
 		(pts
-			(xy 157.48 58.42) (xy 162.56 58.42)
+			(xy 66.04 11.43) (xy 66.04 17.78)
 		)
 		(stroke
@@
 	(wire
 		(pts
-			(xy 66.04 11.43) (xy 66.04 17.78)
+			(xy 147.32 83.82) (xy 162.56 83.82)
 		)
 		(stroke
@@
 	(wire
 		(pts
-			(xy 147.32 83.82) (xy 152.4 83.82)
-		)
-		(stroke
-			(width 0)
-			(type default)
-		)
-	)
-	(wire
-		(pts
 			(xy 179.07 176.53) (xy 179.07 180.34)
 		)
@@
 	(wire
 		(pts
+			(xy 147.32 91.44) (xy 154.94 91.44)
+		)
+		(stroke
+			(width 0)
+			(type default)
+		)
+	)
+	(wire
+		(pts
 			(xy 147.32 20.32) (xy 147.32 22.86)
 		)
@@
 	(wire
 		(pts
-			(xy 153.67 27.94) (xy 161.29 27.94)
+			(xy 147.32 93.98) (xy 154.94 93.98)
 		)
 		(stroke
@@
 	(wire
 		(pts
-			(xy 191.77 26.67) (xy 191.77 27.94)
+			(xy 153.67 27.94) (xy 161.29 27.94)
 		)
 		(stroke
@@
 	(wire
 		(pts
-			(xy 63.5 175.26) (xy 63.5 172.72)
+			(xy 191.77 26.67) (xy 191.77 27.94)
 		)
 		(stroke
@@
 	(wire
 		(pts
-			(xy 147.32 91.44) (xy 162.56 91.44)
+			(xy 63.5 175.26) (xy 63.5 172.72)
 		)
 		(stroke
@@
 	(wire
 		(pts
-			(xy 157.48 86.36) (xy 162.56 86.36)
+			(xy 160.02 93.98) (xy 162.56 93.98)
 		)
 		(stroke
@@
 	(wire
 		(pts
-			(xy 147.32 86.36) (xy 152.4 86.36)
-		)
-		(stroke
-			(width 0)
-			(type default)
-		)
-	)
-	(wire
-		(pts
 			(xy 30.48 96.52) (xy 38.1 96.52)
 		)
@@
 	(wire
 		(pts
-			(xy 157.48 83.82) (xy 162.56 83.82)
+			(xy 160.02 91.44) (xy 162.56 91.44)
 		)
 		(stroke
@@
 	(wire
 		(pts
+			(xy 147.32 86.36) (xy 162.56 86.36)
+		)
+		(stroke
+			(width 0)
+			(type default)
+		)
+	)
+	(wire
+		(pts
 			(xy 256.54 167.64) (xy 260.35 167.64)
 		)
@@
 	)
 	(label "CAMOR_DP"
-		(at 147.32 83.82 0)
+		(at 149.86 91.44 0)
 		(fields_autoplaced yes)
 		(effects
@@
 	)
 	(label "CAMOR_DN"
-		(at 147.32 86.36 0)
+		(at 149.86 93.98 0)
 		(fields_autoplaced yes)
 		(effects
@@
 	(global_label "CAMO_DN"
 		(shape bidirectional)
-		(at 162.56 86.36 0)
+		(at 162.56 93.98 0)
 		(effects
 			(font
@@
 		)
 		(property "Intersheetrefs" "${INTERSHEET_REFS}"
-			(at 162.56 86.36 0)
+			(at 162.56 93.98 0)
 			(effects
 				(font
@@
 	(global_label "FTDI_DP"
 		(shape bidirectional)
-		(at 162.56 91.44 0)
+		(at 162.56 83.82 0)
 		(effects
 			(font
@@
 		)
 		(property "Intersheetrefs" "${INTERSHEET_REFS}"
-			(at 162.56 91.44 0)
+			(at 162.56 83.82 0)
 			(effects
 				(font
@@
 	(global_label "CAMO_DP"
 		(shape bidirectional)
-		(at 162.56 83.82 0)
+		(at 162.56 91.44 0)
 		(effects
 			(font
@@
 		)
 		(property "Intersheetrefs" "${INTERSHEET_REFS}"
-			(at 162.56 83.82 0)
+			(at 162.56 91.44 0)
 			(effects
 				(font
@@
 	(global_label "FTDI_DN"
 		(shape bidirectional)
-		(at 162.56 93.98 0)
+		(at 162.56 86.36 0)
 		(effects
 			(font
@@
 		)
 		(property "Intersheetrefs" "${INTERSHEET_REFS}"
-			(at 162.56 93.98 0)
+			(at 162.56 86.36 0)
 			(effects
 				(font
@@
 	(symbol
 		(lib_id "Device:R_Small")
-		(at 154.94 86.36 270)
+		(at 157.48 93.98 270)
 		(unit 1)
 		(exclude_from_sim no)
@@
 		(dnp no)
 		(property "Reference" "R27"
-			(at 150.876 84.836 90)
+			(at 153.416 92.456 90)
 			(effects
 				(font
@@
 		)
 		(property "Value" "0"
-			(at 158.242 84.836 90)
+			(at 160.782 92.456 90)
 			(effects
 				(font
@@
 		)
 		(property "Footprint" "Resistor_SMD:R_0603_1608Metric"
-			(at 154.94 86.36 0)
+			(at 157.48 93.98 0)
 			(effects
 				(font
@@
 		)
 		(property "Datasheet" "~"
-			(at 154.94 86.36 0)
+			(at 157.48 93.98 0)
 			(effects
 				(font
@@
 		)
 		(property "Description" "Resistor, small symbol"
-			(at 154.94 86.36 0)
+			(at 157.48 93.98 0)
 			(effects
 				(font
@@
 		)
 		(property "LCSC" "C21189"
-			(at 150.876 84.836 0)
+			(at 153.416 92.456 0)
 			(effects
 				(font
@@
 	(symbol
 		(lib_id "Device:R_Small")
-		(at 154.94 83.82 270)
+		(at 157.48 91.44 270)
 		(unit 1)
 		(exclude_from_sim no)
@@
 		(dnp no)
 		(property "Reference" "R26"
-			(at 150.876 82.296 90)
+			(at 153.416 89.916 90)
 			(effects
 				(font
@@
 		)
 		(property "Value" "0"
-			(at 158.242 82.296 90)
+			(at 160.782 89.916 90)
 			(effects
 				(font
@@
 		)
 		(property "Footprint" "Resistor_SMD:R_0603_1608Metric"
-			(at 154.94 83.82 0)
+			(at 157.48 91.44 0)
 			(effects
 				(font
@@
 		)
 		(property "Datasheet" "~"
-			(at 154.94 83.82 0)
+			(at 157.48 91.44 0)
 			(effects
 				(font
@@
 		)
 		(property "Description" "Resistor, small symbol"
-			(at 154.94 83.82 0)
+			(at 157.48 91.44 0)
 			(effects
 				(font
@@
 		)
 		(property "LCSC" "C21189"
-			(at 150.876 82.296 0)
+			(at 153.416 89.916 0)
 			(effects
 				(font

Commit message: route passives near LAN95xx
Parts:
- C10, C9: footprint Capacitor_SMD:C_0603_1608Metric -> Capacitor_SMD:C_0402_1005Metric; LCSC C1658 -> (none)
- R10: footprint Resistor_SMD:R_0603_1608Metric -> Resistor_SMD:R_0402_1005Metric; LCSC C25804 -> (none)
- R11: footprint Resistor_SMD:R_0603_1608Metric -> Capacitor_SMD:C_0402_1005Metric; LCSC C22790 -> (none)
- R6: footprint Resistor_SMD:R_0603_1608Metric -> Resistor_SMD:R_0402_1005Metric; LCSC C22935 -> (none); Supplier Part C26083 -> (none)
- R8: footprint Resistor_SMD:R_0603_1608Metric -> Resistor_SMD:R_0402_1005Metric; LCSC C22859 -> (none)
Changed lines of the file:
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@@
 			)
 		)
-		(property "Footprint" "Resistor_SMD:R_0603_1608Metric"
+		(property "Footprint" "Capacitor_SMD:C_0402_1005Metric"
 			(at 55.88 58.42 0)
 			(effects
@@
 			)
 		)
-		(property "LCSC" "C22790"
+		(property "LCSC" ""
 			(at 53.7718 54.4322 0)
 			(effects
@@
 			)
 		)
-		(property "Footprint" "Resistor_SMD:R_0603_1608Metric"
+		(property "Footprint" "Resistor_SMD:R_0402_1005Metric"
 			(at 57.15 119.38 0)
 			(effects
@@
 			)
 		)
-		(property "LCSC" "C25804"
+		(property "LCSC" ""
 			(at 54.61 123.5456 0)
 			(effects
@@
 			)
 		)
-		(property "Footprint" "Capacitor_SMD:C_0603_1608Metric"
+		(property "Footprint" "Capacitor_SMD:C_0402_1005Metric"
 			(at 25.4 96.52 0)
 			(effects
@@
 			)
 		)
-		(property "LCSC" "C1658"
+		(property "LCSC" ""
 			(at 23.876 91.7956 0)
 			(effects
@@
 			)
 		)
-		(property "Footprint" "Capacitor_SMD:C_0603_1608Metric"
+		(property "Footprint" "Capacitor_SMD:C_0402_1005Metric"
 			(at 25.4 78.74 0)
 			(effects
@@
 			)
 		)
-		(property "LCSC" "C1658"
+		(property "LCSC" ""
 			(at 23.2156 74.0156 0)
 			(effects
@@
 			)
 		)
-		(property "Footprint" "Resistor_SMD:R_0603_1608Metric"
+		(property "Footprint" "Resistor_SMD:R_0402_1005Metric"
 			(at 45.72 87.63 0)
 			(effects
@@
 			)
 		)
-		(property "Supplier Part" "C26083"
+		(property "Supplier Part" ""
 			(at 45.72 87.63 90)
 			(effects
@@
 			)
 		)
-		(property "LCSC" "C22935"
+		(property "LCSC" ""
 			(at 47.498 88.8238 0)
 			(effects
@@
 			)
 		)
-		(property "Footprint" "Resistor_SMD:R_0603_1608Metric"
+		(property "Footprint" "Resistor_SMD:R_0402_1005Metric"
 			(at 243.84 26.67 0)
 			(effects
@@
 			)
 		)
-		(property "LCSC" "C22859"
+		(property "LCSC" ""
 			(at 245.5926 24.257 0)
 			(effects

Commit message: swap USB connectors
Parts:
- USB1: value AF 14.0 CC-T -> USB-226-BRW; footprint x1-expander:USB-A-TH_AF14.0CC-T -> x1-expander:USB-A-TH_USB-226-BRW; symbol x1-expander:AF14.0CC-T -> x1-expander:USB-226-BRW; LCSC C456020 -> C720524; LCSC Part C456020 -> C720524; Manufacturer SHOU HAN(首韩) -> (none); Manufacturer Part 10.0 4C6.3 ZB -> USB-226-BRW; Origin Footprint USB-TH_10.0-4C6.3-ZB -> (none); Supplier Part C456020 -> C720524
- USB2: value AF 14.0 CC-T -> USB-226-BRW; footprint x1-expander:USB-A-TH_AF14.0CC-T -> x1-expander:USB-A-TH_USB-226-BRW; symbol x1-expander:AF14.0CC-T -> x1-expander:USB-226-BRW; LCSC C456020 -> C720524; LCSC Part C456020 -> C720524; Manufacturer SHOU HAN(首韩) -> (none); Manufacturer Part 10.0 4C6.3 ZB -> USB-226-BRW; Origin Footprint USB-TH_10.0-4C6.3-ZB -> USB-226-BRW; Supplier Part C456020 -> C720524
Connections:
- net GND: now also USB1.6 (GND), USB1.7 (GND), USB1.8 (GND), USB2.6 (GND), USB2.7 (GND), USB2.8 (GND)

Commit message: route USB ports
Parts:
- removed R22, R23, R24, R25: 0, Resistor_SMD:R_0603_1608Metric, symbol Device:R_Small
Connections:
- net USB1R_DN is gone; now on net USB1_DN: U1.1 (USBDM2)
- net USB1R_DP is gone; now on net USB1_DP: U1.2 (USBDP2)
- net USB2R_DN is gone; now on net USB2_DN: U1.3 (USBDM3)
- net USB2R_DP is gone; now on net USB2_DP: U1.4 (USBDP3)
- net 5V: no longer D1.5
- net USB2_DN: now also D1.6; no longer D1.4
- net USB2_DP: now also D1.4; no longer D1.6
- net at C45.2, C46.2, F2.2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: now also D1.5

Commit message: add power leds, ground lan1 EH (#22)
Connections:
- net GND: now also LAN1.13 (EH)
- no-connect marks 17 -> 16
Changed lines of the file:
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@@
+	)
+	(junction
+		(at 278.13 54.61)
+		(diameter 0)
+		(color 0 0 0 0)
 	)
 	(junction
@@
 	)
 	(no_connect
-		(at 276.86 49.53)
-	)
-	(no_connect
 		(at 66.04 68.58)
 	)
@@
 	(wire
 		(pts
+			(xy 276.86 49.53) (xy 278.13 49.53)
+		)
+		(stroke
+			(width 0)
+			(type default)
+		)
+	)
+	(wire
+		(pts
 			(xy 26.67 39.37) (xy 34.29 39.37)
 		)
@@
 		)
 		(stroke
+			(width 0)
+			(type default)
+		)
+	)
+	(wire
+		(pts
+			(xy 278.13 49.53) (xy 278.13 54.61)
+		)
+		(stroke
