File: x1p-002/1_MAIN.kicad_sch (KiCad schematic)
At the start: 52 parts, among them P1 A_A4, U2 FT2232HL, U3 TPS54202DDCR, U4 LM1084S-3.3/TR, X2 12MHz

Commit message: clean up LED current, move LEDs, give designators some room to breathe
Parts:
- R22: value 680 -> 330; LCSC C23228 -> (none); Manufacturer UNI-ROYAL(厚声) -> (none); Manufacturer Part 0603WAF6800T5E -> (none); Origin Footprint R0603 -> (none); Supplier LCSC -> (none); Supplier Part C23228 -> (none)
- R23: value 4.7k -> 5.6k; footprint Resistor_SMD:R_1206_3216Metric -> Resistor_SMD:R_0603_1608Metric; LCSC C17936 -> (none); Manufacturer UNI-ROYAL(厚声) -> (none); Manufacturer Part 1206W4F4701T5E -> (none); Origin Footprint R1206 -> (none); Supplier LCSC -> (none); Supplier Part C17936 -> (none)
- R35: value 1k -> 820; JLCPCB Part Class Basic Part -> (none); LCSC C21190 -> (none); Manufacturer UNI-ROYAL(厚声) -> (none); Manufacturer Part 0603WAF1001T5E -> (none); Origin Footprint R0603 -> (none); Supplier LCSC -> (none); Supplier Part C21190 -> (none)
Changed lines of the file:
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@@
 			)
 		)
-		(property "Value" "1k"
+		(property "Value" "820"
 			(at 241.554 152.0698 90)
 			(effects
@@
 			)
 		)
-		(property "JLCPCB Part Class" "Basic Part"
+		(property "JLCPCB Part Class" ""
 			(at 240.03 148.59 90)
 			(effects
@@
 			)
 		)
-		(property "Manufacturer" "UNI-ROYAL(厚声)"
+		(property "Manufacturer" ""
 			(at 240.03 148.59 90)
 			(effects
@@
 			)
 		)
-		(property "Manufacturer Part" "0603WAF1001T5E"
+		(property "Manufacturer Part" ""
 			(at 240.03 148.59 90)
 			(effects
@@
 			)
 		)
-		(property "Origin Footprint" "R0603"
+		(property "Origin Footprint" ""
 			(at 240.03 148.59 90)
 			(effects
@@
 			)
 		)
-		(property "Supplier" "LCSC"
+		(property "Supplier" ""
 			(at 240.03 148.59 90)
 			(effects
@@
 			)
 		)
-		(property "Supplier Part" "C21190"
+		(property "Supplier Part" ""
 			(at 240.03 148.59 90)
 			(effects
@@
 			)
 		)
-		(property "LCSC" "C21190"
+		(property "LCSC" ""
 			(at 241.554 149.7838 0)
 			(effects
@@
 			)
 		)
-		(property "Value" "680"
+		(property "Value" "330"
 			(at 263.144 152.0698 90)
 			(effects
@@
 			)
 		)
-		(property "Manufacturer" "UNI-ROYAL(厚声)"
+		(property "Manufacturer" ""
 			(at 261.62 148.59 90)
 			(effects
@@
 			)
 		)
-		(property "Manufacturer Part" "0603WAF6800T5E"
+		(property "Manufacturer Part" ""
 			(at 261.62 148.59 90)
 			(effects
@@
 			)
 		)
-		(property "Origin Footprint" "R0603"
+		(property "Origin Footprint" ""
 			(at 261.62 148.59 90)
 			(effects
@@
 			)
 		)
-		(property "Supplier" "LCSC"
+		(property "Supplier" ""
 			(at 261.62 148.59 90)
 			(effects
@@
 			)
 		)
-		(property "Supplier Part" "C23228"
+		(property "Supplier Part" ""
 			(at 261.62 148.59 90)
 			(effects
@@
 			)
 		)
-		(property "LCSC" "C23228"
+		(property "LCSC" ""
 			(at 263.144 149.7838 0)
 			(effects
@@
 		)
 		(instances
-			(project ""
+			(project "x1-expander"
 				(path "/5c4052f8-31d6-4de3-b862-4d09b0660e26/1898a0d3-3c33-4600-8778-eef1e2c48cfc"
 					(reference "LED1")
@@
 			)
 		)
-		(property "Value" "4.7k"
+		(property "Value" "5.6k"
 			(at 219.964 152.0698 90)
 			(effects
@@
 			)
 		)
-		(property "Footprint" "Resistor_SMD:R_1206_3216Metric"
+		(property "Footprint" "Resistor_SMD:R_0603_1608Metric"
 			(at 218.44 148.59 0)
 			(effects
@@
 			)
 		)
-		(property "Manufacturer" "UNI-ROYAL(厚声)"
+		(property "Manufacturer" ""
 			(at 218.44 148.59 90)
 			(effects
@@
 			)
 		)
-		(property "Manufacturer Part" "1206W4F4701T5E"
+		(property "Manufacturer Part" ""
 			(at 218.44 148.59 90)
 			(effects
@@
 			)
 		)
-		(property "Origin Footprint" "R1206"
+		(property "Origin Footprint" ""
 			(at 218.44 148.59 90)
 			(effects
@@
 			)
 		)
-		(property "Supplier" "LCSC"
+		(property "Supplier" ""
 			(at 218.44 148.59 90)
 			(effects
@@
 			)
 		)
-		(property "Supplier Part" "C17936"
+		(property "Supplier Part" ""
 			(at 218.44 148.59 90)
 			(effects
@@
 			)
 		)
-		(property "LCSC" "C17936"
+		(property "LCSC" ""
 			(at 219.964 149.7838 0)
 			(effects

Commit message: assign lcsc parts to R23, R35, R22. fix warning about unconnected RXN trace near RN1
Parts:
- R22: LCSC (none) -> C23138; Manufacturer (none) -> UNI-ROYAL(厚声); Manufacturer Part (none) -> 0603WAF3300T5E; Origin Footprint (none) -> R0603; Supplier (none) -> LCSC; Supplier Part (none) -> C23138
- R23: footprint Resistor_SMD:R_0603_1608Metric -> Resistor_SMD:R_1206_3216Metric; JLCPCB Part Class Basic Part -> Extended Part; LCSC (none) -> C26045; Manufacturer Part (none) -> 1206W4J0562T5E; Origin Footprint (none) -> R1206; Supplier (none) -> LCSC; Supplier Part (none) -> C26045
- R35: LCSC (none) -> C23253; Manufacturer (none) -> UNI-ROYAL(厚声); Manufacturer Part (none) -> 0603WAF8200T5E; Supplier (none) -> LCSC; Supplier Part (none) -> C23253
Changed lines of the file:
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@@
 			)
 		)
-		(property "Manufacturer" ""
+		(property "Manufacturer" "UNI-ROYAL(厚声)"
 			(at 240.03 148.59 90)
 			(effects
@@
 			)
 		)
-		(property "Manufacturer Part" ""
+		(property "Manufacturer Part" "0603WAF8200T5E"
 			(at 240.03 148.59 90)
 			(effects
@@
 			)
 		)
-		(property "Supplier" ""
+		(property "Supplier" "LCSC"
 			(at 240.03 148.59 90)
 			(effects
@@
 			)
 		)
-		(property "Supplier Part" ""
+		(property "Supplier Part" "C23253"
 			(at 240.03 148.59 90)
 			(effects
@@
 			)
 		)
-		(property "LCSC" ""
+		(property "LCSC" "C23253"
 			(at 241.554 149.7838 0)
 			(effects
@@
 			)
 		)
-		(property "Manufacturer" ""
+		(property "Manufacturer" "UNI-ROYAL(厚声)"
 			(at 261.62 148.59 90)
 			(effects
@@
 			)
 		)
-		(property "Manufacturer Part" ""
+		(property "Manufacturer Part" "0603WAF3300T5E"
 			(at 261.62 148.59 90)
 			(effects
@@
 			)
 		)
-		(property "Origin Footprint" ""
+		(property "Origin Footprint" "R0603"
 			(at 261.62 148.59 90)
 			(effects
@@
 			)
 		)
-		(property "Supplier" ""
+		(property "Supplier" "LCSC"
 			(at 261.62 148.59 90)
 			(effects
@@
 			)
 		)
-		(property "Supplier Part" ""
+		(property "Supplier Part" "C23138"
 			(at 261.62 148.59 90)
 			(effects
@@
 			)
 		)
-		(property "LCSC" ""
+		(property "LCSC" "C23138"
 			(at 263.144 149.7838 0)
 			(effects
@@
 			)
 		)
-		(property "Footprint" "Resistor_SMD:R_0603_1608Metric"
+		(property "Footprint" "Resistor_SMD:R_1206_3216Metric"
 			(at 218.44 148.59 0)
 			(effects
@@
 			)
 		)
-		(property "Description" ""
-			(at 218.44 148.59 0)
+		(property "Description" "250mw 1206"
+			(at 225.044 153.162 90)
 			(effects
 				(font
 					(size 1.27 1.27)
 				)
-				(hide yes)
 			)
 		)
@@
 			)
 		)
-		(property "JLCPCB Part Class" "Basic Part"
+		(property "JLCPCB Part Class" "Extended Part"
 			(at 218.44 148.59 90)
 			(effects
@@
 			)
 		)
-		(property "Manufacturer Part" ""
+		(property "Manufacturer Part" "1206W4J0562T5E"
 			(at 218.44 148.59 90)
 			(effects
@@
 			)
 		)
-		(property "Origin Footprint" ""
+		(property "Origin Footprint" "R1206"
 			(at 218.44 148.59 90)
 			(effects
@@
 			)
 		)
-		(property "Supplier" ""
+		(property "Supplier" "LCSC"
 			(at 218.44 148.59 90)
 			(effects
@@
 			)
 		)
-		(property "Supplier Part" ""
+		(property "Supplier Part" "C26045"
 			(at 218.44 148.59 90)
 			(effects
@@
 			)
 		)
-		(property "LCSC" ""
+		(property "LCSC" "C26045"
 			(at 219.964 149.7838 0)
 			(effects

Commit message: add test points; replace capacitor with big boi; route USB out of the way of vias for new capacitor
Parts:
- added TP1, TP2, TP3, TP8: TestPoint, TestPoint:TestPoint_Pad_D1.0mm, symbol Connector:TestPoint
- C47: value 100µF -> 35V 47uF; footprint Capacitor_SMD:C_1210_3225Metric -> Capacitor_SMD:CP_Elec_6.3x5.8; symbol x1-expander:100nF -> Device:C_Polarized_Small; LCSC C23742 -> C5246552; Origin Footprint C0603 -> (none)
Connections:
- net 24V: now also C47.1, TP1.1; no longer C47.2
- net 3V3: now also TP3.1
- net 5V: now also TP2.1
- net GND: now also C47.2, TP8.1; no longer C47.1
