File: x1p-002/1_MAIN.kicad_sch (KiCad schematic)
At the start: 56 parts, among them P1 A_A4, U2 FT2232HL, U3 TPS54202DDCR, U4 LM1084S-3.3/TR, X2 12MHz

Commit message: annotated everything with LCSC IDs
Parts:
- LED1, LED2, LED3: LCSC (none) -> C2286
- TP1, TP2, TP3, TP8: now left out of the parts list
Changed lines of the file:
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@@
 		(unit 1)
 		(exclude_from_sim no)
-		(in_bom yes)
+		(in_bom no)
 		(on_board yes)
 		(dnp no)
@@
 		(unit 1)
 		(exclude_from_sim no)
-		(in_bom yes)
+		(in_bom no)
 		(on_board yes)
 		(dnp no)
@@
 			)
 		)
+		(property "LCSC" "C2286"
+			(at 222.25 138.4299 0)
+			(effects
+				(font
+					(size 1.27 1.27)
+				)
+				(hide yes)
+			)
+		)
 		(pin "1"
 		)
@@
 		(unit 1)
 		(exclude_from_sim no)
-		(in_bom yes)
+		(in_bom no)
 		(on_board yes)
 		(dnp no)
@@
 			)
 		)
+		(property "LCSC" "C2286"
+			(at 243.84 138.4299 0)
+			(effects
+				(font
+					(size 1.27 1.27)
+				)
+				(hide yes)
+			)
+		)
 		(pin "1"
 		)
@@
 		(unit 1)
 		(exclude_from_sim no)
-		(in_bom yes)
+		(in_bom no)
 		(on_board yes)
 		(dnp no)
@@
 			(effects
 				(font
+					(size 1.27 1.27)
+				)
+				(hide yes)
+			)
+		)
+		(property "LCSC" "C2286"
+			(at 265.43 138.4299 0)
+			(effects
+				(font

Commit message: add pullup on FTDI EEDATA, swap EEPROM to 4k EEPROM
Parts:
- added R24: 10k, Resistor_SMD:R_0402_1005Metric, symbol Device:R_Small
Connections:
- net 3V3: now also R24.2
- net at U2.61 (EEDATA): now also R24.1
- no-connect marks 8 -> 7
Changed lines of the file:
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@@
 	)
 	(no_connect
-		(at 48.26 154.94)
-	)
-	(no_connect
 		(at 262.89 29.21)
 	)
@@
 	(wire
 		(pts
+			(xy 48.26 154.94) (xy 39.37 154.94)
+		)
+		(stroke
+			(width 0)
+			(type default)
+		)
+	)
+	(wire
+		(pts
 			(xy 25.4 185.42) (xy 43.18 185.42)
 		)
@@
 	(wire
 		(pts
+			(xy 39.37 142.24) (xy 39.37 146.05)
+		)
+		(stroke
+			(width 0)
+			(type default)
+		)
+	)
+	(wire
+		(pts
 			(xy 175.26 16.51) (xy 177.8 16.51)
 		)
@@
 	(wire
 		(pts
+			(xy 39.37 154.94) (xy 39.37 151.13)
+		)
+		(stroke
+			(width 0)
+			(type default)
+		)
+	)
+	(wire
+		(pts
 			(xy 110.49 142.24) (xy 109.22 142.24)
 		)
@@
 		)
 	)
+	(global_label "3V3"
+		(shape bidirectional)
+		(at 39.37 142.24 90)
+		(effects
+			(font
+				(size 1.27 1.27)
+			)
+			(justify left)
+		)
+		(property "Intersheetrefs" "${INTERSHEET_REFS}"
+			(at 39.37 142.24 0)
+			(effects
+				(font
+					(size 1.27 1.27)
+				)
+				(hide yes)
+			)
+		)
+	)
 	(global_label "ACBUS7"
 		(shape bidirectional)
@@
 					(unit 1)
 				)
+			)
+		)
+	)
+	(symbol
+		(lib_id "Device:R_Small")
+		(at 39.37 148.59 180)
+		(unit 1)
+		(exclude_from_sim no)
+		(in_bom yes)
+		(on_board yes)
+		(dnp no)
+		(fields_autoplaced yes)
+		(property "Reference" "R24"
+			(at 40.8686 147.3778 0)
+			(effects
+				(font
+					(size 1.27 1.27)
+				)
+				(justify right)
+			)
+		)
+		(property "Value" "10k"
+			(at 40.8686 149.8021 0)
+			(effects
+				(font
+					(size 1.27 1.27)
+				)
+				(justify right)
+			)
+		)
+		(property "Footprint" "Resistor_SMD:R_0402_1005Metric"
+			(at 39.37 148.59 0)
+			(effects
+				(font
+					(size 1.27 1.27)
+				)
+				(hide yes)
+			)
+		)
+		(property "Datasheet" "~"
+			(at 39.37 148.59 0)
+			(effects
+				(font
+					(size 1.27 1.27)
+				)
+				(hide yes)
+			)
+		)
+		(property "Description" "Resistor, small symbol"
+			(at 39.37 148.59 0)
+			(effects
+				(font
+					(size 1.27 1.27)
+				)
+				(hide yes)
+			)
+		)
+		(property "LCSC" "C25744"
+			(at 34.4889 148.59 0)
+			(effects
+				(font
+					(size 1.27 1.27)
+				)
+				(hide yes)
+			)
+		)
+		(pin "1"
+		)
+		(pin "2"
+		)
+		(instances
+			(project "x1-expander"
+				(path "/5c4052f8-31d6-4de3-b862-4d09b0660e26/1898a0d3-3c33-4600-8778-eef1e2c48cfc"
+					(reference "R24")
+					(unit 1)
+				)

Commit message: replace F1 with proper rated part, relink RN1 with 3d model, adjust lan1 3d model z offset, move TXN & RXN meander near rj45
Parts:
- removed F1: JK-NSMD100-16V, Fuse:Fuse_1206_3216Metric, symbol x1-expander:JK-NSMD100-16V
- added F1: BSMD1206-050-30V, x1-expander:F1206, symbol x1-expander:BSMD1206-050-30V
Connections:
- net 24V: now also F1.1
- net at AP_HARNESS1.2: now also F1.2
Other:
- moved on the sheet: C47, TP1, TP8

Commit message: replace F1 with C5358568 - BHFUSE BSMD1206-100-30V
Parts:
- removed F1: BSMD1206-050-30V, x1-expander:F1206, symbol x1-expander:BSMD1206-050-30V
- added F1: BSMD1206-100-30V, x1-expander:F1206, symbol x1-expander:BSMD1206-100-30V
Connections:
- net 24V: now also F1.1
- net at AP_HARNESS1.2: now also F1.2
Changed lines of the file:
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@@
 	(wire
 		(pts
+			(xy 247.65 39.37) (xy 265.43 39.37)
+		)
+		(stroke
+			(width 0)
+			(type default)
+		)
+	)
+	(wire
+		(pts
 			(xy 44.45 90.17) (xy 44.45 83.82)
 		)
@@
 	(wire
 		(pts
-			(xy 265.43 39.37) (xy 250.19 39.37)
-		)
-		(stroke
-			(width 0)
-			(type default)
-		)
-	)
-	(wire
-		(pts
 			(xy 52.07 19.05) (xy 52.07 15.24)
 		)
@@
 	(wire
 		(pts
-			(xy 228.6 39.37) (xy 234.95 39.37)
+			(xy 228.6 39.37) (xy 237.49 39.37)
 		)
 		(stroke
@@
 	)
 	(symbol
-		(lib_id "x1-expander:BSMD1206-050-30V")
-		(at 242.57 39.37 0)
-		(unit 1)
-		(exclude_from_sim no)
-		(in_bom yes)
-		(on_board yes)
-		(dnp no)
-		(property "Reference" "F1"
-			(at 242.57 37.084 0)
-			(effects
-				(font
-					(size 1.27 1.27)
-				)
-			)
-		)
-		(property "Value" "BSMD1206-050-30V"
-			(at 242.57 35.56 0)
-			(effects
-				(font
-					(size 1.27 1.27)
-				)
-				(hide yes)
-			)
-		)
-		(property "Footprint" "x1-expander:F1206"
-			(at 242.57 46.99 0)
-			(effects
-				(font
-					(size 1.27 1.27)
-				)
-				(hide yes)
-			)
-		)
-		(property "Datasheet" "https://lcsc.com/product-detail/PTC-Resettable-Fuses_BHFUSE-BSMD1206-050-30V_C883126.html"
-			(at 242.57 49.53 0)
-			(effects
-				(font
-					(size 1.27 1.27)
-				)
-				(hide yes)
-			)
-		)
-		(property "Description" "30V 500ma 1A"
-			(at 242.824 36.576 0)
-			(effects
-				(font
-					(size 1.27 1.27)
-				)
-				(hide yes)
-			)
-		)
-		(property "LCSC Part" "C883126"
-			(at 242.57 52.07 0)
-			(effects
-				(font
-					(size 1.27 1.27)
-				)
-				(hide yes)
-			)
-		)
-		(pin "1"
-		)
-		(pin "2"
-		)
-		(instances
-			(project ""
-				(path "/5c4052f8-31d6-4de3-b862-4d09b0660e26/1898a0d3-3c33-4600-8778-eef1e2c48cfc"
-					(reference "F1")
-					(unit 1)
-				)
-			)
-		)
-	)
-	(symbol
 		(lib_id "x1-expander:30pF")
 		(at 43.18 179.07 90)
@@
 					(unit 1)
 				)
+			)
+		)
+	)
+	(symbol
+		(lib_id "x1-expander:BSMD1206-100-30V")
+		(at 242.57 39.37 0)
+		(unit 1)
+		(exclude_from_sim no)
+		(in_bom yes)
+		(on_board yes)
+		(dnp no)
+		(property "Reference" "F1"
+			(at 242.57 37.084 0)
+			(effects
+				(font
+					(size 1.27 1.27)
+				)
+			)
+		)
+		(property "Value" "BSMD1206-100-30V"
+			(at 242.57 35.56 0)
+			(effects
+				(font
+					(size 1.27 1.27)
+				)
+				(hide yes)
+			)
+		)
+		(property "Footprint" "x1-expander:F1206"
+			(at 242.57 46.99 0)
+			(effects
+				(font
+					(size 1.27 1.27)
+				)
+				(hide yes)
+			)
+		)
+		(property "Datasheet" ""
+			(at 242.57 39.37 0)
+			(effects
+				(font
+					(size 1.27 1.27)
+				)
+				(hide yes)
+			)
+		)
+		(property "Description" ""
+			(at 242.57 39.37 0)
+			(effects
+				(font
+					(size 1.27 1.27)
+				)
+				(hide yes)
+			)
+		)
+		(property "LCSC Part" "C5358568"
+			(at 242.57 49.53 0)
+			(effects
+				(font
+					(size 1.27 1.27)
+				)
+				(hide yes)
+			)
+		)
+		(pin "2"
+		)
+		(pin "1"
+		)
+		(instances
+			(project ""
+				(path "/5c4052f8-31d6-4de3-b862-4d09b0660e26/1898a0d3-3c33-4600-8778-eef1e2c48cfc"
+					(reference "F1")
+					(unit 1)
+				)

Commit message: X1P-002: schematic: redesign with larger 5V buck (#60), add 3V3 buck (#63), add OCP circuits for 3V3 and 5V (but not connected to user ports yet; #61)
Parts:
- removed C1: 10µF, Capacitor_SMD:C_0805_2012Metric, symbol x1-expander:100nF
- removed C2: 100nF, Capacitor_SMD:C_0603_1608Metric, symbol x1-expander:100nF
- removed C3: 100nF X7R, Capacitor_SMD:C_0603_1608Metric, symbol x1-expander:100nF
- removed C4, C5: 22uF, Capacitor_SMD:C_0603_1608Metric, symbol x1-expander:22uF
- removed C47: 35V 47uF, Capacitor_SMD:CP_Elec_6.3x5.8, symbol Device:C_Polarized_Small
- removed C6: 75pF, Capacitor_SMD:C_0603_1608Metric, symbol x1-expander:75pF
- removed C7, C8: 10uF, Capacitor_SMD:C_0805_2012Metric, symbol x1-expander:10uF
- removed F1: BSMD1206-100-30V, x1-expander:F1206, symbol x1-expander:BSMD1206-100-30V
- removed L1: 15uH, x1-expander:IND-SMD_L7.2-W6.6_GPSR07X0, symbol x1-expander:15uH
- removed LED1, LED2, LED3: KT-0603R, x1-expander:LED0603-RD, symbol x1-expander:KT-0603R
- removed P1: A_A4, x1-expander:, symbol x1-expander:A_A4
- removed R1: 10k, Resistor_SMD:R_0603_1608Metric, symbol x1-expander:511k
- removed R2: 0, Resistor_SMD:R_0603_1608Metric, symbol Device:R_Small
- removed R22: 330, Resistor_SMD:R_0603_1608Metric, symbol x1-expander:10kΩ
- removed R23: 5.6k, Resistor_SMD:R_1206_3216Metric, symbol x1-expander:10kΩ
- removed R3: 49.9, Resistor_SMD:R_0603_1608Metric, symbol x1-expander:49.9
- removed R35: 820, Resistor_SMD:R_0603_1608Metric, symbol x1-expander:10kΩ
- removed R4: 100k, Resistor_SMD:R_0603_1608Metric, symbol x1-expander:100k
- removed R5: 13.3k, Resistor_SMD:R_0603_1608Metric, symbol x1-expander:13.3k
- removed TP1, TP2, TP3, TP8: TestPoint, TestPoint:TestPoint_Pad_D1.0mm, symbol Connector:TestPoint
- removed U3: TPS54202DDCR, x1-expander:SOT-23-6_L2.9-W1.6-P0.95-LS2.8-BL-2, symbol x1-expander:TPS54202DDCR
- removed U4: LM1084S-3.3/TR, x1-expander:TO-263-3_L8.6-W10.2-P2.54-LS14.4-TL, symbol x1-expander:LM1084S-3.3/TR
Connections:
- net 24V_SYS: now reaches AP_HARNESS1.2
- no-connect marks 7 -> 9
Other:
- note removed: "24V to 5V Buck 2A"
- note removed: "5V to 3V3 LDO 5A"
- title: (none) -> X1Plus Expansion Board: X1P-002
- moved on the sheet: AP_HARNESS1, UART1

Commit message: X1P-002: schematic: add FTDI EEPROM (#62)
Parts:
- removed R24: 10k, Resistor_SMD:R_0402_1005Metric, symbol Device:R_Small
- added C64: 100nF, Capacitor_SMD:C_0402_1005Metric, symbol Device:C_Small
- added R40, R41, R42: 10k, Resistor_SMD:R_0402_1005Metric, symbol Device:R_Small
- added R44: 1k, Resistor_SMD:R_0603_1608Metric, symbol Device:R_Small
- added U8: AT93C66B-SSHM-T, Package_SO:SOIC-8_3.9x4.9mm_P1.27mm, symbol Memory_EEPROM:93CxxA
Connections:
- net 3V3: now also C64.2, R40.2, R41.2, R42.2, U8.6 (ORG), U8.8 (VCC)
- net GND: now also C64.1, U8.5 (GND)
- net FT_EEDATA: now reaches U2.61 (EEDATA)
- net FT_EEDATA: now also R42.1, R44.2, U8.3 (DI)
- net FT_EECLK: now reaches U2.62 (EECLK)
- net FT_EECLK: now also R41.1, U8.2 (SCLK)
- net FT_EECS: now reaches U2.63 (EECS)
- net FT_EECS: now also R40.1, U8.1 (CS)
- new net: R44.1, U8.4 (DO)
- no-connect marks 9 -> 7
