File: x1p-002/1_MAIN.kicad_sch (KiCad schematic)
At the start: 33 parts, among them U2 FT2232HL, U8 AT93C66B-SSHM-T, X2 12MHz

Commit message: X1P-002: schematic: change to FT4232 (#64)
Parts:
- U2: value FT2232HL -> FT4232HL; LCSC C27882 -> C56742; Manufacturer Part FT2232HL-REEL -> FT4232HL-REEL; Supplier Part C27882 -> C56742
Changed lines of the file:
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@@
 			)
 		)
-		(property "Value" "FT2232HL"
+		(property "Value" "FT4232HL"
 			(at 73.1266 129.4384 0)
 			(effects
@@
 			)
 		)
-		(property "Manufacturer Part" "FT2232HL-REEL"
+		(property "Manufacturer Part" "FT4232HL-REEL"
 			(at 78.74 130.81 0)
 			(effects
@@
 			)
 		)
-		(property "Supplier Part" "C27882"
+		(property "Supplier Part" "C56742"
 			(at 78.74 130.81 0)
 			(effects
@@
 			)
 		)
-		(property "LCSC" "C27882"
+		(property "LCSC" "C56742"
 			(at 73.1266 127.2286 0)
 			(effects

Commit message: x1p-002: wire up OCP circuits to user ports (#61)
Connections:
- net 3V3: no longer D10.5, UART1.1
- new net 3V3_USER: D10.5, UART1.1
Changed lines of the file:
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@@
 		)
 	)
-	(global_label "3V3"
+	(global_label "3V3_USER"
 		(shape bidirectional)
 		(at 247.65 95.25 0)
@@
 		)
 	)
-	(global_label "3V3"
+	(global_label "3V3_USER"
 		(shape bidirectional)
 		(at 229.87 45.72 180)
