File: x1p-002/2_LAN.kicad_sch (KiCad schematic)
At the start: 54 parts, among them U1 LAN9514, U5 AT93C66B-SSHM-T, X1 25MHz

Commit message: correct C3021374 footprint, route rj45
Parts:
- renumbered C49 to C19, RN2 to RN1
Connections:
- net 3V3: now also LAN1.11 (LED(G)_A); no longer LAN1.12 (LED(G)_K)
- net LNKA: now also LAN1.12 (LED(G)_K); no longer LAN1.11 (LED(G)_A)
- net RXN: now also RN1.3
- net RXP: no longer RN1.3
- net TXN: now also RN1.1; no longer RN1.2
- net TXP: now also RN1.2; no longer RN1.1

Commit message: move fuse downstream of bulk USB caps; ethernet jack mechanical pins are NPTH
Connections:
- net 5V: now also C45.2, C46.2
- net at D1.5, F2.2, USB1.1 (VBUS)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: no longer C45.2, C46.2
Other:
- moved on the sheet: C45, C46, F2
