File: x1p-002/2_LAN.kicad_sch (KiCad schematic)
At the start: 54 parts, among them U1 LAN9514, U5 AT93C66B-SSHM-T, X1 25MHz

Commit message: X1P-002: schematic: redesign with larger 5V buck (#60), add 3V3 buck (#63), add OCP circuits for 3V3 and 5V (but not connected to user ports yet; #61)
Other:
- title: (none) -> X1Plus Expansion Board: X1P-002
- moved on the sheet: C10, C11, C12, C13, C14, C15, C16, C17, C18, C19, C21, C22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

Commit message: x1p-002: wire up OCP circuits to user ports (#61)
Parts:
- removed F2: JK-NSMD100-16V, Fuse:Fuse_1206_3216Metric, symbol x1-expander:JK-NSMD100-16V
Connections:
- net 5V is gone; now on net 5V_USER: C45.2, C46.2
- net 5V_USER: now reaches D1.5, USB1.1 (VBUS), USB2.1 (VBUS)
- net OCP_ACT_N: now reaches U1.14 (PRTCTL2)
- net OCP_ACT_N: now also U1.16 (PRTCTL3)
- no-connect marks 17 -> 15
Changed lines of the file:
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@@
 	)
 	(junction
+		(at 105.41 96.52)
+		(diameter 0)
+		(color 0 0 0 0)
+	)
+	(junction
 		(at 191.77 86.36)
 		(diameter 0)
@@
 	)
 	(no_connect
-		(at 107.95 96.52)
-	)
-	(no_connect
 		(at 74.93 123.19)
 	)
@@
 	)
 	(no_connect
-		(at 107.95 104.14)
-	)
-	(no_connect
 		(at 107.95 111.76)
 	)
@@
 	(wire
 		(pts
+			(xy 105.41 96.52) (xy 107.95 96.52)
+		)
+		(stroke
+			(width 0)
+			(type default)
+		)
+	)
+	(wire
+		(pts
 			(xy 287.02 72.39) (xy 287.02 90.17)
 		)
@@
 	(wire
 		(pts
+			(xy 105.41 104.14) (xy 105.41 96.52)
+		)
+		(stroke
+			(width 0)
+			(type default)
+		)
+	)
+	(wire
+		(pts
 			(xy 220.98 204.47) (xy 220.98 208.28)
 		)
@@
 	(wire
 		(pts
+			(xy 102.87 96.52) (xy 105.41 96.52)
+		)
+		(stroke
+			(width 0)
+			(type default)
+		)
+	)
+	(wire
+		(pts
 			(xy 298.45 195.58) (xy 302.26 195.58)
 		)
@@
 	(wire
 		(pts
+			(xy 107.95 104.14) (xy 105.41 104.14)
+		)
+		(stroke
+			(width 0)
+			(type default)
+		)
+	)
+	(wire
+		(pts
 			(xy 279.4 46.99) (xy 276.86 46.99)
 		)
@@
 	(wire
 		(pts
-			(xy 270.51 157.48) (xy 276.86 157.48)
-		)
-		(stroke
-			(width 0)
-			(type default)
-		)
-	)
-	(wire
-		(pts
 			(xy 234.95 215.9) (xy 234.95 218.44)
 		)
@@
 	(wire
 		(pts
-			(xy 254 157.48) (xy 260.35 157.48)
+			(xy 254 157.48) (xy 276.86 157.48)
 		)
 		(stroke
@@
 		)
 	)
+	(global_label "OCP_ACT_N"
+		(shape input)
+		(at 102.87 96.52 180)
+		(fields_autoplaced yes)
+		(effects
+			(font
+				(size 1.27 1.27)
+			)
+			(justify right)
+		)
+		(property "Intersheetrefs" "${INTERSHEET_REFS}"
+			(at 89.4224 96.52 0)
+			(effects
+				(font
+					(size 1.27 1.27)
+				)
+				(justify right)
+				(hide yes)
+			)
+		)
+	)
 	(global_label "3V3"
 		(shape bidirectional)
@@
 		)
 	)
-	(global_label "5V"
+	(global_label "5V_USER"
 		(shape bidirectional)
 		(at 240.03 157.48 180)
@@
 					(unit 1)
 				)
-			)
-		)
-	)
-	(symbol
-		(lib_id "x1-expander:JK-NSMD100-16V")
-		(at 265.43 157.48 0)
-		(unit 1)
-		(exclude_from_sim no)
-		(in_bom yes)
-		(on_board yes)
-		(dnp no)
-		(property "Reference" "F2"
-			(at 264.033 156.1338 0)
-			(effects
-				(font
-					(size 1.27 1.27)
-				)
-				(justify left bottom)
-			)
-		)
-		(property "Value" "JK-NSMD100-16V"
-			(at 264.033 156.3116 0)
-			(effects
-				(font
-					(size 1.27 1.27)
-				)
-				(justify left bottom)
-				(hide yes)
-			)
-		)
-		(property "Footprint" "Fuse:Fuse_1206_3216Metric"
-			(at 265.43 157.48 0)
-			(effects
-				(font
-					(size 1.27 1.27)
-				)
-				(hide yes)
-			)
-		)
-		(property "Datasheet" ""
-			(at 265.43 157.48 0)
-			(effects
-				(font
-					(size 1.27 1.27)
-				)
-				(hide yes)
-			)
-		)
-		(property "Description" ""
-			(at 265.43 157.48 0)
-			(effects
-				(font
-					(size 1.27 1.27)
-				)
-				(hide yes)
-			)
-		)
-		(property "Add into BOM" "yes"
-			(at 265.43 157.48 0)
-			(effects
-				(font
-					(size 1.27 1.27)
-				)
-				(justify left bottom)
-				(hide yes)
-			)
-		)
-		(property "Convert to PCB" "yes"
-			(at 265.43 157.48 0)
-			(effects
-				(font
-					(size 1.27 1.27)
-				)
-				(justify left bottom)
-				(hide yes)
-			)
-		)
-		(property "JLCPCB Part Class" "Extended Part"
-			(at 265.43 157.48 0)
-			(effects
-				(font
-					(size 1.27 1.27)
-				)
-				(justify left bottom)
-				(hide yes)
-			)
-		)
-		(property "Manufacturer" "JK(金科)"
-			(at 265.43 157.48 0)
-			(effects
-				(font
-					(size 1.27 1.27)
-				)
-				(justify left bottom)
-				(hide yes)
-			)
-		)
-		(property "Manufacturer Part" "JK-nSMD100-16"
-			(at 265.43 157.48 0)
-			(effects
-				(font
-					(size 1.27 1.27)
-				)
-				(justify left bottom)
-				(hide yes)
-			)
-		)
-		(property "Origin Footprint" "F1206"
-			(at 265.43 157.48 0)
-			(effects
-				(font
-					(size 1.27 1.27)
-				)
-				(justify left bottom)
-				(hide yes)
-			)
-		)
-		(property "Supplier" "LCSC"
-			(at 265.43 157.48 0)
-			(effects
-				(font
-					(size 1.27 1.27)
-				)
-				(justify left bottom)
-				(hide yes)
-			)
-		)
-		(property "Supplier Part" "C369161"
-			(at 265.43 157.48 0)
-			(effects
-				(font
-					(size 1.27 1.27)
-				)
-				(justify left bottom)
-				(hide yes)
-			)
-		)
-		(property "LCSC" "C2830246"
-			(at 264.033 156.1338 0)
-			(effects
-				(font
-					(size 1.27 1.27)
-				)
-				(hide yes)
-			)
-		)
-		(pin "2"
-		)
-		(pin "1"
-		)
-		(instances
-			(project "x1-expander"
-				(path "/5c4052f8-31d6-4de3-b862-4d09b0660e26/59f5b442-dc6c-49f9-8b13-7a2ac6495930"
-					(reference "F2")
-					(unit 1)
-				)

Commit message: X1P-002: finish connecting GPIO ports to RP2040
Connections:
- net RP2040_RST_N: now reaches U1.43 (GPIO7)
- no-connect marks 15 -> 14
Changed lines of the file:
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@@
+	)
+	(junction
+		(at 60.96 106.68)
+		(diameter 0)
+		(color 0 0 0 0)
 	)
 	(junction
@@
 	)
 	(junction
-		(at 62.23 124.46)
-		(diameter 0)
-		(color 0 0 0 0)
-	)
-	(junction
 		(at 107.95 45.72)
 		(diameter 0)
@@
 	(junction
 		(at 226.06 55.88)
-		(diameter 0)
-		(color 0 0 0 0)
-	)
-	(junction
-		(at 62.23 106.68)
 		(diameter 0)
 		(color 0 0 0 0)
@@
 	)
 	(no_connect
-		(at 189.23 177.8)
-	)
-	(no_connect
 		(at 107.95 167.64)
 	)
@@
 	(wire
 		(pts
-			(xy 62.23 124.46) (xy 63.5 124.46)
-		)
-		(stroke
-			(width 0)
-			(type default)
-		)
-	)
-	(wire
-		(pts
 			(xy 189.23 58.42) (xy 189.23 60.96)
 		)
@@
 	(wire
 		(pts
+			(xy 60.96 106.68) (xy 60.96 124.46)
+		)
+		(stroke
+			(width 0)
+			(type default)
+		)
+	)
+	(wire
+		(pts
 			(xy 74.93 106.68) (xy 74.93 107.95)
 		)
@@
 	(wire
 		(pts
-			(xy 62.23 106.68) (xy 62.23 124.46)
-		)
-		(stroke
-			(width 0)
-			(type default)
-		)
-	)
-	(wire
-		(pts
 			(xy 107.95 203.2) (xy 105.41 203.2)
 		)
@@
 	(wire
 		(pts
-			(xy 59.69 106.68) (xy 62.23 106.68)
-		)
-		(stroke
-			(width 0)
-			(type default)
-		)
-	)
-	(wire
-		(pts
 			(xy 270.51 80.01) (xy 276.86 80.01)
 		)
@@
 	(wire
 		(pts
-			(xy 63.5 106.68) (xy 62.23 106.68)
-		)
-		(stroke
-			(width 0)
-			(type default)
-		)
-	)
-	(wire
-		(pts
 			(xy 279.4 67.31) (xy 297.18 67.31)
 		)
@@
 	(wire
 		(pts
+			(xy 189.23 177.8) (xy 204.47 177.8)
+		)
+		(stroke
+			(width 0)
+			(type default)
+		)
+	)
+	(wire
+		(pts
 			(xy 243.84 168.91) (xy 243.84 173.99)
 		)
@@
 	(wire
 		(pts
+			(xy 62.23 124.46) (xy 60.96 124.46)
+		)
+		(stroke
+			(width 0)
+			(type default)
+		)
+	)
+	(wire
+		(pts
 			(xy 87.63 124.46) (xy 80.01 124.46)
 		)
@@
 	(wire
 		(pts
+			(xy 59.69 106.68) (xy 60.96 106.68)
+		)
+		(stroke
+			(width 0)
+			(type default)
+		)
+	)
+	(wire
+		(pts
 			(xy 68.58 59.69) (xy 76.2 59.69)
 		)
@@
 		(pts
 			(xy 189.23 104.14) (xy 204.47 104.14)
+		)
+		(stroke
+			(width 0)
+			(type default)
+		)
+	)
+	(wire
+		(pts
+			(xy 60.96 106.68) (xy 62.23 106.68)
 		)
 		(stroke
@@
 			(effects
 				(font
+					(size 1.27 1.27)
+				)
+				(hide yes)
+			)
+		)
+	)
+	(global_label "RP2040_RST_N"
+		(shape bidirectional)
+		(at 204.47 177.8 0)
+		(effects
+			(font
+				(size 1.27 1.27)
+			)
+			(justify left)
+		)
+		(property "Intersheetrefs" "${INTERSHEET_REFS}"
+			(at 204.47 177.8 0)
+			(effects
+				(font

Commit message: x1p-002: layout rp2040 and new buck converters
Parts:
- LAN1: LCSC (none) -> C3021374
Changed lines of the file:
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@@
+			)
+		)
+		(property "LCSC" "C3021374"
+			(at 309.5341 54.61 0)
+			(effects
+				(font
+					(size 1.27 1.27)
+				)
+				(hide yes)
 			)
 		)

Commit message: x1p-002: move arrows, remove LAN1 silk, remove 0 ohm straps, add noozle and hatguy
Parts:
- removed R28, R29, R31, R32: 0, Resistor_SMD:R_0402_1005Metric, symbol Device:R_Small
Connections:
- net 3V3: now also U1.11 (VBUS_DET), U1.40 (TEST3)
- net GND: now also U1.34 (TEST2), U1.44 (CLK24_EN)

Commit message: X1P-002: scrub BOM and remove a stray 0402 0R
Parts:
- removed R33: 0, Resistor_SMD:R_0402_1005Metric, symbol Device:R_Small
- C10, C9: value 29pF -> 27pF C0G; Manufacturer (none) -> Guangdong Fenghua Advanced Tech; Manufacturer Part (none) -> 0402CG270J500NT
- C11, C29: Manufacturer SAMSUNG(三星) -> Samsung Electro-Mechanics
- C12, C13, C14, C15, C16, C17, C18, C22, C23, C24, C25, C26, C27, C28, C48: value 100nF -> 100nF X7R; Manufacturer SAMSUNG(三星) -> Samsung Electro-Mechanics
- C19: value .022uF -> 22nF X7R; Manufacturer (none) -> Samsung Electro-Mechanics; Manufacturer Part (none) -> CL10B223KB8NNNC; Origin Footprint C0805 -> C0603
- C21: value 100nF -> 100nF X7R; Manufacturer SAMSUNG(三星) -> Samsung Electro-Mechanics; Origin Footprint (none) -> C0402
- C45, C46: Manufacturer (none) -> Samsung Electro-Mechanics; Manufacturer Part (none) -> CL32A107MPVNNNE; Origin Footprint C0603 -> C1210
- D1: Origin Footprint SOT-23-6_L2.9-W1.6-P0.95-LS2.8-BL -> SOT-23-6
- FB1, FB2: Manufacturer muRata(村田) -> Murata Electronics
- LAN1: Manufacturer (none) -> HCTL; Manufacturer Part (none) -> HC913550A-M899-A
- R10, R12: Manufacturer (none) -> UNI-ROYAL; Manufacturer Part (none) -> 0402WGF1002TCE
- R11: Manufacturer (none) -> UNI-ROYAL; Manufacturer Part (none) -> 0402WGF1202TCE; Origin Footprint R0603 -> R0402
- R13, R9: Manufacturer (none) -> UNI-ROYAL; Manufacturer Part (none) -> 0603WAF3300T5E; Origin Footprint R0402 -> R0603
- R21, R26, R27, R30: Manufacturer (none) -> UNI-ROYAL; Manufacturer Part (none) -> 0603WAF0000T5E; Origin Footprint (none) -> R0603
- R25: Manufacturer (none) -> UNI-ROYAL; Manufacturer Part (none) -> 0402WGF100JTCE
- R34: Manufacturer (none) -> UNI-ROYAL; Manufacturer Part (none) -> 0402WGF1002TCE; Origin Footprint (none) -> R0402
- R6: Manufacturer UNI-ROYAL(厚声) -> UNI-ROYAL
- R7: Manufacturer (none) -> UNI-ROYAL; Manufacturer Part (none) -> 0603WAF1242T5E; Origin Footprint R0402 -> R0603
- RN1: Manufacturer YAGEO(国巨) -> YAGEO; Origin Footprint RES-ARRAY-SMD_0402-8P-L2.0-W1.0-BL -> 0402x4
- U1: Manufacturer MICROCHIP(美国微芯) -> Microchip Tech; Origin Footprint QFN64G-0.5-9X9MM -> QFN-64-EP
- U5: Manufacturer (none) -> Microchip Tech; Manufacturer Part (none) -> AT93C66B-SSHM-T; Origin Footprint (none) -> SOIC-8
- USB1: Manufacturer (none) -> XUNPU
- USB2: Manufacturer (none) -> XUNPU; Origin Footprint USB-226-BRW -> (none)
- X1: Manufacturer YXC(扬兴晶振) -> YXC Crystal Oscillators; Origin Footprint OSC-SMD_4P-L3.2-W2.5-BL -> SMD3225-4P
Connections:
- net GND: now also U5.6 (ORG)

Commit message: BOM scrub from mfg feedback
Parts:
- R10, R12: value 10K 1/10W 1% -> 10k
- R11: value 12k 1/10W 1% -> 12k 1%
- RN1: value 49.9 -> 4x 49.9
Changed lines of the file:
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@@
 			)
 		)
-		(property "Value" "12k 1/10W 1%"
+		(property "Value" "12k 1%"
 			(at 91.3384 85.0138 0)
 			(effects
@@
 			)
 		)
-		(property "Value" "10K 1/10W 1%"
+		(property "Value" "10k"
 			(at 92.71 154.0256 0)
 			(effects
@@
 			)
 		)
-		(property "Value" "49.9"
+		(property "Value" "4x 49.9"
 			(at 266.9286 58.3438 0)
 			(effects
@@
 			)
 		)
-		(property "Value" "10K 1/10W 1%"
+		(property "Value" "10k"
 			(at 92.4052 173.9138 0)
 			(effects
