File: x1p-002/x1-expander.kicad_pcb (KiCad board)
At the start: 4 copper layers, 145 x 57 mm, 130 parts, among them U1 LAN9514, U2 FT2232HL, U3 TPS54202DDCR, U4 LM1084S-3.3/TR, U5 M93C86-WMN6TP, X1 25MHz, X2 12MHz

Commit message: add pullup on FTDI EEDATA, swap EEPROM to 4k EEPROM
Parts:
- added R24: 10k, Resistor_SMD:R_0402_1005Metric, B.Cu at (180.8, 112.2)
- U5: value M93C86-WMN6TP -> AT93C66B-SSHM-T
- moved C40 0.40 mm to (182.8, 111.8), turned to -90 degrees
Connections:
- U2 pad 61: unconnected-(U2-EEDATA-Pad61) -> Net-(U2-EEDATA)
Routing:
- net Net-(U2-EEDATA): track 0.00 -> 5.94 mm
- net VCORE: track 11.1 -> 12.4 mm
- net 3V3: track 126.1 -> 126.9 mm, vias 41 -> 42

Commit message: replace rj45 component
Parts:
- added C49: .022uF, Capacitor_SMD:C_0603_1608Metric, F.Cu at (62.9, 105.0)
- added R25: 10 1/16W 1%, Resistor_SMD:R_0402_1005Metric, F.Cu at (61.0, 96.9)
- added RN2: 49.9, x1-expander:RES-ARRAY-SMD_0402-8P-L2.0-W1.0-BL, B.Cu at (79.7, 99.0)
- LAN1: value HR911103A -> HC913550A-M899-A; footprint x1-expander:RJ45-TH_HR911103A -> easyeda2kicad:RJ45-TH_HC913550A-M899-A
Connections:
- LAN1 pad 10: LNKA -> GND
- LAN1 pad 11: SPD -> LNKA
- LAN1 pad 13: GND -> SPD
- LAN1 pad 3: Net-(LAN1-RCT) -> RXP
- LAN1 pad 4: GND -> Net-(LAN1-RCT)
- LAN1 pad 5: GND -> Net-(LAN1-RCT)
- LAN1 pad 6: Net-(LAN1-RCT) -> RXN
- LAN1 pad 7: RXP -> unconnected-(LAN1-NC-Pad7)
- LAN1 pad 8: RXN -> GND
- LAN1 pad 9: 3V3 -> GND
Routing:
- net Net-(LAN1-RCT): track 11.4 -> 6.54 mm
- net TXN: track 37.2 -> 42.0 mm

Commit message: correct C3021374 footprint, route rj45
Parts:
- removed the C19 at (82.7, 99.5)
- removed R8: 10 1/16W 1%, Resistor_SMD:R_0402_1005Metric
- removed the RN1 at (102.1, 113.2)
- C19: renamed from C49; moved to B.Cu
- R25: moved to B.Cu
- moved RN1 26.6 mm to (102.2, 113.3), turned to 0 degrees
- moved R25 22.5 mm to (82.5, 103.4), turned to -90 degrees
- moved C19 20.1 mm to (82.5, 100.4), turned to -90 degrees
- moved R9 0.23 mm to (75.2, 97.2)
- renumbered RN2 to RN1
Connections:
- LAN1 pad 11: LNKA -> 3V3
- LAN1 pad 12: 3V3 -> LNKA
- RN1 pad 1: TXP -> TXN
- RN1 pad 2: TXN -> TXP
- RN1 pad 3: RXP -> RXN
Routing:
- net TXN: track 42.0 -> 36.7 mm
- net RXP: track 34.5 -> 37.0 mm
- net RXN: track 34.2 -> 36.5 mm
- net GND: track 82.7 -> 80.5 mm
- net 3V3: track 126.9 -> 128.7 mm
- net TXP: track 34.1 -> 33.5 mm

Commit message: replace F1 with proper rated part, relink RN1 with 3d model, adjust lan1 3d model z offset, move TXN & RXN meander near rj45
Parts:
- F1: value JK-NSMD100-16V -> BSMD1206-050-30V; footprint Fuse:Fuse_1206_3216Metric -> x1-expander:F1206

Commit message: replace F1 with C5358568 - BHFUSE BSMD1206-100-30V
Parts:
- F1: value BSMD1206-050-30V -> BSMD1206-100-30V
Changed lines of the file:
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@@
 		)
 	)
+	(footprint "x1-expander:F1206"
+		(layer "F.Cu")
+		(at 141.9 120.85 90)
+		(property "Reference" "F1"
+			(at 3.35 0 90)
+			(layer "F.SilkS")
+			(effects
+				(font
+					(size 1 1)
+					(thickness 0.15)
+				)
+			)
+		)
+		(property "Value" "BSMD1206-100-30V"
+			(at 0 4 90)
+			(layer "F.Fab")
+			(effects
+				(font
+					(size 1 1)
+					(thickness 0.15)
+				)
+			)
+		)
+		(property "Footprint" "x1-expander:F1206"
+			(at 0 0 90)
+			(layer "F.Fab")
+			(hide yes)
+			(effects
+				(font
+					(size 1.27 1.27)
+					(thickness 0.15)
+				)
+			)
+		)
+		(property "Datasheet" ""
+			(at 0 0 90)
+			(layer "F.Fab")
+			(hide yes)
+			(effects
+				(font
+					(size 1.27 1.27)
+					(thickness 0.15)
+				)
+			)
+		)
+		(property "Description" ""
+			(at 0 0 90)
+			(layer "F.Fab")
+			(hide yes)
+			(effects
+				(font
+					(size 1.27 1.27)
+					(thickness 0.15)
+				)
+			)
+		)
+		(property "LCSC Part" "C5358568"
+			(at 0 0 90)
+			(unlocked yes)
+			(layer "F.Fab")
+			(hide yes)
+			(effects
+				(font
+					(size 1 1)
+					(thickness 0.15)
+				)
+			)
+		)
+		(sheetname "MAIN")
+		(sheetfile "1_MAIN.kicad_sch")
+		(attr smd)
+		(fp_line
+			(start 0.93 -1.09)
+			(end 2.12 -1.09)
+			(stroke
+				(width 0.15)
+				(type solid)
+			)
+			(layer "F.SilkS")
+		)
+		(fp_line
+			(start -0.93 -1.09)
+			(end -2.12 -1.09)
+			(stroke
+				(width 0.15)
+				(type solid)
+			)
+			(layer "F.SilkS")
+		)
+		(fp_line
+			(start 2.27 -0.94)
+			(end 2.27 0.94)
+			(stroke
+				(width 0.15)
+				(type solid)
+			)
+			(layer "F.SilkS")
+		)
+		(fp_line
+			(start -2.27 -0.94)
+			(end -2.27 0.94)
+			(stroke
+				(width 0.15)
+				(type solid)
+			)
+			(layer "F.SilkS")
+		)
+		(fp_line
+			(start 2.12 1.09)
+			(end 0.93 1.09)
+			(stroke
+				(width 0.15)
+				(type solid)
+			)
+			(layer "F.SilkS")
+		)
+		(fp_line
+			(start -2.12 1.09)
+			(end -0.93 1.09)
+			(stroke
+				(width 0.15)
+				(type solid)
+			)
+			(layer "F.SilkS")
+		)
+		(fp_arc
+			(start -0.001269 -0.002199)
+			(mid 0.112199 0.418731)
+			(end 0 0.84)
+			(stroke
+				(width 0.08)
+				(type solid)
+			)
+			(layer "F.SilkS")
+		)
+		(fp_arc
+			(start 0.001269 0.002199)
+			(mid -0.112199 -0.418731)
+			(end 0 -0.84)
+			(stroke
+				(width 0.08)
+				(type solid)
+			)
+			(layer "F.SilkS")
+		)
+		(fp_circle
+			(center -1.6 0.8)
+			(end -1.57 0.8)
+			(stroke
+				(width 0.06)
+				(type solid)
+			)
+			(fill none)
+			(layer "F.Fab")
+		)
+		(fp_text user "${REFERENCE}"
+			(at 0 0 90)
+			(layer "F.Fab")
+			(effects
+				(font
+					(size 1 1)
+					(thickness 0.15)
+				)
+			)
+		)
+		(pad "1" smd rect
+			(at -1.45 0 90)
+			(size 1.19 1.73)
+			(layers "F.Cu" "F.Paste" "F.Mask")
+			(net 45 "24V")
+			(pinfunction "1")
+			(pintype "unspecified")
+		)
+		(pad "2" smd rect
+			(at 1.45 0 90)
+			(size 1.19 1.73)
+			(layers "F.Cu" "F.Paste" "F.Mask")
+			(net 1 "Net-(AP_HARNESS1-Pad2)")
+			(pinfunction "2")
+			(pintype "unspecified")
+		)
+		(model "/x1-expander.3dshapes/F1206_L3.2-W1.7-H0.6.wrl"
+			(offset
+				(xyz 0 -0 -0)
+			)
+			(scale
+				(xyz 1 1 1)
+			)
+			(rotate
+				(xyz 0 0 0)
+			)
+		)
+	)
 	(footprint "Resistor_SMD:R_0402_1005Metric"
 		(layer "F.Cu")
@@
 			)
 			(scale
-				(xyz 1 1 1)
-			)
-			(rotate
-				(xyz 0 0 0)
-			)
-		)
-	)
-	(footprint "x1-expander:F1206"
-		(layer "F.Cu")
-		(at 141.9 120.85 90)
-		(property "Reference" "F1"
-			(at 3.65 0 90)
-			(layer "F.SilkS")
-			(effects
-				(font
-					(size 1 1)
-					(thickness 0.15)
-				)
-			)
-		)
-		(property "Value" "BSMD1206-050-30V"
-			(at 0 4 90)
-			(layer "F.Fab")
-			(effects
-				(font
-					(size 1 1)
-					(thickness 0.15)
-				)
-			)
-		)
-		(property "Footprint" "x1-expander:F1206"
-			(at 0 0 90)
-			(layer "F.Fab")
-			(hide yes)
-			(effects
-				(font
-					(size 1.27 1.27)
-					(thickness 0.15)
-				)
-			)
-		)
-		(property "Datasheet" "https://lcsc.com/product-detail/PTC-Resettable-Fuses_BHFUSE-BSMD1206-050-30V_C883126.html"
-			(at 0 0 90)
-			(layer "F.Fab")
-			(hide yes)
-			(effects
-				(font
-					(size 1.27 1.27)
-					(thickness 0.15)
-				)
-			)
-		)
-		(property "Description" "30V 500ma 1A"
-			(at 0 0 90)
-			(layer "F.Fab")
-			(hide yes)
-			(effects
-				(font
-					(size 1.27 1.27)
-					(thickness 0.15)
-				)
-			)
-		)
-		(property "LCSC Part" "C883126"
-			(at 0 0 90)
-			(unlocked yes)
-			(layer "F.Fab")
-			(hide yes)
-			(effects
-				(font
-					(size 1 1)
-					(thickness 0.15)
-				)
-			)
-		)
-		(sheetname "MAIN")
-		(sheetfile "1_MAIN.kicad_sch")
-		(attr smd)
-		(fp_line
-			(start 0.93 -1.09)
-			(end 2.12 -1.09)
-			(stroke
-				(width 0.15)
-				(type solid)
-			)
-			(layer "F.SilkS")
-		)
-		(fp_line
-			(start -0.93 -1.09)
-			(end -2.12 -1.09)
-			(stroke
-				(width 0.15)
-				(type solid)
-			)
-			(layer "F.SilkS")
-		)
-		(fp_line
-			(start 2.27 -0.94)
-			(end 2.27 0.94)
-			(stroke
-				(width 0.15)
-				(type solid)
-			)
-			(layer "F.SilkS")
-		)
-		(fp_line
-			(start -2.27 -0.94)
-			(end -2.27 0.94)
-			(stroke
-				(width 0.15)
-				(type solid)
-			)
-			(layer "F.SilkS")
-		)
-		(fp_line
-			(start 2.12 1.09)
-			(end 0.93 1.09)
-			(stroke
-				(width 0.15)
-				(type solid)
-			)
-			(layer "F.SilkS")
-		)
-		(fp_line
-			(start -2.12 1.09)
-			(end -0.93 1.09)
-			(stroke
-				(width 0.15)
-				(type solid)
-			)
-			(layer "F.SilkS")
-		)
-		(fp_arc
-			(start -0.001269 -0.002199)
-			(mid 0.112199 0.418731)
-			(end 0 0.84)
-			(stroke
-				(width 0.08)
-				(type solid)
-			)
-			(layer "F.SilkS")
-		)
-		(fp_arc
-			(start 0.001269 0.002199)
-			(mid -0.112199 -0.418731)
-			(end 0 -0.84)
-			(stroke
-				(width 0.08)
-				(type solid)
-			)
-			(layer "F.SilkS")
-		)
-		(fp_circle
-			(center -1.6 0.8)
-			(end -1.57 0.8)
-			(stroke
-				(width 0.06)
-				(type solid)
-			)
-			(fill none)
-			(layer "F.Fab")
-		)
-		(fp_text user "${REFERENCE}"
-			(at 0 0 90)
-			(layer "F.Fab")
-			(effects
-				(font
-					(size 1 1)
-					(thickness 0.15)
-				)
-			)
-		)
-		(pad "1" smd rect
-			(at -1.45 0 90)
-			(size 1.19 1.73)
-			(layers "F.Cu" "F.Paste" "F.Mask")
-			(net 45 "24V")
-			(pinfunction "1")
-			(pintype "unspecified")
-		)
-		(pad "2" smd rect
-			(at 1.45 0 90)
-			(size 1.19 1.73)
-			(layers "F.Cu" "F.Paste" "F.Mask")
-			(net 1 "Net-(AP_HARNESS1-Pad2)")
-			(pinfunction "2")
-			(pintype "unspecified")
-		)
-		(model "/x1-expander.3dshapes/F1206_L3.2-W1.7-H0.6.wrl"
-			(offset
-				(xyz 0 -0 -0)
-			)
-			(scale
