File: x1p-002/x1-expander.kicad_pcb (KiCad board)
At the start: 4 copper layers, 145 x 57 mm, 149 parts, among them J1 TC2050-IDC-NL, U1 LAN9514, U2 RP2040, U3 AP22615AWU-7, U4 SY8205FCC, U5 AT93C66B-SSHM-T, U6 SY8205FCC, U7 AP22615AWU-7, X1 25MHz, Y1 ABM8-272-T3

Commit message: X1P-002: scrub BOM and remove a stray 0402 0R
Parts:
- removed R33: 0, Resistor_SMD:R_0402_1005Metric
- C10, C9: value 29pF -> 27pF C0G
- C12, C13, C14, C15, C16, C17, C18, C21, C22, C23, C24, C25, C26, C27, C28, C33, C34, C35, C36, C37, C38, C39, C40, C41, C48, C53: value 100nF -> 100nF X7R
- C19: value .022uF -> 22nF X7R
- C20, C30: value 15p -> 15pF
- C4, C55, C6: value 100nF 35V -> 100nF X7R
- C47, C50, C52, C57, C58, C60, C8: value 22uF -> 22uF 6.3V
- C49, C59: value 75pF -> 75pF NP0
Connections:
- U5 pad 6: Net-(U5-ORG) -> GND
Routing:
- net GND: track 72.6 -> 70.5 mm
- net Net-(U5-ORG): track 2.01 -> 0.00 mm
Other:
- board text added: "X1P-002-Cxx"
- board text removed: "X1P-002-C01"

Commit message: BOM scrub from mfg feedback
Other:
- rule pad_to_mask_clearance: 0.038 -> 0
- board text added: "0"
- board text added: "0 mm"
- board text added: "0.01 mm"
- board text added: "0.02"
- board text added: "0.035 mm"
- board text added: "0.0900 mm / 0.1270 mm"
- board text added: "0.1 mm"
- board text added: "0.2000 mm"
- board text added: "1"
- board text added: "1.24 mm"
- board text added: "1.6000 mm"
- board text added: "145.0000 mm x 57.0000 mm"
- board text added: "4"
- board text added: "4.5"
- board text added: "BOARD CHARACTERISTICS"
- board text added: "Board Thickness:"
- board text added: "Board overall dimensions:"
- board text added: "Bottom Layer"
- board text added: "Bottom Paste Mask Layer"
- board text added: "Bottom Silk Screen"
- board text added: "Bottom Silkscreen Layer"
- board text added: "Bottom Solder Mask"
- board text added: "Bottom Solder Mask Layer"
- board text added: "Bottom Solder Paste"
- board text added: "Castellated pads:"
- board text added: "Color"
- board text added: "Copper Finish:"
- board text added: "Copper Layer Count:"
- board text added: "Dielectric 1"
- board text added: "Dielectric 2"
- board text added: "Dielectric 3"
- board text added: "Edge card connectors:"
- board text added: "Epsilon R"
- board text added: "FR4"
- board text added: "HASL lead-free (ENIG OK)"
- board text added: "Impedance Control:"
- board text added: "In1.Cu"
- board text added: "In2.Cu"
- board text added: "Layer Name"
- board text added: "Loss Tangent"
- board text added: "Material"
- board text added: "Min hole diameter:"
- board text added: "Min track/spacing:"
- board text added: "No"
- board text added: "Not specified"
- board text added: "Plated Board Edge:"
- board text added: "Stackup may be modified subject to X1Plus approval and appropriate impedance controls"
- board text added: "Thickness (mm)"
- board text added: "Top Layer"
- board text added: "Top Paste Mask Layer"
- board text added: "Top Silk Screen"
- board text added: "Top Silkscreen Layer"
- board text added: "Top Solder Mask"
- board text added: "Top Solder Mask Layer"
- board text added: "Top Solder Paste"
- board text added: "Type"
- board text added: "X1P-002-Cx1"
- board text added: "Yes"
- board text added: "copper"
- board text added: "core"
- board text added: "prepreg"
- board text removed: "X1P-002-Cxx"

Commit message: X1P-002: set 5V OCP to 1.8A (fixes #74)
Parts:
- R10, R12: value 10K 1/10W 1% -> 10k
- R11: value 12k 1/10W 1% -> 12k 1%
- R38: value 3.4k -> 3.74k
- RN1: value 49.9 -> 4x 49.9
- UART1: value P125-1104A0BR138A1 -> DZ254W-11-04-65
Changed lines of the file:
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@@
 		)
 		(fp_text user "${REFERENCE}"
-			(at 0 0 270)
+			(at 0 0 -90)
 			(layer "F.Fab")
 			(hide yes)
@@
 			)
 		)
-		(property "Value" "P125-1104A0BR138A1"
+		(property "Value" "DZ254W-11-04-65"
 			(at 0 0 0)
 			(unlocked yes)
@@
 			)
 		)
-		(property "Value" "10K 1/10W 1%"
+		(property "Value" "10k"
 			(at 0 1.17 0)
 			(layer "F.Fab")
@@
 			)
 		)
-		(property "Value" "12k 1/10W 1%"
+		(property "Value" "12k 1%"
 			(at 0 1.17 90)
 			(layer "F.Fab")
@@
 			)
 		)
-		(property "Value" "3.4k"
+		(property "Value" "3.74k"
 			(at 0 1.17 0)
 			(layer "F.Fab")
@@
 			)
 		)
-		(property "LCSC" "C4940"
+		(property "LCSC" "C15172"
 			(at 0 0 180)
 			(unlocked yes)
@@
 			)
 		)
-		(property "Manufacturer Part" "0402WGF3401TCE"
+		(property "Manufacturer Part" "0402WGF3741TCE"
 			(at 0 0 180)
 			(unlocked yes)
@@
 			)
 		)
-		(property "Manufacturer Part" "CYA0630-15UH"
+		(property "Manufacturer Part" "CYA0630-6.8UH"
 			(at 0 0 -90)
 			(unlocked yes)
@@
 			)
 		)
-		(property "LCSC" "C5189959"
+		(property "LCSC" "C5189749"
 			(at 0 0 -90)
 			(unlocked yes)
@@
 			)
 		)
-		(property "Value" "10K 1/10W 1%"
+		(property "Value" "10k"
 			(at 0 1.17 180)
 			(layer "F.Fab")
@@
 			)
 		)
-		(property "Manufacturer Part" "0402WGF1002TCE"
+		(property "Manufacturer Part" "0603WAF4701T5E"
 			(at 0 0 90)
 			(unlocked yes)
@@
 			)
 		)
-		(property "Manufacturer Part" "0402WGF1002TCE"
+		(property "Manufacturer Part" "0603WAF4701T5E"
 			(at 0 0 90)
 			(unlocked yes)
@@
 			)
 		)
-		(property "Value" "49.9"
+		(property "Value" "4x 49.9"
 			(at 0 0 180)
 			(unlocked yes)

Commit message: X1P-002: remove LLM-generated art; make sticker space 1" x 0.5" (fixes #72)
Parts:
- removed the G*** at (185.9, 134.6)
- moved G*** 36.6 mm to (208.5, 114.4)
- moved G*** 20.2 mm to (208.5, 121.5)
- moved REF** 9.28 mm to (208.5, 129.0)
Other:
- board text added: "RP2040 SWD+UART"
- board text removed: "RP2040 debug (see schem)"
