File: x1p-002/x1-expander.kicad_pcb (KiCad board)
At the start: 4 copper layers, 145 x 57 mm, 147 parts, among them J1 TC2050-IDC-NL, U1 LAN9514, U2 RP2040, U3 AP22615AWU-7, U4 SY8205FCC, U5 AT93C66B-SSHM-T, U6 SY8205FCC, U7 AP22615AWU-7, X1 25MHz, Y1 ABM8-272-T3

Commit message: X1P-002: clean up 5V power supply errata (fixes #73)
Parts:
- C47, C50, C8: value 22uF 6.3V -> 22uF 6.3V X7R; footprint Capacitor_SMD:C_0603_1608Metric -> Capacitor_SMD:C_1210_3225Metric
- C49: value 75pF NP0 -> 100pF NP0
- moved C8 4.12 mm to (148.2, 132.2), turned to 180 degrees
- moved C50 2.42 mm to (143.2, 131.6)
- moved C47 1.07 mm to (142.1, 128.4)
Routing:
- net Net-(U6-BS): track 6.91 -> 7.61 mm
- net GND: vias 296 -> 300
- net 5V: vias 16 -> 19
Other:
- board text added: "RP2040"
- board text removed: "RP2040 SWD+UART"

Commit message: tweak logo positions, tweak testpoint footprints; release x1p-002-c02
Parts:
- added REF**: UKCA-Logo_6x6mm_SilkScreen, Symbol:UKCA-Logo_6x6mm_SilkScreen, B.Cu at (201.0, 133.0)
- added REF**: WEEE-Logo_4.2x6mm_SilkScreen, Symbol:WEEE-Logo_4.2x6mm_SilkScreen, B.Cu at (179.5, 133.0)
- added REF**: CE-Logo_8.5x6mm_SilkScreen, Symbol:CE-Logo_8.5x6mm_SilkScreen, B.Cu at (190.0, 133.0)
- C11: footprint Capacitor_SMD:C_0805_2012Metric -> Capacitor_SMD:C_0603_1608Metric
- G***: moved to B.Cu
- TP1, TP2, TP3, TP4, TP5, TP6, TP7, TP8: footprint TestPoint:TestPoint_Pad_D1.0mm -> TestPoint:TestPoint_Pad_D1.5mm
- moved G*** 39.7 mm to (170.5, 133.0), turned to 180 degrees
- moved G*** 5.62 mm to (208.5, 120.0)
- moved REF** 1.50 mm to (208.5, 127.5)
Routing:
- net GND: vias 300 -> 299
Other:
- outline, holes or cut-outs redrawn
- board text added: "Black"
- board text added: "ENIG"
- board text added: "Solder mask color:"
- board text added: "X1P-002-C02"
- board text removed: "HASL lead-free (ENIG OK)"
- board text removed: "X1P-002-Cx1"

Commit message: x1p-002: fix silkscreen placement
Other:
- board text added: "X1P-002-C03"
- board text removed: "X1P-002-C02"
Changed lines of the file:
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@@
 	(title_block
 		(title "X1Plus Expander Board X1P-002")
-		(date "2024-12-20")
-		(rev "C02")
+		(date "2024-01-03")
+		(rev "C03")
 	)
 	(layers
@@
 		(tags "resistor")
 		(property "Reference" "R36"
-			(at 2.5 -1.125 90)
+			(at 2.5 0.125 90)
 			(layer "F.SilkS")
 			(effects
@@
 		(tags "capacitor")
 		(property "Reference" "C55"
-			(at -2.5 -1.25 90)
+			(at -2.5 0.125 90)
 			(layer "F.SilkS")
 			(effects
@@
 		)
 	)
-	(gr_text "X1P-002-C02"
+	(gr_text "X1P-002-C03"
 		(at 177.375 137.625 0)
 		(layer "F.SilkS")

Commit message: x1p-002: feedforward component and silkscreen changes
Parts:
- C49: value 100pF NP0 -> 470pF NP0
- C59: value 75pF NP0 -> 220pF NP0
Changed lines of the file:
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@@
 	(paper "A4")
 	(title_block
-		(title "X1Plus Expander Board X1P-002")
+		(title "X1Plus Expander X1P-002")
 		(date "2024-01-03")
 		(rev "C03")
@@
 		(tags "resistor")
 		(property "Reference" "R17"
-			(at -2.5 -1.25 0)
+			(at -2.625 0.25 0)
 			(layer "F.SilkS")
 			(effects
@@
 		(tags "capacitor")
 		(property "Reference" "C8"
-			(at 0 -2.3 0)
+			(at 0 -3.75 0)
 			(layer "F.SilkS")
 			(effects
@@
 		(at 148 126.355 -90)
 		(property "Reference" "L1"
-			(at 4.475 -2.625 0)
+			(at 8.145 -0.25 0)
 			(layer "F.SilkS")
 			(effects
@@
 		(tags "resistor")
 		(property "Reference" "R14"
-			(at 2.5 -1.25 0)
+			(at 2.625 0.25 0)
 			(layer "F.SilkS")
 			(effects
@@
 			)
 		)
-		(property "Value" "75pF NP0"
+		(property "Value" "220pF NP0"
 			(at 0 1.16 0)
 			(layer "F.Fab")
@@
 			)
 		)
-		(property "LCSC" "C107010"
+		(property "LCSC" "C107001"
 			(at 0 0 180)
 			(unlocked yes)
@@
 			)
 		)
-		(property "Manufacturer Part" "CC0402JRNPO9BN750"
+		(property "Manufacturer Part" "CC0402JRNPO9BN221"
 			(at 0 0 180)
 			(unlocked yes)
@@
 			)
 		)
-		(property "Value" "100pF NP0"
+		(property "Value" "470pF NP0"
 			(at 0 1.16 0)
 			(layer "F.Fab")
@@
 			)
 		)
-		(property "LCSC" "C106200"
+		(property "LCSC" "C526993"
 			(at 0 0 180)
 			(unlocked yes)
@@
 			)
 		)
-		(property "Manufacturer Part" "CC0402JRNPO9BN101"
+		(property "Manufacturer Part" "CC0402JRNPO7BN471"
 			(at 0 0 180)
 			(unlocked yes)
@@
 		(end 203.75 138.25)
 		(stroke
-			(width 0.5)
+			(width 0.3)
 			(type solid)
 		)
@@
 	)
 	(gr_text "X1P-002-C03"
-		(at 177.375 137.625 0)
+		(at 190.25 131.75 0)
 		(layer "F.SilkS")
 		(effects
@@
 				(bold yes)
 			)
-			(justify left bottom)
 		)
 	)
