File: x1p-002/x1-expander.kicad_sch (KiCad schematic)
At the start: 0 parts

Commit message: X1P-002: schematic: redesign with larger 5V buck (#60), add 3V3 buck (#63), add OCP circuits for 3V3 and 5V (but not connected to user ports yet; #61)
Other:
- sheet LAN renamed LAN9514
- sheet MAIN renamed FTDI
- added sheet Power (power.kicad_sch)
- note added: "24Vsys polyfuse 24V -> 5V Buck 5V -> 3V3 Buck User power OCP Power status LEDs"
- title: (none) -> X1Plus Expansion Board: X1P-002
Changed lines of the file:
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@@
 	(generator "eeschema")
 	(generator_version "8.0")
-	(paper "A4")
+	(paper "USLetter")
+	(title_block
+		(title "X1Plus Expansion Board: X1P-002")
+		(rev "X1P-002-B01")
+	)
+	(text "24Vsys polyfuse\n24V -> 5V Buck\n5V -> 3V3 Buck\nUser power OCP\nPower status LEDs"
+		(exclude_from_sim no)
+		(at 51.054 55.626 0)
+		(effects
+			(font
+				(size 1.27 1.27)
+			)
+		)
+	)
 	(sheet
-		(at 5.08 5.08)
+		(at 34.29 43.18)
+		(size 34.29 24.13)
+		(fields_autoplaced yes)
+		(stroke
+			(width 0.1524)
+			(type solid)
+		)
+		(fill
+			(color 0 0 0 0.0000)
+		)
+		(property "Sheetname" "Power"
+			(at 34.29 42.4684 0)
+			(effects
+				(font
+					(size 1.27 1.27)
+				)
+				(justify left bottom)
+			)
+		)
+		(property "Sheetfile" "power.kicad_sch"
+			(at 34.29 67.8946 0)
+			(effects
+				(font
+					(size 1.27 1.27)
+				)
+				(justify left top)
+			)
+		)
+		(instances
+			(project "x1-expander"
+				(path "/5c4052f8-31d6-4de3-b862-4d09b0660e26"
+					(page "5")
+				)
+			)
+		)
+	)
+	(sheet
+		(at 86.36 43.18)
 		(size 12.7 3.81)
 		(fields_autoplaced yes)
@@
 			(color 0 0 0 0.0000)
 		)
-		(property "Sheetname" "MAIN"
-			(at 5.08 4.3684 0)
+		(property "Sheetname" "FTDI"
+			(at 86.36 42.4684 0)
 			(effects
 				(font
@@
 		)
 		(property "Sheetfile" "1_MAIN.kicad_sch"
-			(at 5.08 9.4746 0)
+			(at 86.36 47.5746 0)
 			(effects
 				(font
@@
 	)
 	(sheet
-		(at 5.08 22.86)
+		(at 86.36 60.96)
 		(size 12.7 3.81)
 		(fields_autoplaced yes)
@@
 		)
 		(property "Sheetname" "GPIO"
-			(at 5.08 22.1484 0)
+			(at 86.36 60.2484 0)
 			(effects
 				(font
@@
 		)
 		(property "Sheetfile" "3_GPIO.kicad_sch"
-			(at 5.08 27.2546 0)
+			(at 86.36 65.3546 0)
 			(effects
 				(font
@@
 	)
 	(sheet
-		(at 5.08 13.97)
+		(at 86.36 52.07)
 		(size 12.7 3.81)
 		(fields_autoplaced yes)
@@
 			(color 0 0 0 0.0000)
 		)
-		(property "Sheetname" "LAN"
-			(at 5.08 13.2584 0)
+		(property "Sheetname" "LAN9514"
+			(at 86.36 51.3584 0)
 			(effects
 				(font
@@
 		)
 		(property "Sheetfile" "2_LAN.kicad_sch"
-			(at 5.08 18.3646 0)
+			(at 86.36 56.4646 0)
 			(effects
 				(font
