File: x1p-002/x1-expander.kicad_sch (KiCad schematic)
At the start: 0 parts

Commit message: x1p-002: WIP: rp2040 schematic
Parts:
- added AP_HARNESS1: HC-1.25-12PWT, x1-expander:CONN-SMD_12P-P1.25_HCTL_HC-1.25-12PWT, symbol x1-expander:HC-1.25-12PWT
- added D10: SRV05-4.TCT_C2687126, x1-expander:SOT-23-6_L2.9-W1.6-P0.95-LS2.8-BL, symbol x1-expander:SRV05-4.TCT_C2687126
- added UART1: P125-1104A0BR138A1, x1-expander:HDR-TH_4P-P2.54-H-M-W10.3, symbol x1-expander:P125-1104A0BR138A1
Connections:
- new net 24V_SYS: AP_HARNESS1.2
- new net 3V3_USER: D10.5, UART1.1
- new net 5V: AP_HARNESS1.12
- new net CAMO_DN: AP_HARNESS1.11
- new net CAMO_DP: AP_HARNESS1.10
- new net GND: AP_HARNESS1.1, AP_HARNESS1.3, AP_HARNESS1.9, D10.2, UART1.4
- new net MBDN: AP_HARNESS1.8
- new net MBDP: AP_HARNESS1.7
- new net UARTRX: AP_HARNESS1.5, D10.1, D10.6, UART1.2
- new net UARTTX: AP_HARNESS1.4, D10.3, D10.4, UART1.3
- no-connect marks 0 -> 3
Other:
- sheet FTDI renamed RP2040
- sheet RP2040: file FTDI.kicad_sch -> RP2040.kicad_sch
- note added: "AP UART PASSTHROUGH"
- note added: "Main AP harness UART passthrough"
- note added: "UART ESD"

Commit message: X1P-002: finish connecting GPIO ports to RP2040
Changed lines of the file:
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@@
 	(symbol
 		(lib_id "Graphic:Logo_Open_Hardware_Small")
-		(at 40.64 114.3 0)
+		(at 165.1 111.76 0)
 		(unit 1)
 		(exclude_from_sim yes)
@@
 		(fields_autoplaced yes)
 		(property "Reference" "#SYM1"
-			(at 40.64 107.315 0)
+			(at 165.1 104.775 0)
 			(effects
 				(font
@@
 		)
 		(property "Value" "Logo_Open_Hardware_Small"
-			(at 40.64 120.015 0)
+			(at 165.1 117.475 0)
 			(effects
 				(font
@@
 		)
 		(property "Footprint" ""
-			(at 40.64 114.3 0)
+			(at 165.1 111.76 0)
 			(effects
 				(font
@@
 		)
 		(property "Datasheet" "~"
-			(at 40.64 114.3 0)
+			(at 165.1 111.76 0)
 			(effects
 				(font
@@
 		)
 		(property "Description" "Open Hardware logo, small"
-			(at 40.64 114.3 0)
+			(at 165.1 111.76 0)
 			(effects
 				(font

Commit message: X1P-002: scrub BOM and remove a stray 0402 0R
Parts:
- D10: Origin Footprint SOT-23-6_L2.9-W1.6-P0.95-LS2.8-BL -> SOT-23-6
- UART1: Manufacturer Yxcon(宇熙精密) -> DEALON; Manufacturer Part P125-1104A0BR138A1 -> DZ254W-11-04-65; Origin Footprint HDR-TH_4P-P2.54-H-M-W10.3 -> (none)
Changed lines of the file:
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@@
 			)
 		)
-		(property "Manufacturer" "Yxcon(宇熙精密)"
-			(at 224.79 66.04 0)
-			(effects
-				(font
-					(size 1.27 1.27)
-				)
-				(justify left bottom)
-				(hide yes)
-			)
-		)
-		(property "Manufacturer Part" "P125-1104A0BR138A1"
-			(at 224.79 66.04 0)
-			(effects
-				(font
-					(size 1.27 1.27)
-				)
-				(justify left bottom)
-				(hide yes)
-			)
-		)
-		(property "Origin Footprint" "HDR-TH_4P-P2.54-H-M-W10.3"
+		(property "Manufacturer" "DEALON"
+			(at 224.79 66.04 0)
+			(effects
+				(font
+					(size 1.27 1.27)
+				)
+				(justify left bottom)
+				(hide yes)
+			)
+		)
+		(property "Manufacturer Part" "DZ254W-11-04-65"
+			(at 224.79 66.04 0)
+			(effects
+				(font
+					(size 1.27 1.27)
+				)
+				(justify left bottom)
+				(hide yes)
+			)
+		)
+		(property "Origin Footprint" ""
 			(at 224.79 66.04 0)
 			(effects
@@
 			)
 		)
-		(property "Origin Footprint" "SOT-23-6_L2.9-W1.6-P0.95-LS2.8-BL"
-			(at 228.6 101.6 90)
-			(effects
+		(property "Origin Footprint" "SOT-23-6"
+			(at 228.6 101.6 90)
+			(effects

Commit message: BOM scrub from mfg feedback
Parts:
- UART1: value P125-1104A0BR138A1 -> DZ254W-11-04-65
Changed lines of the file:
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@@
 			)
 		)
-		(property "Value" "P125-1104A0BR138A1"
+		(property "Value" "DZ254W-11-04-65"
 			(at 221.742 59.2074 0)
 			(effects
