File: x1p-002/power.kicad_sch (KiCad schematic)
At the start: 51 parts, among them U3 AP22615AWU-7, U4 SY8205FCC, U6 SY8205FCC, U7 AP22615AWU-7

Commit message: x1p-002: layout rp2040 and new buck converters
Parts:
- C4, C55, C6, C7: footprint Capacitor_SMD:C_0603_1608Metric -> Capacitor_SMD:C_0402_1005Metric; LCSC C14663 -> C1525; Origin Footprint C0603 -> (none)
- C49, C59: footprint Capacitor_SMD:C_0603_1608Metric -> Capacitor_SMD:C_0402_1005Metric; LCSC C1681 -> C107010; Origin Footprint C0603 -> (none)
- C53, C56: footprint Capacitor_SMD:C_0603_1608Metric -> Capacitor_SMD:C_0402_1005Metric; LCSC C14663 -> C1525
- F1: LCSC (none) -> C21714343
- R37: LCSC (none) -> C93940
- R38: LCSC (none) -> C4940
- R4: footprint Resistor_SMD:R_1206_3216Metric -> Resistor_SMD:R_0603_1608Metric; LCSC C26045 -> C138278; Manufacturer Part 1206W4J0562T5E -> (none); Origin Footprint R1206 -> (none); Supplier Part C26045 -> (none)
- U3, U7: LCSC (none) -> C2680357
- U4, U6: LCSC (none) -> C111875
Changed lines of the file:
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@@
 			)
 		)
+		(property "LCSC" "C111875"
+			(at 132.08 27.7325 0)
+			(effects
+				(font
+					(size 1.27 1.27)
+				)
+				(hide yes)
+			)
+		)
 		(pin "9"
 		)
@@
 			)
 		)
-		(property "Footprint" "Capacitor_SMD:C_0603_1608Metric"
+		(property "Footprint" "Capacitor_SMD:C_0402_1005Metric"
 			(at 80.01 118.11 0)
 			(effects
@@
 			)
 		)
-		(property "LCSC" "C14663"
+		(property "LCSC" "C1525"
 			(at 75.2856 119.634 0)
 			(effects
@@
 			)
 		)
+		(property "LCSC" "C21714343"
+			(at 36.83 34.3325 0)
+			(effects
+				(font
+					(size 1.27 1.27)
+				)
+				(hide yes)
+			)
+		)
 		(pin "2"
 		)
@@
 			)
 		)
+		(property "LCSC" "C93940"
+			(at 186.9186 115.6278 0)
+			(effects
+				(font
+					(size 1.27 1.27)
+				)
+				(hide yes)
+			)
+		)
 		(pin "2"
 		)
@@
 			)
 		)
+		(property "LCSC" "C2680357"
+			(at 198.12 135.6825 0)
+			(effects
+				(font
+					(size 1.27 1.27)
+				)
+				(hide yes)
+			)
+		)
 		(pin "3"
 		)
@@
 			)
 		)
-		(property "Footprint" "Capacitor_SMD:C_0603_1608Metric"
+		(property "Footprint" "Capacitor_SMD:C_0402_1005Metric"
 			(at 31.75 118.11 0)
 			(effects
@@
 			)
 		)
-		(property "LCSC" "C14663"
+		(property "LCSC" "C1525"
 			(at 32.9438 115.57 0)
 			(effects
@@
 			)
 		)
-		(property "Footprint" "Capacitor_SMD:C_0603_1608Metric"
+		(property "Footprint" "Capacitor_SMD:C_0402_1005Metric"
 			(at 120.65 133.35 0)
 			(effects
@@
 			)
 		)
-		(property "Origin Footprint" "C0603"
+		(property "Origin Footprint" ""
 			(at 120.65 133.35 90)
 			(effects
@@
 			)
 		)
-		(property "LCSC" "C1681"
+		(property "LCSC" "C107010"
 			(at 121.8438 130.81 0)
 			(effects
@@
 			)
 		)
+		(property "LCSC" "C2680357"
+			(at 198.12 100.1225 0)
+			(effects
+				(font
+					(size 1.27 1.27)
+				)
+				(hide yes)
+			)
+		)
 		(pin "3"
 		)
@@
 			)
 		)
-		(property "Footprint" "Resistor_SMD:R_1206_3216Metric"
+		(property "Footprint" "Resistor_SMD:R_0603_1608Metric"
 			(at 232.41 54.61 0)
 			(effects
@@
 			)
 		)
-		(property "Manufacturer Part" "1206W4J0562T5E"
+		(property "Manufacturer Part" ""
 			(at 232.41 54.61 90)
 			(effects
@@
 			)
 		)
-		(property "Origin Footprint" "R1206"
+		(property "Origin Footprint" ""
 			(at 232.41 54.61 90)
 			(effects
@@
 			)
 		)
-		(property "Supplier Part" "C26045"
+		(property "Supplier Part" ""
 			(at 232.41 54.61 90)
 			(effects
@@
 			)
 		)
-		(property "LCSC" "C26045"
+		(property "LCSC" "C138278"
 			(at 233.6038 53.086 0)
 			(effects
@@
 			)
 		)
-		(property "Footprint" "Capacitor_SMD:C_0603_1608Metric"
+		(property "Footprint" "Capacitor_SMD:C_0402_1005Metric"
 			(at 104.14 44.45 0)
 			(effects
@@
 			)
 		)
-		(property "Origin Footprint" "C0603"
+		(property "Origin Footprint" ""
 			(at 104.14 44.45 90)
 			(effects
@@
 			)
 		)
-		(property "LCSC" "C14663"
+		(property "LCSC" "C1525"
 			(at 105.3338 41.91 0)
 			(effects
@@
 			)
 		)
-		(property "Footprint" "Capacitor_SMD:C_0603_1608Metric"
+		(property "Footprint" "Capacitor_SMD:C_0402_1005Metric"
 			(at 73.66 128.27 0)
 			(effects
@@
 			)
 		)
-		(property "Origin Footprint" "C0603"
+		(property "Origin Footprint" ""
 			(at 73.66 128.27 90)
 			(effects
@@
 			)
 		)
-		(property "LCSC" "C14663"
+		(property "LCSC" "C1525"
 			(at 74.8538 125.73 0)
 			(effects
@@
 			)
 		)
+		(property "LCSC" "C4940"
+			(at 186.9186 151.1878 0)
+			(effects
+				(font
+					(size 1.27 1.27)
+				)
+				(hide yes)
+			)
+		)
 		(pin "2"
 		)
@@
 			)
 		)
-		(property "Footprint" "Capacitor_SMD:C_0603_1608Metric"
+		(property "Footprint" "Capacitor_SMD:C_0402_1005Metric"
 			(at 152.4 44.45 0)
 			(effects
@@
 			)
 		)
-		(property "Origin Footprint" "C0603"
+		(property "Origin Footprint" ""
 			(at 152.4 44.45 0)
 			(effects
@@
 			)
 		)
-		(property "LCSC" "C14663"
+		(property "LCSC" "C1525"
 			(at 147.6756 45.974 0)
 			(effects
@@
 			)
 		)
-		(property "Footprint" "Capacitor_SMD:C_0603_1608Metric"
+		(property "Footprint" "Capacitor_SMD:C_0402_1005Metric"
 			(at 146.05 54.61 0)
 			(effects
@@
 			)
 		)
-		(property "Origin Footprint" "C0603"
+		(property "Origin Footprint" ""
 			(at 146.05 54.61 90)
 			(effects
@@
 			)
 		)
-		(property "LCSC" "C14663"
+		(property "LCSC" "C1525"
 			(at 147.2438 52.07 0)
 			(effects
@@
 			)
 		)
-		(property "Footprint" "Capacitor_SMD:C_0603_1608Metric"
+		(property "Footprint" "Capacitor_SMD:C_0402_1005Metric"
 			(at 193.04 59.69 0)
 			(effects
@@
 			)
 		)
-		(property "Origin Footprint" "C0603"
+		(property "Origin Footprint" ""
 			(at 193.04 59.69 90)
 			(effects
@@
 			)
 		)
-		(property "LCSC" "C1681"
+		(property "LCSC" "C107010"
 			(at 194.2338 57.15 0)
 			(effects
@@
 			(effects
 				(font
+					(size 1.27 1.27)
+				)
+				(hide yes)
+			)
+		)
+		(property "LCSC" "C111875"
+			(at 59.69 101.3925 0)
+			(effects
+				(font

Commit message: x1p-002: replace lytic with 4x MLCC
Parts:
- removed C51: 35V 47uF, Capacitor_SMD:CP_Elec_6.3x5.8, symbol Device:C_Polarized_Small
- added C42, C43, C44, C51: GCM32EC71H106KA03L, Capacitor_SMD:C_1210_3225Metric, symbol Device:C_Small
Connections:
- net 24V: now also C42.1, C43.1, C44.1, C51.1
- net GND: now also C42.2, C43.2, C44.2, C51.2
Other:
- note added: "GCM32EC71H106KA03L is 10uF 1210 X7R; spec capacitance 6.4uF at 24V"

Commit message: X1P-002: scrub BOM and remove a stray 0402 0R
Parts:
- C1, C2, C5, C54, C61, C62, C63: Manufacturer SAMSUNG(三星) -> Samsung Electro-Mechanics
- C3: Manufacturer (none) -> Murata Electronics; Manufacturer Part (none) -> GRM21BR6YA106ME43L; Origin Footprint C0603 -> C0805
- C4, C55, C6: value 100nF 35V -> 100nF X7R; Manufacturer (none) -> Samsung Electro-Mechanics; Manufacturer Part (none) -> CL05B104KO5NNNC; Origin Footprint (none) -> C0402
- C42, C43, C44, C51: Manufacturer (none) -> Murata Electronics; Manufacturer Part (none) -> GCM32EC71H106KA03L; Origin Footprint (none) -> C1210
- C47, C50, C52, C57, C58, C60, C8: value 22uF -> 22uF 6.3V; Manufacturer SAMSUNG(三星) -> Samsung Electro-Mechanics
- C49, C59: value 75pF -> 75pF NP0; Manufacturer (none) -> YAGEO; Manufacturer Part (none) -> CC0402JRNPO9BN750; Origin Footprint (none) -> C0402
- C53: value 100nF -> 100nF X7R; Manufacturer (none) -> Samsung Electro-Mechanics; Manufacturer Part (none) -> CL05B104KO5NNNC; Origin Footprint C0603 -> C0402
- C56: Manufacturer (none) -> Samsung Electro-Mechanics; Manufacturer Part (none) -> CL05B104KO5NNNC; Origin Footprint C0603 -> C0402
- C7: Manufacturer (none) -> Samsung Electro-Mechanics; Manufacturer Part (none) -> CL05B104KO5NNNC; Origin Footprint (none) -> C0402
- F1: Manufacturer (none) -> BHFUSE; Manufacturer Part (none) -> BSMD1206-110-30V; Origin Footprint (none) -> F1206
- L1: Origin Footprint L0603 -> 7.2x6.6mm
- L2: Origin Footprint L0603 -> 4.4x4.2mm
- LED1, LED2, LED3: Manufacturer (none) -> Hubei KENTO Elec; Manufacturer Part (none) -> KT-0603R; Origin Footprint (none) -> D0603
- R1, R2, R22, R23, R36, R39, R8: Manufacturer UNI-ROYAL(厚声) -> UNI-ROYAL
- R3: Manufacturer (none) -> UNI-ROYAL; Manufacturer Part (none) -> 0402WGF1372TCE
- R35: Manufacturer (none) -> UNI-ROYAL; Manufacturer Part (none) -> 0402WGF2212TCE
- R37: Manufacturer (none) -> YAGEO; Manufacturer Part (none) -> RC0402FR-076K8L; Origin Footprint (none) -> R0402
- R38: Manufacturer (none) -> UNI-ROYAL; Manufacturer Part (none) -> 0402WGF3401TCE; Origin Footprint (none) -> R0402
- R4: Manufacturer (none) -> YAGEO; Manufacturer Part (none) -> AC0603FR-075K6L; Origin Footprint (none) -> R0603
- R5: Manufacturer UNI-ROYAL(厚声) -> UNI-ROYAL; Origin Footprint (none) -> R0603
- U3, U7: Manufacturer (none) -> Diodes Incorporated; Manufacturer Part (none) -> AP22615AWU-7; Origin Footprint (none) -> TSOT-23-6
- U4, U6: Manufacturer (none) -> Silergy Corp; Manufacturer Part (none) -> SY8205FCC; Origin Footprint (none) -> SOIC-8-EP

Commit message: BOM scrub from mfg feedback
Parts:
- L1: LCSC C5189959 -> C5189749; Manufacturer Part CYA0630-15UH -> CYA0630-6.8UH
Changed lines of the file:
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@@
 			)
 		)
-		(property "Manufacturer Part" "CYA0630-15UH"
+		(property "Manufacturer Part" "CYA0630-6.8UH"
 			(at 165.1 41.91 0)
 			(effects
@@
 			)
 		)
-		(property "LCSC" "C5189959"
+		(property "LCSC" "C5189749"
 			(at 163.7792 38.1254 0)
 			(effects

Commit message: X1P-002: set 5V OCP to 1.8A (fixes #74)
Parts:
- R38: value 3.4k -> 3.74k; LCSC C4940 -> C15172; Manufacturer Part 0402WGF3401TCE -> 0402WGF3741TCE
Other:
- note added: "Iset = 6800 / Rlim 3V3_USER set at 1A 5V_USER set at 1.82A"
- note removed: "Iset = 6800 / Rlim 3V3_USER set at 1A 5V_USER set at 2A"
Changed lines of the file:
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@@
 		)
 	)
-	(text "Iset = 6800 / Rlim\n3V3_USER set at 1A\n5V_USER set at 2A"
+	(text "Iset = 6800 / Rlim\n3V3_USER set at 1A\n5V_USER set at 1.82A"
 		(exclude_from_sim no)
 		(at 234.442 116.84 0)
@@
 			)
 		)
-		(property "Value" "3.4k"
+		(property "Value" "3.74k"
 			(at 186.9186 153.6121 0)
 			(effects
@@
 			)
 		)
-		(property "LCSC" "C4940"
+		(property "LCSC" "C15172"
 			(at 186.9186 151.1878 0)
 			(effects
@@
 			)
 		)
-		(property "Manufacturer Part" "0402WGF3401TCE"
+		(property "Manufacturer Part" "0402WGF3741TCE"
 			(at 185.42 152.4 0)
 			(effects

Commit message: X1P-002: clean up 5V power supply errata (fixes #73)
Parts:
- C47, C50, C8: value 22uF 6.3V -> 22uF 6.3V X7R; footprint Capacitor_SMD:C_0603_1608Metric -> Capacitor_SMD:C_1210_3225Metric; LCSC C59461 -> C55530; Manufacturer Part CL10A226MQ8NRNC -> CL32B226KOJNNNE; Origin Footprint C0603 -> C1210; Supplier Part C59461 -> C55530
- C49: value 75pF NP0 -> 100pF NP0; LCSC C107010 -> C106200; Manufacturer Part CC0402JRNPO9BN750 -> CC0402JRNPO9BN101
- L1: Supplier Part C5189959 -> C5189749
Changed lines of the file:
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@@
 			)
 		)
-		(property "Value" "22uF 6.3V"
+		(property "Value" "22uF 6.3V X7R"
 			(at 176.3141 48.1957 0)
 			(effects
@@
 			)
 		)
-		(property "Footprint" "Capacitor_SMD:C_0603_1608Metric"
+		(property "Footprint" "Capacitor_SMD:C_1210_3225Metric"
 			(at 173.99 46.99 0)
 			(effects
@@
 			)
 		)
-		(property "Manufacturer Part" "CL10A226MQ8NRNC"
+		(property "Manufacturer Part" "CL32B226KOJNNNE"
 			(at 173.99 46.99 90)
 			(effects
@@
 			)
 		)
-		(property "Origin Footprint" "C0603"
+		(property "Origin Footprint" "C1210"
 			(at 173.99 46.99 90)
 			(effects
@@
 			)
 		)
-		(property "Supplier Part" "C59461"
+		(property "Supplier Part" "C55530"
 			(at 173.99 46.99 90)
 			(effects
@@
 			)
 		)
-		(property "LCSC" "C59461"
+		(property "LCSC" "C55530"
 			(at 175.1838 44.45 0)
 			(effects
@@
 			)
 		)
-		(property "Value" "22uF 6.3V"
+		(property "Value" "22uF 6.3V X7R"
 			(at 196.6341 48.1957 0)
 			(effects
@@
 			)
 		)
-		(property "Footprint" "Capacitor_SMD:C_0603_1608Metric"
+		(property "Footprint" "Capacitor_SMD:C_1210_3225Metric"
 			(at 194.31 46.99 0)
 			(effects
@@
 			)
 		)
-		(property "Manufacturer Part" "CL10A226MQ8NRNC"
+		(property "Manufacturer Part" "CL32B226KOJNNNE"
 			(at 194.31 46.99 90)
 			(effects
@@
 			)
 		)
-		(property "Origin Footprint" "C0603"
+		(property "Origin Footprint" "C1210"
 			(at 194.31 46.99 90)
 			(effects
@@
 			)
 		)
-		(property "Supplier Part" "C59461"
+		(property "Supplier Part" "C55530"
 			(at 194.31 46.99 90)
 			(effects
@@
 			)
 		)
-		(property "LCSC" "C59461"
+		(property "LCSC" "C55530"
 			(at 195.5038 44.45 0)
 			(effects
@@
 			)
 		)
-		(property "Value" "75pF NP0"
+		(property "Value" "100pF NP0"
 			(at 195.3641 60.8957 0)
 			(effects
@@
 			)
 		)
-		(property "LCSC" "C107010"
+		(property "LCSC" "C106200"
 			(at 194.2338 57.15 0)
 			(effects
@@
 			)
 		)
-		(property "Manufacturer Part" "CC0402JRNPO9BN750"
+		(property "Manufacturer Part" "CC0402JRNPO9BN101"
 			(at 193.04 59.69 0)
 			(effects
@@
 			)
 		)
-		(property "Value" "22uF 6.3V"
+		(property "Value" "22uF 6.3V X7R"
 			(at 186.4741 48.1957 0)
 			(effects
@@
 			)
 		)
-		(property "Footprint" "Capacitor_SMD:C_0603_1608Metric"
+		(property "Footprint" "Capacitor_SMD:C_1210_3225Metric"
 			(at 184.15 46.99 0)
 			(effects
@@
 			)
 		)
-		(property "Manufacturer Part" "CL10A226MQ8NRNC"
+		(property "Manufacturer Part" "CL32B226KOJNNNE"
 			(at 184.15 46.99 90)
 			(effects
@@
 			)
 		)
-		(property "Origin Footprint" "C0603"
+		(property "Origin Footprint" "C1210"
 			(at 184.15 46.99 90)
 			(effects
@@
 			)
 		)
-		(property "Supplier Part" "C59461"
+		(property "Supplier Part" "C55530"
 			(at 184.15 46.99 90)
 			(effects
@@
 			)
 		)
-		(property "LCSC" "C59461"
+		(property "LCSC" "C55530"
 			(at 185.3438 44.45 0)
 			(effects
@@
 			)
 		)
-		(property "Supplier Part" "C5189959"
+		(property "Supplier Part" "C5189749"
 			(at 165.1 41.91 0)
 			(effects

Commit message: tweak logo positions, tweak testpoint footprints; release x1p-002-c02
Parts:
- TP1, TP2, TP3, TP8: footprint TestPoint:TestPoint_Pad_D1.0mm -> TestPoint:TestPoint_Pad_D1.5mm
Changed lines of the file:
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@@
 	(title_block
 		(title "X1Plus Expansion Board: X1P-002")
-		(rev "X1P-002-B01")
+		(date "2024-12-20")
+		(rev "X1P-002-C02")
 	)
 	(junction
@@
 			)
 		)
-		(property "Footprint" "TestPoint:TestPoint_Pad_D1.0mm"
+		(property "Footprint" "TestPoint:TestPoint_Pad_D1.5mm"
 			(at 52.07 38.1 0)
 			(effects
@@
 			)
 		)
-		(property "Footprint" "TestPoint:TestPoint_Pad_D1.0mm"
+		(property "Footprint" "TestPoint:TestPoint_Pad_D1.5mm"
 			(at 67.31 48.26 0)
 			(effects
@@
 			)
 		)
-		(property "Footprint" "TestPoint:TestPoint_Pad_D1.0mm"
+		(property "Footprint" "TestPoint:TestPoint_Pad_D1.5mm"
 			(at 134.62 114.3 0)
 			(effects
@@
 			)
 		)
-		(property "Description" "5V"
+		(property "Description" "3V3"
 			(at 129.54 114.3 0)
 			(effects
@@
 			)
 		)
-		(property "Footprint" "TestPoint:TestPoint_Pad_D1.0mm"
+		(property "Footprint" "TestPoint:TestPoint_Pad_D1.5mm"
 			(at 207.01 40.64 0)
 			(effects

Commit message: x1p-002: feedforward component and silkscreen changes
Parts:
- C49: value 100pF NP0 -> 470pF NP0; LCSC C106200 -> C526993; Manufacturer Part CC0402JRNPO9BN101 -> CC0402JRNPO7BN471
- C59: value 75pF NP0 -> 220pF NP0; LCSC C107010 -> C107001; Manufacturer Part CC0402JRNPO9BN750 -> CC0402JRNPO9BN221
Changed lines of the file:
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@@
 			)
 		)
-		(property "Value" "75pF NP0"
+		(property "Value" "220pF NP0"
 			(at 122.9741 134.5557 0)
 			(effects
@@
 			)
 		)
-		(property "LCSC" "C107010"
+		(property "LCSC" "C107001"
 			(at 121.8438 130.81 0)
 			(effects
@@
 			)
 		)
-		(property "Manufacturer Part" "CC0402JRNPO9BN750"
+		(property "Manufacturer Part" "CC0402JRNPO9BN221"
 			(at 120.65 133.35 0)
 			(effects
@@
 			)
 		)
-		(property "Value" "100pF NP0"
+		(property "Value" "470pF NP0"
 			(at 195.3641 60.8957 0)
 			(effects
@@
 			)
 		)
-		(property "LCSC" "C106200"
+		(property "LCSC" "C526993"
 			(at 194.2338 57.15 0)
 			(effects
@@
 			)
 		)
-		(property "Manufacturer Part" "CC0402JRNPO9BN101"
+		(property "Manufacturer Part" "CC0402JRNPO7BN471"
 			(at 193.04 59.69 0)
 			(effects
