File: x1p-002/power.kicad_sch (KiCad schematic)
At the start: 54 parts, among them U3 AP22615AWU-7, U4 SY8205FCC, U6 SY8205FCC, U7 AP22615AWU-7

Commit message: x1p-002: bump version
Other:
- title: X1Plus Expansion Board: X1P-002 -> X1Plus Expander: X1P-002
Changed lines of the file:
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@@
 	(paper "USLetter")
 	(title_block
-		(title "X1Plus Expansion Board: X1P-002")
+		(title "X1Plus Expander: X1P-002")
 		(date "2024-12-20")
-		(rev "X1P-002-C02")
+		(rev "X1P-002-C03")
 	)
 	(junction
