File: x1p-002/RP2040.kicad_sch (KiCad schematic)
At the start: 13 parts, among them J1 TC2050-IDC-NL, U2 RP2040, Y1 ABM8-272-T3

Commit message: X1P-002: finish connecting GPIO ports to RP2040
Parts:
- added C31: 1uF, Capacitor_SMD:C_0402_1005Metric, symbol Device:C_Small
- added C35, C36, C37, C38, C39, C40, C41: 100nF, Capacitor_SMD:C_0402_1005Metric, symbol Device:C_Small
Connections:
- net +3V3: now also C31.2, C35.1, C36.1, C37.1, C38.1, C39.1, C40.1, C41.1
- net GND: now also C31.1, C35.2, C36.2, C37.2, C38.2, C39.2, C40.2, C41.2
- net RP2040_DBGRX: now also U2.37 (GPIO25)
- net RP2040_DBGTX: now also U2.36 (GPIO24)
- net PORTB3: now reaches U2.11 (GPIO8)
- net PORTB2: now reaches U2.12 (GPIO9)
- net PORTB1: now reaches U2.13 (GPIO10)
- net PORTB0: now reaches U2.14 (GPIO11)
- net PORTC7: now reaches U2.15 (GPIO12)
- net PORTC6: now reaches U2.16 (GPIO13)
- net PORTC3: now reaches U2.17 (GPIO14)
- net PORTC2: now reaches U2.18 (GPIO15)
- net PORTA7: now reaches U2.2 (GPIO0)
- net PORTC1: now reaches U2.27 (GPIO16)
- net PORTC0: now reaches U2.28 (GPIO17)
- net PORTD7: now reaches U2.29 (GPIO18)
- net PORTA6: now reaches U2.3 (GPIO1)
- net PORTD6: now reaches U2.30 (GPIO19)
- net PORTD3: now reaches U2.31 (GPIO20)
- net PORTD2: now reaches U2.32 (GPIO21)
- net PORTD1: now reaches U2.34 (GPIO22)
- net PORTD0: now reaches U2.35 (GPIO23)
- net PORTA4: now reaches U2.38 (GPIO26_ADC0)
- net PORTB4: now reaches U2.39 (GPIO27_ADC1)
- net PORTA3: now reaches U2.4 (GPIO2)
- net PORTC4: now reaches U2.40 (GPIO28_ADC2)
- net PORTD4: now reaches U2.41 (GPIO29_ADC3)
- net PORTA2: now reaches U2.5 (GPIO3)
- net PORTD5: now reaches U2.51 (QSPI_SD3)
- net PORTA5: now reaches U2.53 (QSPI_SD0)
- net PORTC5: now reaches U2.54 (QSPI_SD2)
- net PORTB5: now reaches U2.55 (QSPI_SD1)
- net PORTA1: now reaches U2.6 (GPIO4)
- net PORTA0: now reaches U2.7 (GPIO5)
- net PORTB7: now reaches U2.8 (GPIO6)
- net PORTB6: now reaches U2.9 (GPIO7)
- no-connect marks 0 -> 4
Other:
- note added: "Place C31 at U2.44"
- note added: "Port functionality: D0: SIO / PIO D1: SIO / PIO D2: SIO / PIO D3: SIO / PIO D4: SIO / PIO / ADC D5: SIO D6: SIO / PIO D7: SIO / PIO"
- note added: "RP2040 debug UART on TC2050 hdr is UART1"
- note removed: "TODO: decaps for 3v3"
- moved on the sheet: C20, C30, C32, C33, C34, J1, R14, R15, R16, R17, R24, U2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

Commit message: x1p-002: layout rp2040 and new buck converters
Parts:
- C20, C30: LCSC (none) -> C1548
- R14, R17: LCSC (none) -> C274349
- R15, R16, R24: LCSC (none) -> C11702
- U2: LCSC (none) -> C2040
- Y1: footprint (none) -> Crystal:Crystal_SMD_3225-4Pin_3.2x2.5mm; LCSC (none) -> C20625731
Connections:
- net PORTA4: now also U2.41 (GPIO29_ADC3); no longer U2.38 (GPIO26_ADC0)
- net PORTA5: now also U2.55 (QSPI_SD1); no longer U2.53 (QSPI_SD0)
- net PORTB4: now also U2.40 (GPIO28_ADC2); no longer U2.39 (GPIO27_ADC1)
- net PORTB5: now also U2.54 (QSPI_SD2); no longer U2.55 (QSPI_SD1)
- net PORTC4: now also U2.39 (GPIO27_ADC1); no longer U2.40 (GPIO28_ADC2)
- net PORTC5: now also U2.53 (QSPI_SD0); no longer U2.54 (QSPI_SD2)
- net PORTD4: now also U2.38 (GPIO26_ADC0); no longer U2.41 (GPIO29_ADC3)
- net RP2040_DBGRX: now also J1.8 (Pin_8); no longer J1.7 (Pin_7)
- net RP2040_DBGTX: now also J1.9 (Pin_9); no longer J1.6 (Pin_6)
- net RP2040_SWCLK: now also J1.3 (Pin_3); no longer J1.2 (Pin_2)
- net RP2040_SWDIO: now also J1.2 (Pin_2); no longer J1.3 (Pin_3)
- net RP_INT_DN: now reaches R14.1, U2.46 (USB_DM)
- net RP_INT_DP: now reaches R17.2, U2.47 (USB_DP)
- net +1V1_RP2040 renamed 1V1_RP2040
- net +3V3 renamed 3V3
- no-connect marks 4 -> 2
Other:
- moved on the sheet: R14, R17

Commit message: X1P-002: scrub BOM and remove a stray 0402 0R
Parts:
- C20, C30: value 15p -> 15pF; Manufacturer (none) -> Guangdong Fenghua Advanced Tech; Manufacturer Part (none) -> 0402CG150J500NT; Origin Footprint (none) -> C0402
- C31, C32: Manufacturer SAMSUNG(三星) -> Samsung Electro-Mechanics
- C33, C34, C35, C36, C37, C38, C39, C40, C41: value 100nF -> 100nF X7R; Manufacturer SAMSUNG(三星) -> Samsung Electro-Mechanics
- R14, R17: Manufacturer (none) -> YAGEO; Manufacturer Part (none) -> RC0402FR-0727R4L; Origin Footprint (none) -> R0402
- R15, R16, R24: Manufacturer (none) -> UNI-ROYAL; Manufacturer Part (none) -> 0402WGF1001TCE; Origin Footprint (none) -> R0402
- U2: Manufacturer (none) -> Raspberry Pi; Manufacturer Part (none) -> RP2040; Origin Footprint (none) -> LQFN-56
- Y1: Manufacturer (none) -> Abracon LLC; Manufacturer Part (none) -> ABM8-272-T3; Origin Footprint (none) -> SMD3225-4P

Commit message: tweak logo positions, tweak testpoint footprints; release x1p-002-c02
Connections:
- no-connect marks 2 -> 4
Changed lines of the file:
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@@
 	(title_block
 		(title "X1Plus Expansion Board: X1P-002")
-		(rev "X1P-002-B01")
+		(date "2024-12-20")
+		(rev "X1P-002-C02")
 	)
 	(junction
@@
 	)
 	(no_connect
+		(at 228.6 121.92)
+	)
+	(no_connect
 		(at 77.47 111.76)
 	)
@@
 		(at 215.9 119.38)
 	)
+	(no_connect
+		(at 228.6 119.38)
+	)
 	(wire
