File: x1p-004/x1p-004.kicad_pcb (KiCad board)
At the start: 2 copper layers, 21 x 28 mm, 10 parts, among them U1 AD24C02, U2 TXS0102DCUR, U3 PM254-2-08-W-8.5, U4 2060-452/998-404, U5 2060-452/998-404

Commit message: unidirectional shifters, decouple eeprom, add jumper for sourcing 5v
Parts:
- added C2: 0.1uf, lcsc:C0402, B.Cu at (73.3, 115.6)
- added HDR1: PM254-2-08-W-8.5, lcsc:HDR-TH_16P-P2.54-H-F-R2-C8-W8.5, F.Cu at (68.4, 122.6)
- added JP1: SolderJumper_2_Open, Jumper:SolderJumper-2_P1.3mm_Open_RoundedPad1.0x1.5mm, B.Cu at (68.5, 106.7)
- added R3: 0, lcsc:R0603, B.Cu at (67.3, 115.8)
- U2: value TXS0102DCUR -> SN74LVC1T45DBVR; footprint lcsc:VSON8_L2.0-W2.3-P0.50-LS3.1-BL -> lcsc:SOT-23-6_L2.9-W1.6-P0.95-LS2.8-BR
- U3: value PM254-2-08-W-8.5 -> SN74LVC1T45DBVR; footprint lcsc:HDR-TH_16P-P2.54-H-F-R2-C8-W8.5 -> lcsc:SOT-23-6_L2.9-W1.6-P0.95-LS2.8-BR; moved to B.Cu
- moved U3 6.63 mm to (64.7, 117.2), turned to -90 degrees
- moved U2 1.88 mm to (60.5, 117.2)
Connections:
- C1 pad 1: 5V -> EXT_5V
- D1 pad 1: 5V -> EXT_5V
- F1 pad 1: 5V -> EXT_5V
- U2 pad 1: HD1 -> 3V3
- U2 pad 3: 3V3 -> LD0
- U2 pad 4: LD1 -> HD0
- U2 pad 5: LD0 -> 3V3
- U2 pad 6: GND -> EXT_5V
- U3 pad 1: GND -> 3V3
- U3 pad 2: LD0 -> GND
- U3 pad 3: GND -> LD1
- U3 pad 4: LD1 -> HD1
- U3 pad 6: unconnected-(U3-Pad6) -> EXT_5V
Routing:
- net EXT_5V: track 0.00 -> 25.6 mm
- net 5V: track 32.1 -> 10.3 mm
- net 3V3: track 33.9 -> 45.5 mm
- net Net-(JP1-B): track 0.00 -> 8.51 mm
- net GND: track 27.3 -> 20.4 mm, vias 5 -> 10
- net Net-(JP1-A): track 14.1 -> 19.9 mm, vias 1 -> 2
- net HD1: track 17.8 -> 16.5 mm
- net LD1: track 4.07 -> 3.54 mm
Other:
- board text added: "D0 CLK"
- board text added: "D1 DAT"
- board text removed: "D0 SDA"
- board text removed: "D1 SCL"

Commit message: changes round 2
Parts:
- removed JP1: SolderJumper_2_Open, Jumper:SolderJumper-2_P1.3mm_Open_RoundedPad1.0x1.5mm
- removed U5: 2060-452/998-404, lcsc:CONN-SMD_2060-452
- added D2: SRV05-4.TCT_C2687126, x1p-004:SOT-23-6_L2.9-W1.6-P0.95-LS2.8-BL, B.Cu at (62.5, 107.0)
- added EXT_POWER1: 2060-452/998-404, x1p-004:CONN-SMD_2060-452, F.Cu at (74.2, 107.0)
- added LED1: 2060-452/998-404, x1p-004:CONN-SMD_2060-452, F.Cu at (62.6, 107.0)
- added Q1: BC857BS,115, x1p-004:SOT-363_L2.0-W1.3-P0.65-LS2.1-TL, B.Cu at (71.4, 105.1)
- added R4: 68k, x1p-004:R0402, B.Cu at (69.0, 104.4)
- added SW1: DSIC01THGET, x1p-004:SW-TH_DSIC01THGET, F.Cu at (68.4, 110.2)
- C1: footprint lcsc:C0603 -> x1p-004:C0603
- C2: footprint lcsc:C0402 -> x1p-004:C0402
- D1: value 5.1V -> 6.2V; footprint lcsc:SOD-123_L2.8-W1.8-LS3.7-RD -> x1p-004:SOD-123_L2.8-W1.8-LS3.7-RD
- F1: footprint lcsc:F0805 -> x1p-004:F0805
- HDR1: footprint lcsc:HDR-TH_16P-P2.54-H-F-R2-C8-W8.5 -> x1p-004:HDR-TH_16P-P2.54-H-F-R2-C8-W8.5
- R1, R2: footprint lcsc:R0402 -> x1p-004:R0402
- R3: value 0 -> 100k; footprint lcsc:R0603 -> x1p-004:R0402
- U1: footprint lcsc:SOT-23-5_L2.9-W1.6-P0.95-LS2.8-BL -> x1p-004:SOT-23-5_L2.9-W1.6-P0.95-LS2.8-BL
- U2, U3: footprint lcsc:SOT-23-6_L2.9-W1.6-P0.95-LS2.8-BR -> x1p-004:SOT-23-6_L2.9-W1.6-P0.95-LS2.8-BR
- U4: value 2060-452/998-404 -> SI2301-ZE; footprint lcsc:CONN-SMD_2060-452 -> x1p-004:SOT-23-3_L2.9-W1.3-P1.90-LS2.4-BR; moved to B.Cu
- moved R3 12.6 mm to (73.8, 105.0)
- moved U4 8.74 mm to (71.4, 108.0), turned to 0 degrees
- moved C1 1.17 mm to (70.9, 118.0)
- moved D1 0.30 mm to (70.4, 112.2)
Connections:
- C1 pad 1: EXT_5V -> 5V_INT
- D1 pad 1: EXT_5V -> 5V_INT
- F1 pad 1: EXT_5V -> 5V_INT
- R3 pad 1: Net-(JP1-B) -> GND
- R3 pad 2: 5V -> Net-(U4-G)
- U2 pad 6: EXT_5V -> 5V_INT
- U3 pad 6: EXT_5V -> 5V_INT
- U4 pad 1: HD1 -> Net-(U4-G)
- U4 pad 2: HD0 -> 5V_INT
Routing:
- net GND: track 20.4 -> 48.3 mm
- net EXT_5V: track 25.6 -> 0.00 mm
- net Net-(JP1-B): track 8.51 -> 0.00 mm
- net HD1: track 16.5 -> 24.4 mm
- net HD0: track 19.9 -> 26.1 mm
- net Net-(EXT_POWER1-Pad1): track 19.9 -> 14.1 mm, vias 2 -> 1
- net 5V_INT: track 0.00 -> 3.64 mm, vias 0 -> 2
- net Net-(Q1-Pad2): track 0.00 -> 3.57 mm
- net Net-(U4-G): track 0.00 -> 2.94 mm
- net 5V: track 10.3 -> 12.4 mm
- added copper zone on B.Cu, net 5V_INT
- removed copper zone on B.Cu, net GND
Other:
- board text added: "Switch enables Internal 5V !! 500mA Limit !!"

Commit message: reorient switch, update text
Parts:
- moved SW1 2.40 mm to (68.4, 107.8), turned to 0 degrees
- moved Q1 2.01 mm to (73.4, 105.3)
- moved R3 2.01 mm to (75.8, 105.2)
- moved R4 2.01 mm to (71.0, 104.6)
- moved F1 1.91 mm to (75.9, 110.8), turned to 180 degrees
- moved D1 1.90 mm to (71.0, 114.0)
- moved U4 1.81 mm to (73.2, 108.2)
Connections:
- EXT_POWER1 pad 1: Net-(EXT_POWER1-Pad1) -> GND
- EXT_POWER1 pad 2: GND -> Net-(EXT_POWER1-Pad2)
- F1 pad 2: Net-(EXT_POWER1-Pad1) -> Net-(EXT_POWER1-Pad2)
- SW1 pad 1: 5V -> GND
- SW1 pad 2: GND -> 5V
Routing:
- net Net-(EXT_POWER1-Pad1): track 14.1 -> 0.00 mm, vias 1 -> 0
- net Net-(EXT_POWER1-Pad2): track 0.00 -> 13.4 mm, vias 0 -> 1
- net GND: track 48.3 -> 56.9 mm
- net 5V: track 12.4 -> 15.8 mm
- net HD1: track 24.4 -> 23.7 mm
Other:
- board size 21 x 28 mm -> 20.8 x 28 mm
- board text added: "CLK"
- board text added: "DAT"
- board text added: "Internal 5V enable 500mA limit: see manual!"
- board text added: "X1Plus 5V LED Level Shifter"
- board text removed: "D0 CLK"
- board text removed: "D1 DAT"
- board text removed: "Switch enables Internal 5V !! 500mA Limit !!"
