File: x1p-004/x1p-004.kicad_pcb (KiCad board)
At the start: 2 copper layers, 20.8 x 28 mm, 18 parts, among them Q1 BC857BS,115, SW1 DSIC01THGET, U1 AD24C02, U2 SN74LVC1T45DBVR, U3 SN74LVC1T45DBVR, U4 SI2301-ZE

Commit message: x1p-004 layout: swap 5V and GND labels, improve chomnkiness of 5V and GND traces
Routing:
- net Net-(EXT_POWER1-Pad2): track 13.4 -> 17.3 mm, vias 1 -> 2
Changed lines of the file:
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@@
 	)
 	(gr_text "5V"
-		(at 75.4 115 0)
+		(at 72.2 115 0)
 		(layer "F.SilkS")
 		(effects
@@
 				(thickness 0.1)
 			)
-			(justify left bottom)
+			(justify bottom)
 		)
 	)
 	(gr_text "GND"
-		(at 71 115 0)
+		(at 76.2 115 0)
 		(layer "F.SilkS")
 		(effects
@@
 				(thickness 0.1)
 			)
-			(justify left bottom)
+			(justify bottom)
 		)
 	)
@@
 	)
 	(segment
-		(start 74.9 109.6)
-		(end 74.9 102.5)
-		(width 0.4)
-		(layer "F.Cu")
-		(net 2)
-	)
-	(segment
-		(start 74.9 102.5)
-		(end 76.2 101.2)
-		(width 0.4)
-		(layer "F.Cu")
-		(net 2)
-	)
-	(segment
-		(start 76.2 110.9)
-		(end 74.9 109.6)
-		(width 0.4)
+		(start 77.4 110.7)
+		(end 76.2 111.9)
+		(width 0.8)
+		(layer "F.Cu")
+		(net 2)
+	)
+	(segment
+		(start 77.4 103.4)
+		(end 77.4 110.7)
+		(width 0.8)
+		(layer "F.Cu")
+		(net 2)
+	)
+	(segment
+		(start 76.2 102.2)
+		(end 77.4 103.4)
+		(width 0.8)
 		(layer "F.Cu")
 		(net 2)
@@
 		(start 62.55 105.8)
 		(end 62.55 104)
-		(width 0.2)
+		(width 0.8)
 		(layer "B.Cu")
 		(net 2)
@@
 		(start 62.55 104)
 		(end 62.55 102.65)
-		(width 0.2)
+		(width 0.8)
 		(layer "B.Cu")
 		(net 2)
@@
 		(start 68.4 103.98)
 		(end 62.57 103.98)
-		(width 0.2)
+		(width 0.8)
 		(layer "B.Cu")
 		(net 2)
@@
 	)
 	(segment
-		(start 73.8 110.4)
-		(end 73.6 110.6)
-		(width 0.2)
+		(start 73.6 110.8)
+		(end 73.6 111.4)
+		(width 0.8)
+		(layer "F.Cu")
+		(net 17)
+	)
+	(segment
+		(start 72.3 112)
+		(end 72.2 111.9)
+		(width 0.8)
+		(layer "F.Cu")
+		(net 17)
+	)
+	(segment
+		(start 72.2 102.272793)
+		(end 73.4 103.472793)
+		(width 0.8)
+		(layer "F.Cu")
+		(net 17)
+	)
+	(segment
+		(start 73.6 111.4)
+		(end 73.6 112)
+		(width 0.8)
 		(layer "F.Cu")
 		(net 17)
@@
 	)
 	(segment
-		(start 73.2 102.2)
-		(end 73.8 102.8)
-		(width 0.2)
-		(layer "F.Cu")
-		(net 17)
-	)
-	(segment
-		(start 73.5 110.6)
+		(start 73.6 111.4)
+		(end 72.7 111.4)
+		(width 0.8)
+		(layer "F.Cu")
+		(net 17)
+	)
+	(segment
+		(start 73.6 112)
+		(end 72.3 112)
+		(width 0.8)
+		(layer "F.Cu")
+		(net 17)
+	)
+	(segment
+		(start 73.4 103.472793)
+		(end 73.4 110.5)
+		(width 0.8)
+		(layer "F.Cu")
+		(net 17)
+	)
+	(segment
+		(start 72.7 111.4)
 		(end 72.2 111.9)
-		(width 0.2)
-		(layer "F.Cu")
-		(net 17)
-	)
-	(segment
-		(start 73.6 110.6)
-		(end 73.5 110.6)
-		(width 0.2)
-		(layer "F.Cu")
-		(net 17)
-	)
-	(segment
-		(start 73.8 102.8)
-		(end 73.8 110.4)
-		(width 0.2)
+		(width 0.8)
 		(layer "F.Cu")
 		(net 17)
@@
 	(segment
 		(start 72.2 102.2)
-		(end 73.2 102.2)
-		(width 0.2)
-		(layer "F.Cu")
-		(net 17)
-	)
-	(segment
-		(start 73.6 110.5)
-		(end 73.6 110.5)
-		(width 0.2)
-		(layer "F.Cu")
-		(net 17)
-	)
-	(via
-		(at 73.6 110.6)
-		(size 0.6)
-		(drill 0.3)
-		(layers "F.Cu" "B.Cu")
-		(net 17)
-	)
-	(segment
-		(start 73.6 110.6)
-		(end 74.6 110.6)
-		(width 0.2)
-		(layer "B.Cu")
-		(net 17)
-	)
-	(segment
-		(start 74.6 110.6)
+		(end 72.2 102.272793)
+		(width 0.8)
+		(layer "F.Cu")
+		(net 17)
+	)
+	(via
+		(at 73.6 110.8)
+		(size 0.6)
+		(drill 0.3)
+		(layers "F.Cu" "B.Cu")
+		(net 17)
+	)
+	(via
+		(at 73.6 112)
+		(size 0.6)
+		(drill 0.3)
+		(layers "F.Cu" "B.Cu")
+		(net 17)
+	)
+	(segment
+		(start 73.6 111.2)
+		(end 74.4 111.2)
+		(width 0.8)
+		(layer "B.Cu")
+		(net 17)
+	)
+	(segment
+		(start 73.6 110.8)
+		(end 73.6 111.2)
+		(width 0.8)
+		(layer "B.Cu")
+		(net 17)
+	)
+	(segment
+		(start 74.4 111.2)
 		(end 74.8 110.8)
-		(width 0.2)
-		(layer "B.Cu")
-		(net 17)
+		(width 0.8)
+		(layer "B.Cu")
+		(net 17)
+	)
+	(segment
+		(start 74.8 110.8)
+		(end 73.6 110.8)
+		(width 0.8)
+		(layer "B.Cu")
+		(net 17)
+	)
+	(segment
+		(start 73.6 111.2)
+		(end 73.6 112)
+		(width 0.8)
+		(layer "B.Cu")
+		(net 17)

Commit message: x1p-004 layout: optimize some, and match schematic
Parts:
- added R5: 3.3k, x1p-004:R0402, B.Cu at (60.0, 119.4)
- added R6: 3.3k, x1p-004:R0402, B.Cu at (64.2, 119.4)
- moved U2 0.50 mm to (60.5, 116.7)
- moved U3 0.50 mm to (64.7, 116.7)
Connections:
- Q1 pad 1: GND -> /5V_SW
- SW1 pad 1: GND -> /5V_SW
- U4 pad 3: GND -> /5V_SW
Routing:
- net /5V_SW: track 0.00 -> 13.9 mm
- net GND: track 56.8 -> 50.9 mm, vias 10 -> 8
- net 5V_INT: track 3.64 -> 0.01 mm, vias 2 -> 0
- net LD1: track 3.54 -> 4.23 mm
- net LD0: track 2.89 -> 3.51 mm
- net HD0: track 26.2 -> 25.7 mm
- net HD1: track 23.7 -> 23.3 mm, vias 1 -> 3

Commit message: x1p-004: add decap for level shifters
Parts:
- added C3: 0.1uf, x1p-004:C0402, B.Cu at (62.9, 116.8)
- moved R6 0.65 mm to (64.8, 119.4)
- moved U3 0.57 mm to (65.2, 116.7)
Routing:
- net GND: track 50.9 -> 58.3 mm
- net 3V3: track 45.3 -> 46.7 mm
- net HD1: track 23.3 -> 24.7 mm
- net LD1: track 4.23 -> 5.07 mm

Commit message: x1p-004 layout: thermals are good enough for ground, do not override those
Routing:
- net GND: track 58.3 -> 47.8 mm
Changed lines of the file:
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@@
 		(net 1)
 	)
-	(segment
-		(start 77.4 110.7)
-		(end 76.2 111.9)
-		(width 0.8)
-		(layer "F.Cu")
-		(net 2)
-	)
-	(segment
-		(start 77.4 103.4)
-		(end 77.4 105.6)
-		(width 0.8)
-		(layer "F.Cu")
-		(net 2)
-	)
-	(segment
-		(start 77.4 105.6)
-		(end 77.4 110.7)
-		(width 0.8)
-		(layer "F.Cu")
-		(net 2)
-	)
-	(segment
-		(start 76.2 102.2)
-		(end 77.4 103.4)
-		(width 0.8)
-		(layer "F.Cu")
-		(net 2)
-	)
-	(via
-		(at 77.4 105.6)
+	(via
+		(at 76.8 106.3)
 		(size 0.6)
 		(drill 0.3)
@@
 	)
 	(segment
+		(start 76.8 106.3)
+		(end 76.8 105.445)
+		(width 0.2)
+		(layer "B.Cu")
+		(net 2)
+	)
+	(segment
 		(start 60.57 122.85)
 		(end 60.57 119.57)
@@
 	)
 	(segment
+		(start 76.095 104.74)
+		(end 75.8 104.74)
+		(width 0.2)
+		(layer "B.Cu")
+		(net 2)
+	)
+	(segment
 		(start 62.75 117.35)
 		(end 62.95 117.15)
@@
 	)
 	(segment
+		(start 76.8 105.445)
+		(end 76.095 104.74)
+		(width 0.2)
+		(layer "B.Cu")
+		(net 2)
+	)
+	(segment
 		(start 65.05 119.57)
 		(end 65.05 119.4)
@@
 	)
 	(segment
-		(start 75.8 104.74)
-		(end 76.54 104.74)
-		(width 0.2)
-		(layer "B.Cu")
-		(net 2)
-	)
-	(segment
 		(start 65.15 120)
 		(end 65.28 119.87)
@@
 		(width 0.2)
 		(layer "B.Cu")
-		(net 2)
-	)
-	(segment
-		(start 76.54 104.74)
-		(end 77.4 105.6)
-		(width 0.2)
-		(layer "B.Cu")

Commit message: x1p-004: B01 pseudofinal
Parts:
- removed EXT_POWER1, LED1: 2060-452/998-404, x1p-004:CONN-SMD_2060-452
- removed R5: 3.3k, x1p-004:R0402
- added CN1: HC-PH-3AWT, x1p-004:CONN-SMD_3P-P2.0-HC-PH-3AWT, F.Cu at (61.5, 89.5)
- added H1: MountingHole, MountingHole:MountingHole_2.2mm_M2, F.Cu at (68.5, 117.8)
- added H2: MountingHole, MountingHole:MountingHole_2.2mm_M2, F.Cu at (68.5, 106.0)
- C1, C2, C3, D1, D2, F1, Q1, R1, R2, R3, R4, R6, U1, U3, U4: moved to F.Cu
- HDR1: value PM254-2-08-W-8.5 -> 220R-2*10P H=8.5MM Ytype Gold-plated black; footprint x1p-004:HDR-TH_16P-P2.54-H-F-R2-C8-W8.5 -> x1p-004:HDR-TH_20P-P2.54-H-F-R2-C10-S2.54-W10.2
- U2: value SN74LVC1T45DBVR -> 2060-453/998-404; footprint x1p-004:SOT-23-6_L2.9-W1.6-P0.95-LS2.8-BR -> x1p-004:CONN-SMD_2060-453; moved to F.Cu
- moved U2 27.9 mm to (74.5, 92.5)
- moved D2 15.2 mm to (77.5, 109.8), turned to 90 degrees
- moved SW1 10.2 mm to (58.8, 104.5)
- moved R3 9.40 mm to (71.0, 113.2), turned to 90 degrees
- moved R4 8.74 mm to (69.8, 113.2), turned to 90 degrees
- moved C1 8.59 mm to (65.0, 111.8), turned to -90 degrees
- moved R1 7.93 mm to (78.0, 112.2), turned to 0 degrees
- moved Q1 6.01 mm to (69.8, 110.0), turned to 90 degrees
- moved U3 5.39 mm to (61.5, 112.8)
- moved C3 5.30 mm to (58.8, 113.5), turned to 90 degrees
- moved R2 5.19 mm to (78.0, 114.2)
- moved R6 5.16 mm to (64.5, 114.2)
- moved F1 4.66 mm to (73.2, 107.0)
- moved D1 4.27 mm to (67.0, 112.5), turned to -90 degrees
- moved U1 3.53 mm to (75.2, 113.2), turned to 90 degrees
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Connections:
- D2 pad 1: HD0 -> unconnected-(D2-Pad1)
- D2 pad 6: HD0 -> unconnected-(D2-Pad6)
- F1 pad 2: Net-(EXT_POWER1-Pad2) -> Net-(CN1-Pad2)
- HDR1 pad 1: GND -> unconnected-(HDR1-Pad1)
- HDR1 pad 10: unconnected-(HDR1-Pad10) -> 5V
- HDR1 pad 11: 3V3 -> unconnected-(HDR1-Pad11)
- HDR1 pad 12: unconnected-(HDR1-Pad12) -> 5V
- HDR1 pad 13: GND -> unconnected-(HDR1-Pad13)
- HDR1 pad 14: LD6 -> 3V3
- HDR1 pad 15: GND -> LD6
- HDR1 pad 16: LD7 -> GND
- HDR1 pad 2: LD0 -> unconnected-(HDR1-Pad2)
- HDR1 pad 3: GND -> unconnected-(HDR1-Pad3)
- HDR1 pad 4: LD1 -> GND
- HDR1 pad 5: 3V3 -> LD1
- HDR1 pad 6: unconnected-(HDR1-Pad6) -> GND
- HDR1 pad 7: 5V -> unconnected-(HDR1-Pad7)
- HDR1 pad 8: unconnected-(HDR1-Pad8) -> 3V3
- HDR1 pad 9: 5V -> unconnected-(HDR1-Pad9)
- U2 pad 1: 3V3 -> HD1
- U2 pad 2: GND -> Net-(CN1-Pad2)
- U2 pad 3: LD0 -> GND
Routing:
- net Net-(CN1-Pad2): track 0.00 -> 39.6 mm
- net 3V3: track 46.7 -> 9.08 mm, vias 0 -> 3
- net HD1: track 24.7 -> 57.2 mm, vias 3 -> 4
- net GND: track 47.8 -> 17.0 mm, vias 8 -> 2
- net HD0: track 25.7 -> 0.00 mm, vias 1 -> 0
- net 5V_INT: track 0.01 -> 21.8 mm
- net Net-(EXT_POWER1-Pad2): track 17.3 -> 0.00 mm, vias 2 -> 0
- net 5V: track 15.8 -> 0.85 mm
- net LD6: track 3.67 -> 11.9 mm, vias 0 -> 1
- net LD7: track 3.73 -> 10.9 mm, vias 0 -> 1
- net /5V_SW: track 13.9 -> 21.0 mm, vias 0 -> 3
- net LD1: track 5.07 -> 9.20 mm
- net LD0: track 3.51 -> 0.00 mm
- net Net-(U4-G): track 2.45 -> 5.51 mm
- net Net-(Q1-Pad2): track 3.57 -> 4.39 mm
- added copper zone on B.Cu, net 3V3
- added copper zone on B.Cu, net 5V
Other:
- board size 20.8 x 28 mm -> 26.4 x 42.5 mm
- board text added: "PH 2.0mm (NeoPixel et al)"
- board text added: "X1P-004-B01"
- board text added: "X1Plus Addressable-LED Level Shifter"
- board text removed: "CLK"
- board text removed: "X1P-004-A01"
- board text removed: "X1Plus 5V LED Level Shifter"

Commit message: x1p-005: fix up board layout to align with x1p-004
Parts:
- moved H1 84.6 mm to (150.0, 95.0)
- moved C1 84.5 mm to (146.5, 89.2)
- moved C2 84.5 mm to (154.2, 90.8)
- moved C3 84.5 mm to (140.2, 91.0)
- moved CN1 84.5 mm to (143.0, 67.0)
- moved D1 84.5 mm to (148.5, 90.0)
- moved D2 84.5 mm to (159.0, 87.2)
- moved F1 84.5 mm to (154.8, 84.5)
- moved HDR1 84.5 mm to (150.0, 100.0)
- moved Q1 84.5 mm to (151.2, 87.5)
- moved R1 84.5 mm to (159.5, 89.8)
- moved R2 84.5 mm to (159.5, 91.8)
- moved R3 84.5 mm to (152.5, 90.8)
- moved R4 84.5 mm to (151.2, 90.8)
- moved R6 84.5 mm to (146.0, 91.8)
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
Commit message: X1P-004: homogenize footprints
Parts:
- C1: footprint x1p-004:C0603 -> Capacitor_SMD:C_0603_1608Metric
- C2, C3: footprint x1p-004:C0402 -> Capacitor_SMD:C_0402_1005Metric
- R1, R2, R3, R4, R6: footprint x1p-004:R0402 -> Resistor_SMD:R_0402_1005Metric

Commit message: reduce overall BOM on panels, load manufacturer and MPN in
Parts:
- C2, C3: value 0.1uf -> 0.1uF
- F1: value 500ma -> BSMD0805-050-15V
- HDR1: value 220R-2*10P H=8.5MM Ytype Gold-plated black -> B-2200R20P-B120
- R1, R2, R6: value 3.3k -> 2.2k
