File: x1p-004/x1p-004.kicad_sch (KiCad schematic)
At the start: 10 parts, among them U1 AD24C02, U2 TXS0102DCUR, U3 PM254-2-08-W-8.5, U4 2060-452/998-404, U5 2060-452/998-404

Commit message: unidirectional shifters, decouple eeprom, add jumper for sourcing 5v
Parts:
- removed U2: TXS0102DCUR, lcsc:VSON8_L2.0-W2.3-P0.50-LS3.1-BL, symbol lcsc:TXS0102DCUR
- added C2: 0.1uf, lcsc:C0402, symbol lcsc:CL05B104KO5NNNC
- added JP1: SolderJumper_2_Open, Jumper:SolderJumper-2_P1.3mm_Open_RoundedPad1.0x1.5mm, symbol Jumper:SolderJumper_2_Open
- added R3: 0, lcsc:R0603, symbol lcsc:0603WAF0000T5E
- added U2, U3: SN74LVC1T45DBVR, lcsc:SOT-23-6_L2.9-W1.6-P0.95-LS2.8-BR, symbol lcsc:SN74LVC1T45DBVR
- renumbered U3 to HDR1
Connections:
- net 3V3: now also C2.1, U2.1 (VCCA), U2.5 (DIR), U3.1 (VCCA), U3.5 (DIR)
- net 5V: now also HDR1.7, HDR1.9, R3.2; no longer C1.1, D1.1 (K), F1.1
- net GND: now also C2.2, U2.2 (GND), U3.2 (GND)
- net HD0: now also U2.4 (B)
- net HD1: now also U3.4 (B)
- net LD0: now also U2.3 (A)
- net LD1: now also U3.3 (A)
- net at F1.2, U5.1: now also JP1.1 (A)
- new net: JP1.2 (B), R3.1
- new net EXT_5V: C1.1, D1.1 (K), F1.1, U2.6 (VCCB), U3.6 (VCCB)
- no-connect marks 6 -> 4
Other:
- moved on the sheet: C1, D1, F1, U4, U5

Commit message: changes round 2
Parts:
- removed D1: 5.1V, lcsc:SOD-123_L2.8-W1.8-LS3.7-RD, symbol lcsc:MMSZ5231B-7-F
- removed JP1: SolderJumper_2_Open, Jumper:SolderJumper-2_P1.3mm_Open_RoundedPad1.0x1.5mm, symbol Jumper:SolderJumper_2_Open
- removed R3: 0, lcsc:R0603, symbol lcsc:0603WAF0000T5E
- removed U5: 2060-452/998-404, lcsc:CONN-SMD_2060-452, symbol lcsc:2060-452_998-404
- added D1: 6.2V, x1p-004:SOD-123_L2.8-W1.8-LS3.7-RD, symbol x1p-004:MMSZ5234BT1G
- added D2: SRV05-4.TCT_C2687126, x1p-004:SOT-23-6_L2.9-W1.6-P0.95-LS2.8-BL, symbol x1p-004:SRV05-4.TCT_C2687126
- added EXT_POWER1: 2060-452/998-404, x1p-004:CONN-SMD_2060-452, symbol lcsc:2060-452_998-404
- added Q1: BC857BS,115, x1p-004:SOT-363_L2.0-W1.3-P0.65-LS2.1-TL, symbol lcsc:BC857BS,115
- added R3: 100k, x1p-004:R0402, symbol lcsc:0402WGF1003TCE
- added R4: 68k, x1p-004:R0402, symbol lcsc:0402WGF6802TCE
- added SW1: DSIC01THGET, x1p-004:SW-TH_DSIC01THGET, symbol x1p-004:DSIC01THGET
- added U4: SI2301-ZE, x1p-004:SOT-23-3_L2.9-W1.3-P1.90-LS2.4-BR, symbol lcsc:SI2301-ZE
- C1: footprint lcsc:C0603 -> x1p-004:C0603
- C2: footprint lcsc:C0402 -> x1p-004:C0402
- HDR1: footprint lcsc:HDR-TH_16P-P2.54-H-F-R2-C8-W8.5 -> x1p-004:HDR-TH_16P-P2.54-H-F-R2-C8-W8.5
- LED1: renamed from U4; footprint lcsc:CONN-SMD_2060-452 -> x1p-004:CONN-SMD_2060-452
- R1, R2: footprint lcsc:R0402 -> x1p-004:R0402
- U1: footprint lcsc:SOT-23-5_L2.9-W1.6-P0.95-LS2.8-BL -> x1p-004:SOT-23-5_L2.9-W1.6-P0.95-LS2.8-BL
- U2, U3: footprint lcsc:SOT-23-6_L2.9-W1.6-P0.95-LS2.8-BR -> x1p-004:SOT-23-6_L2.9-W1.6-P0.95-LS2.8-BR
Connections:
- net 5V: now also SW1.1
- net GND: now also D1.2 (A), D2.2, EXT_POWER1.2, Q1.1, R3.1, R4.1, SW1.2, U4.3 (D)
- net HD0: now also D2.1, D2.6
- net HD1: now also D2.3, D2.4
- net at F1.2: now also EXT_POWER1.1
- net EXT_5V renamed 5V_INT
- net 5V_INT: now also D1.1 (C), D2.5, Q1.4, U4.2 (S)
- new net: Q1.3, R3.2, U4.1 (G)
- new net: Q1.2, Q1.5, Q1.6, R4.2
Other:
- note added: "3.3V -> 5V Shifters"
- note added: "EEPROM"
- note added: "ESD Protection"
- note added: "External 5V WAGO Connector"
- note added: "Int 5V Enable + reverse protection"
- note added: "LED WAGO Connector"
- note added: "X1Plus-Expander Connector"
- moved on the sheet: C2, HDR1, LED1, R1, R2, U1, U2, U3

Commit message: reorient switch, update text
Parts:
- F1: footprint lcsc:F0805 -> x1p-004:F0805
Connections:
- net 5V: now also SW1.2; no longer SW1.1
- net GND: now also EXT_POWER1.1, SW1.1; no longer EXT_POWER1.2, SW1.2
- net at F1.2: now also EXT_POWER1.2; no longer EXT_POWER1.1
Other:
- moved on the sheet: SW1
Changed lines of the file:
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@@
 		(lib_id "lcsc:2060-452_998-404")
 		(at 71.12 39.37 0)
+		(mirror x)
 		(unit 1)
 		(exclude_from_sim no)
@@
 		(dnp no)
 		(property "Reference" "EXT_POWER1"
-			(at 67.056 31.75 0)
+			(at 66.802 32.766 0)
 			(effects
 				(font
@@
 		)
 		(property "Value" "2060-452/998-404"
-			(at 67.056 34.29 0)
+			(at 66.802 34.544 0)
 			(effects
 				(font
@@
 		)
 		(property "Footprint" "x1p-004:CONN-SMD_2060-452"
-			(at 71.12 48.26 0)
+			(at 71.12 30.48 0)
 			(effects
 				(font
@@
 		)
 		(property "LCSC Part" "C2765055"
-			(at 71.12 50.8 0)
+			(at 71.12 27.94 0)
 			(effects
 				(font
@@
 			)
 		)
-		(property "Footprint" "lcsc:F0805"
+		(property "Footprint" "x1p-004:F0805"
 			(at 57.15 41.91 0)
 			(effects
@@
 	(symbol
 		(lib_id "x1p-004:DSIC01THGET")
-		(at 26.67 69.85 270)
+		(at 26.67 69.85 90)
 		(unit 1)
 		(exclude_from_sim no)
@@
 		(dnp no)
 		(property "Reference" "SW1"
-			(at 30.48 69.85 0)
+			(at 22.86 69.85 0)
 			(effects
 				(font
@@
 		)
 		(property "Value" "DSIC01THGET"
-			(at 31.75 69.85 0)
+			(at 21.59 69.85 0)
 			(effects
 				(font
@@
 		)
 		(property "Footprint" "x1p-004:SW-TH_DSIC01THGET"
-			(at 19.05 69.85 0)
+			(at 34.29 69.85 0)
 			(effects
 				(font
@@
 		)
 		(property "Datasheet" "https://lcsc.com/product-detail/DIP-Switches_2-54mm-1-Plugin_C126858.html"
-			(at 16.51 69.85 0)
+			(at 36.83 69.85 0)
 			(effects
 				(font
@@
 		)
 		(property "LCSC Part" "C126858"
-			(at 13.97 69.85 0)
-			(effects
-				(font
+			(at 39.37 69.85 0)
+			(effects
+				(font

Commit message: x1p-004 schem: add pull down resistors on level shifter inputs, add image for DIR input
Parts:
- added R5, R6: 3.3k, x1p-004:R0402, symbol lcsc:0402WGF3301TCE
Connections:
- net GND: now also R5.2, R6.2
- net LD0: now also R5.1
- net LD1: now also R6.1
Other:
- moved on the sheet: D2, U3

Commit message: x1p-004 schem: fix 5V_SW to GND short
Connections:
- net GND: no longer Q1.1, SW1.1, U4.3 (D)
- new net 5V_SW: Q1.1, SW1.1, U4.3 (D)
Changed lines of the file:
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@@
-	)
-	(junction
-		(at 35.56 95.25)
-		(diameter 0)
-		(color 0 0 0 0)
 	)
 	(junction
@@
 	)
 	(junction
-		(at 35.56 80.01)
+		(at 33.02 80.01)
 		(diameter 0)
 		(color 0 0 0 0)
@@
 	(wire
 		(pts
-			(xy 26.67 80.01) (xy 35.56 80.01)
+			(xy 26.67 80.01) (xy 33.02 80.01)
 		)
 		(stroke
@@
 	(wire
 		(pts
-			(xy 35.56 95.25) (xy 35.56 111.76)
-		)
-		(stroke
-			(width 0)
-			(type default)
-		)
-	)
-	(wire
-		(pts
 			(xy 138.43 118.11) (xy 137.16 118.11)
 		)
@@
 	(wire
 		(pts
-			(xy 35.56 80.01) (xy 35.56 95.25)
+			(xy 33.02 80.01) (xy 33.02 111.76)
 		)
 		(stroke
@@
 	(wire
 		(pts
-			(xy 35.56 111.76) (xy 40.64 111.76)
+			(xy 33.02 111.76) (xy 40.64 111.76)
 		)
 		(stroke
@@
 	(wire
 		(pts
-			(xy 35.56 80.01) (xy 48.26 80.01)
-		)
-		(stroke
-			(width 0)
-			(type default)
-		)
-	)
-	(wire
-		(pts
 			(xy 45.72 87.63) (xy 45.72 68.58)
+		)
+		(stroke
+			(width 0)
+			(type default)
+		)
+	)
+	(wire
+		(pts
+			(xy 33.02 80.01) (xy 48.26 80.01)
 		)
 		(stroke
@@
 		)
 	)
+	(label "5V_SW"
+		(at 33.02 80.01 0)
+		(fields_autoplaced yes)
+		(effects
+			(font
+				(size 1.27 1.27)
+			)
+			(justify left bottom)
+		)
+	)

Commit message: x1p-004: add decap for level shifters
Parts:
- added C3: 0.1uf, x1p-004:C0402, symbol lcsc:CL05B104KO5NNNC
Connections:
- net 3V3: now also C3.1
- net GND: now also C3.2
Changed lines of the file:
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@@
+		)
+	)
+	(global_label "3V3"
+		(shape input)
+		(at 214.63 26.67 90)
+		(fields_autoplaced yes)
+		(effects
+			(font
+				(size 1.27 1.27)
+			)
+			(justify left)
+		)
+		(property "Intersheetrefs" "${INTERSHEET_REFS}"
+			(at 214.63 20.1772 90)
+			(effects
+				(font
+					(size 1.27 1.27)
+				)
+				(justify left)
+				(hide yes)
+			)
 		)
 	)
@@
 		(property "Intersheetrefs" "${INTERSHEET_REFS}"
 			(at 162.0543 38.1 0)
+			(effects
+				(font
+					(size 1.27 1.27)
+				)
+				(justify right)
+				(hide yes)
+			)
+		)
+	)
+	(global_label "GND"
+		(shape input)
+		(at 214.63 34.29 270)
+		(fields_autoplaced yes)
+		(effects
+			(font
+				(size 1.27 1.27)
+			)
+			(justify right)
+		)
+		(property "Intersheetrefs" "${INTERSHEET_REFS}"
+			(at 214.63 41.1457 90)
 			(effects
 				(font
@@
 					(unit 1)
 				)
+			)
+		)
+	)
+	(symbol
+		(lib_id "lcsc:CL05B104KO5NNNC")
+		(at 214.63 30.48 270)
+		(unit 1)
+		(exclude_from_sim no)
+		(in_bom yes)
+		(on_board yes)
+		(dnp no)
+		(property "Reference" "C3"
+			(at 217.17 29.718 90)
+			(effects
+				(font
+					(size 1.27 1.27)
+				)
+				(justify left)
+			)
+		)
+		(property "Value" "0.1uf"
+			(at 216.916 32.258 90)
+			(effects
+				(font
+					(size 1.27 1.27)
+				)
+				(justify left)
+			)
+		)
+		(property "Footprint" "x1p-004:C0402"
+			(at 207.01 30.48 0)
+			(effects
+				(font
+					(size 1.27 1.27)
+				)
+				(hide yes)
+			)
+		)
+		(property "Datasheet" "https://lcsc.com/product-detail/Multilayer-Ceramic-Capacitors-MLCC-SMD-SMT_SAMSUNG_CL05B104KO5NNNC_100nF-104-10-16V_C1525.html"
+			(at 204.47 30.48 0)
+			(effects
+				(font
+					(size 1.27 1.27)
+				)
+				(hide yes)
+			)
+		)
+		(property "Description" ""
+			(at 214.63 30.48 0)
+			(effects
+				(font
+					(size 1.27 1.27)
+				)
+				(hide yes)
+			)
+		)
+		(property "LCSC Part" "C1525"
+			(at 201.93 30.48 0)
+			(effects
+				(font
+					(size 1.27 1.27)
+				)
+				(hide yes)
+			)
+		)
+		(pin "2"
+		)
+		(pin "1"
+		)
+		(instances
+			(project "x1p-004"
+				(path "/730ef4da-dc57-4617-8546-a344005f5ae4"
+					(reference "C3")
+					(unit 1)
+				)

Commit message: x1p-004: B01 pseudofinal
Parts:
- removed EXT_POWER1, LED1: 2060-452/998-404, x1p-004:CONN-SMD_2060-452, symbol lcsc:2060-452_998-404
- removed HDR1: PM254-2-08-W-8.5, x1p-004:HDR-TH_16P-P2.54-H-F-R2-C8-W8.5, symbol lcsc:PM254-2-08-W-8.5
- removed R5: 3.3k, x1p-004:R0402, symbol lcsc:0402WGF3301TCE
- removed U2: SN74LVC1T45DBVR, x1p-004:SOT-23-6_L2.9-W1.6-P0.95-LS2.8-BR, symbol lcsc:SN74LVC1T45DBVR
- added CN1: HC-PH-3AWT, x1p-004:CONN-SMD_3P-P2.0-HC-PH-3AWT, symbol x1p-004:HC-PH-3AWT
- added H1, H2: MountingHole, MountingHole:MountingHole_2.2mm_M2, symbol Mechanical:MountingHole
- added HDR1: 220R-2*10P H=8.5MM Ytype Gold-plated black, x1p-004:HDR-TH_20P-P2.54-H-F-R2-C10-S2.54-W10.2, symbol x1p-004:220R-2*10PH=8.5MMYtypeGold-platedblack
- added U2: 2060-453/998-404, x1p-004:CONN-SMD_2060-453, symbol x1p-004:2060-453_998-404
Connections:
- net 3V3: now also HDR1.14, HDR1.8
- net 5V: now also HDR1.10, HDR1.12
- net GND: now also CN1.3, CN1.4, CN1.5, HDR1.16, HDR1.18, HDR1.4, HDR1.6, U2.3
- net HD1: now also CN1.1, U2.1
- net LD1: now also HDR1.5
- net LD6: now also HDR1.15
- net LD7: now also HDR1.17
- net at F1.2: now also CN1.2, U2.2
- net HD0: no longer names the net of D2.1
- net HD0: no longer D2.6
- no-connect marks 4 -> 9
Other:
- note added: "X1Plus Expander Connector"
- note removed: "External 5V WAGO Connector"
- note removed: "X1Plus-Expander Connector"
- moved on the sheet: Q1, R3, R4, SW1, U4

Commit message: X1P-004: homogenize footprints
Parts:
- C1: footprint x1p-004:C0603 -> Capacitor_SMD:C_0603_1608Metric
- C2, C3: footprint x1p-004:C0402 -> Capacitor_SMD:C_0402_1005Metric
- R1, R2, R3, R4, R6: footprint x1p-004:R0402 -> Resistor_SMD:R_0402_1005Metric
Changed lines of the file:
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@@
 			)
 		)
-		(property "Footprint" "x1p-004:R0402"
+		(property "Footprint" "Resistor_SMD:R_0402_1005Metric"
 			(at 40.64 120.65 0)
 			(effects
@@
 			)
 		)
-		(property "Footprint" "x1p-004:C0603"
+		(property "Footprint" "Capacitor_SMD:C_0603_1608Metric"
 			(at 29.21 39.37 0)
 			(effects
@@
 			)
 		)
-		(property "Footprint" "x1p-004:C0402"
+		(property "Footprint" "Capacitor_SMD:C_0402_1005Metric"
 			(at 130.81 121.92 0)
 			(effects
@@
 			)
 		)
-		(property "Footprint" "x1p-004:R0402"
+		(property "Footprint" "Resistor_SMD:R_0402_1005Metric"
 			(at 124.46 104.14 0)
 			(effects
@@
 			)
 		)
-		(property "Footprint" "x1p-004:C0402"
+		(property "Footprint" "Capacitor_SMD:C_0402_1005Metric"
 			(at 207.01 30.48 0)
 			(effects
@@
 			)
 		)
-		(property "Footprint" "x1p-004:R0402"
+		(property "Footprint" "Resistor_SMD:R_0402_1005Metric"
 			(at 175.26 80.01 0)
 			(effects
@@
 			)
 		)
-		(property "Footprint" "x1p-004:R0402"
+		(property "Footprint" "Resistor_SMD:R_0402_1005Metric"
 			(at 68.58 90.17 0)
 			(effects
@@
 			)
 		)
-		(property "Footprint" "x1p-004:R0402"
+		(property "Footprint" "Resistor_SMD:R_0402_1005Metric"
 			(at 116.84 104.14 0)
 			(effects
