File: x1p-004/x1p-004.kicad_sch (KiCad schematic)
At the start: 21 parts, among them CN1 HC-PH-3AWT, Q1 BC857BS,115, SW1 DSIC01THGET, U1 AD24C02, U2 2060-453/998-404, U3 SN74LVC1T45DBVR, U4 SI2301-ZE

Commit message: reduce overall BOM on panels, load manufacturer and MPN in
Parts:
- C2, C3: value 0.1uf -> 0.1uF
- CN1: MPN (none) -> HC-PH-3AWT; Manufacturer (none) -> HCTL
- D1: MPN (none) -> MMSZ5234BT1G; Manufacturer (none) -> onsemi
- D2: MPN (none) -> SRV05-4.TCT; Manufacturer (none) -> UMW
- F1: value 500ma -> BSMD0805-050-15V; MPN (none) -> BSMD0805-050-15V; Manufacturer (none) -> BHFUSE
- H1, H2: now not fitted
- HDR1: value 220R-2*10P H=8.5MM Ytype Gold-plated black -> B-2200R20P-B120; MPN (none) -> B-2200R20P-B120; Manufacturer (none) -> CKMTW
- Q1: MPN (none) -> BC857BS,115; Manufacturer (none) -> Nexperia
- R1, R2, R6: value 3.3k -> 2.2k; LCSC Part C25890 -> C25879
- SW1: MPN (none) -> DSIC01THGET; Manufacturer (none) -> DongGuan KINGTEK Industrial Co. Ltd.
- U1: MPN (none) -> AD24C02; Manufacturer (none) -> IDCHIP
- U2: MPN (none) -> 2060-453/998-404; Manufacturer (none) -> WAGO
- U3: MPN (none) -> SN74LVC1T45DBVR; Manufacturer (none) -> Texas Instruments
- U4: MPN (none) -> SI2301-ZE; Manufacturer (none) -> HXY MOSFET
Changed lines of the file:
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@@
+			)
+		)
+		(property "Manufacturer" "onsemi"
+			(at 45.72 39.37 0)
+			(effects
+				(font
+					(size 1.27 1.27)
+				)
+				(hide yes)
+			)
+		)
+		(property "MPN" "MMSZ5234BT1G"
+			(at 45.72 39.37 0)
+			(effects
+				(font
+					(size 1.27 1.27)
+				)
+				(hide yes)
 			)
 		)
@@
 			)
 		)
+		(property "MPN" "SRV05-4.TCT"
+			(at 185.42 111.76 0)
+			(effects
+				(font
+					(size 1.27 1.27)
+				)
+				(hide yes)
+			)
+		)
+		(property "Manufacturer" "UMW"
+			(at 185.42 111.76 0)
+			(effects
+				(font
+					(size 1.27 1.27)
+				)
+				(hide yes)
+			)
+		)
 		(pin "2"
 		)
@@
 			)
 		)
+		(property "MPN" "SI2301-ZE"
+			(at 45.72 129.54 0)
+			(effects
+				(font
+					(size 1.27 1.27)
+				)
+				(hide yes)
+			)
+		)
+		(property "Manufacturer" "HXY MOSFET"
+			(at 45.72 129.54 0)
+			(effects
+				(font
+					(size 1.27 1.27)
+				)
+				(hide yes)
+			)
+		)
 		(pin "3"
 		)
@@
 		(in_bom no)
 		(on_board yes)
-		(dnp no)
+		(dnp yes)
 		(fields_autoplaced yes)
 		(property "Reference" "H1"
@@
 			)
 		)
-		(property "Value" "0.1uf"
+		(property "Value" "0.1uF"
 			(at 140.716 123.698 90)
 			(effects
@@
 			)
 		)
-		(property "Value" "3.3k"
+		(property "Value" "2.2k"
 			(at 118.11 105.41 90)
 			(effects
@@
 			)
 		)
-		(property "Datasheet" "https://lcsc.com/product-detail/Chip-Resistor-Surface-Mount-UniOhm_3-3KR-3301-1_C25890.html"
+		(property "Datasheet" "https://lcsc.com/product-detail/Chip-Resistor-Surface-Mount-UniOhm_2-2KR-2201-1_C25879.html"
 			(at 127 104.14 0)
 			(effects
@@
 			)
 		)
-		(property "LCSC Part" "C25890"
+		(property "LCSC Part" "C25879"
 			(at 129.54 104.14 0)
 			(effects
@@
 			)
 		)
-		(property "Value" "500ma"
+		(property "Value" "BSMD0805-050-15V"
 			(at 57.15 36.576 0)
 			(effects
@@
 			)
 		)
+		(property "MPN" "BSMD0805-050-15V"
+			(at 57.15 34.29 0)
+			(effects
+				(font
+					(size 1.27 1.27)
+				)
+				(hide yes)
+			)
+		)
+		(property "Manufacturer" "BHFUSE"
+			(at 57.15 34.29 0)
+			(effects
+				(font
+					(size 1.27 1.27)
+				)
+				(hide yes)
+			)
+		)
 		(pin "2"
 		)
@@
 		(in_bom no)
 		(on_board yes)
-		(dnp no)
+		(dnp yes)
 		(fields_autoplaced yes)
 		(property "Reference" "H2"
@@
 			)
 		)
-		(property "Value" "220R-2*10P H=8.5MM Ytype Gold-plated black"
+		(property "Value" "B-2200R20P-B120"
 			(at 124.46 50.8 0)
 			(effects
@@
 		(property "LCSC Part" "C124406"
 			(at 124.46 90.17 0)
+			(effects
+				(font
+					(size 1.27 1.27)
+				)
+				(hide yes)
+			)
+		)
+		(property "MPN" "B-2200R20P-B120"
+			(at 124.46 66.04 0)
+			(effects
+				(font
+					(size 1.27 1.27)
+				)
+				(hide yes)
+			)
+		)
+		(property "Manufacturer" "CKMTW"
+			(at 124.46 66.04 0)
 			(effects
 				(font
@@
 			)
 		)
-		(property "Value" "0.1uf"
+		(property "Value" "0.1uF"
 			(at 216.916 32.258 90)
 			(effects
@@
 			)
 		)
-		(property "Value" "3.3k"
+		(property "Value" "2.2k"
 			(at 173.99 73.66 90)
 			(effects
@@
 			)
 		)
-		(property "Datasheet" "https://lcsc.com/product-detail/Chip-Resistor-Surface-Mount-UniOhm_3-3KR-3301-1_C25890.html"
+		(property "Datasheet" "https://lcsc.com/product-detail/Chip-Resistor-Surface-Mount-UniOhm_2-2KR-2201-1_C25879.html"
 			(at 175.26 82.55 0)
 			(effects
@@
 			)
 		)
-		(property "LCSC Part" "C25890"
+		(property "LCSC Part" "C25879"
 			(at 175.26 85.09 0)
 			(effects
@@
 			)
 		)
+		(property "MPN" "SN74LVC1T45DBVR"
+			(at 184.15 64.77 0)
+			(effects
+				(font
+					(size 1.27 1.27)
+				)
+				(hide yes)
+			)
+		)
+		(property "Manufacturer" "Texas Instruments"
+			(at 184.15 64.77 0)
+			(effects
+				(font
+					(size 1.27 1.27)
+				)
+				(hide yes)
+			)
+		)
 		(pin "1"
 		)
@@
 			)
 		)
+		(property "MPN" "BC857BS,115"
+			(at 54.61 105.41 0)
+			(effects
+				(font
+					(size 1.27 1.27)
+				)
+				(hide yes)
+			)
+		)
+		(property "Manufacturer" "Nexperia"
+			(at 54.61 105.41 0)
+			(effects
+				(font
+					(size 1.27 1.27)
+				)
+				(hide yes)
+			)
+		)
 		(pin "1"
 		)
@@
 			)
 		)
-		(property "Value" "3.3k"
+		(property "Value" "2.2k"
 			(at 110.49 105.41 90)
 			(effects
@@
 			)
 		)
-		(property "Datasheet" "https://lcsc.com/product-detail/Chip-Resistor-Surface-Mount-UniOhm_3-3KR-3301-1_C25890.html"
+		(property "Datasheet" "https://lcsc.com/product-detail/Chip-Resistor-Surface-Mount-UniOhm_2-2KR-2201-1_C25879.html"
 			(at 119.38 104.14 0)
 			(effects
@@
 			)
 		)
-		(property "LCSC Part" "C25890"
+		(property "LCSC Part" "C25879"
 			(at 121.92 104.14 0)
 			(effects
@@
 			)
 		)
+		(property "MPN" "AD24C02"
+			(at 128.27 115.57 0)
+			(effects
+				(font
+					(size 1.27 1.27)
+				)
+				(hide yes)
+			)
+		)
+		(property "Manufacturer" "IDCHIP"
+			(at 128.27 115.57 0)
+			(effects
+				(font
+					(size 1.27 1.27)
+				)
+				(hide yes)
+			)
+		)
 		(pin "4"
 		)
@@
 		(property "LCSC Part" "C126858"
 			(at 39.37 87.63 0)
+			(effects
+				(font
+					(size 1.27 1.27)
+				)
+				(hide yes)
+			)
+		)
+		(property "MPN" "DSIC01THGET"
+			(at 26.67 87.63 0)
+			(effects
+				(font
+					(size 1.27 1.27)
+				)
+				(hide yes)
+			)
+		)
+		(property "Manufacturer" "DongGuan KINGTEK Industrial Co. Ltd."
+			(at 26.67 87.63 0)
 			(effects
 				(font
@@
 			)
 		)
+		(property "MPN" "HC-PH-3AWT"
+			(at 76.2 57.15 0)
+			(effects
+				(font
+					(size 1.27 1.27)
+				)
+				(hide yes)
+			)
+		)
+		(property "Manufacturer" "HCTL"
+			(at 76.2 57.15 0)
+			(effects
+				(font
+					(size 1.27 1.27)
+				)
+				(hide yes)
+			)
+		)
 		(pin "2"
 		)
@@
 			(effects
 				(font
+					(size 1.27 1.27)
+				)
+				(hide yes)
+			)
+		)
+		(property "MPN" "2060-453/998-404"
+			(at 77.47 38.1 0)
+			(effects
+				(font
+					(size 1.27 1.27)
+				)
+				(hide yes)
+			)
+		)
+		(property "Manufacturer" "WAGO"
+			(at 77.47 38.1 0)
+			(effects
+				(font

Commit message: add King Credie recommended components, fix panel placement, fix pulldown on x1p-005, fix bridges on x1p-006
Parts:
- C1: MPN (none) -> CL10A105KB8NNNC; Manufacturer (none) -> Samsung
- C2, C3: MPN (none) -> CL05B104KB54PNC; Manufacturer (none) -> Samsung
- R1, R2, R6: MPN (none) -> RC0402FR-072K2L; Manufacturer (none) -> Yageo
- R3: MPN (none) -> RC0402FR-07100KL; Manufacturer (none) -> Yageo
- R4: MPN (none) -> RC0402FR-0768KL; Manufacturer (none) -> Yageo
Changed lines of the file:
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@@
 	(label "5V_SW"
 		(at 33.02 97.79 0)
-		(fields_autoplaced yes)
 		(effects
 			(font
@@
 			)
 		)
+		(property "MPN" "RC0402FR-07100KL"
+			(at 40.64 113.03 0)
+			(effects
+				(font
+					(size 1.27 1.27)
+				)
+				(hide yes)
+			)
+		)
+		(property "Manufacturer" "Yageo"
+			(at 40.64 113.03 0)
+			(effects
+				(font
+					(size 1.27 1.27)
+				)
+				(hide yes)
+			)
+		)
 		(pin "2"
 		)
@@
 		(property "LCSC Part" "C15849"
 			(at 24.13 39.37 0)
+			(effects
+				(font
+					(size 1.27 1.27)
+				)
+				(hide yes)
+			)
+		)
+		(property "MPN" "CL10A105KB8NNNC"
+			(at 36.83 39.37 0)
+			(effects
+				(font
+					(size 1.27 1.27)
+				)
+				(hide yes)
+			)
+		)
+		(property "Manufacturer" "Samsung"
+			(at 36.83 39.37 0)
 			(effects
 				(font
@@
 			)
 		)
+		(property "MPN" "CL05B104KB54PNC"
+			(at 138.43 121.92 0)
+			(effects
+				(font
+					(size 1.27 1.27)
+				)
+				(hide yes)
+			)
+		)
+		(property "Manufacturer" "Samsung"
+			(at 138.43 121.92 0)
+			(effects
+				(font
+					(size 1.27 1.27)
+				)
+				(hide yes)
+			)
+		)
 		(pin "2"
 		)
@@
 			)
 		)
+		(property "MPN" "RC0402FR-072K2L"
+			(at 116.84 104.14 0)
+			(effects
+				(font
+					(size 1.27 1.27)
+				)
+				(hide yes)
+			)
+		)
+		(property "Manufacturer" "Yageo"
+			(at 116.84 104.14 0)
+			(effects
+				(font
+					(size 1.27 1.27)
+				)
+				(hide yes)
+			)
+		)
 		(pin "2"
 		)
@@
 			)
 		)
+		(property "MPN" "CL05B104KB54PNC"
+			(at 214.63 30.48 0)
+			(effects
+				(font
+					(size 1.27 1.27)
+				)
+				(hide yes)
+			)
+		)
+		(property "Manufacturer" "Samsung"
+			(at 214.63 30.48 0)
+			(effects
+				(font
+					(size 1.27 1.27)
+				)
+				(hide yes)
+			)
+		)
 		(pin "2"
 		)
@@
 			)
 		)
+		(property "MPN" "RC0402FR-072K2L"
+			(at 175.26 72.39 0)
+			(effects
+				(font
+					(size 1.27 1.27)
+				)
+				(hide yes)
+			)
+		)
+		(property "Manufacturer" "Yageo"
+			(at 175.26 72.39 0)
+			(effects
+				(font
+					(size 1.27 1.27)
+				)
+				(hide yes)
+			)
+		)
 		(pin "2"
 		)
@@
 			)
 		)
+		(property "MPN" "RC0402FR-0768KL"
+			(at 68.58 97.79 0)
+			(effects
+				(font
+					(size 1.27 1.27)
+				)
+				(hide yes)
+			)
+		)
+		(property "Manufacturer" "Yageo"
+			(at 68.58 97.79 0)
+			(effects
+				(font
+					(size 1.27 1.27)
+				)
+				(hide yes)
+			)
+		)
 		(pin "1"
 		)
@@
 			(effects
 				(font
+					(size 1.27 1.27)
+				)
+				(hide yes)
+			)
+		)
+		(property "MPN" "RC0402FR-072K2L"
+			(at 109.22 104.14 0)
+			(effects
+				(font
+					(size 1.27 1.27)
+				)
+				(hide yes)
+			)
+		)
+		(property "Manufacturer" "Yageo"
+			(at 109.22 104.14 0)
+			(effects
+				(font
