File: x1p-006/x1p-006.kicad_pcb (KiCad board)
At the start: 2 copper layers, 20.8 x 27.4 mm, 11 parts, among them U1 AD24C02, U3 TLP172GM(TPL,E(O, U6 TLP172GM(TPL,E(O

Commit message: fix 3dshapes
Parts:
- C1: footprint x1p-005:C0402 -> x1p-006:C0402
- HDR1: footprint x1p-005:HDR-TH_16P-P2.54-H-F-R2-C8-W8.5 -> x1p-006:HDR-TH_16P-P2.54-H-F-R2-C8-W8.5
- R1, R2: footprint x1p-005:R0402 -> x1p-006:R0402
- U1: footprint x1p-005:SOT-23-5_L2.9-W1.6-P0.95-LS2.8-BL -> x1p-006:SOT-23-5_L2.9-W1.6-P0.95-LS2.8-BL
Connections:
- HDR1 pad 7: 5V -> unconnected-(HDR1-Pad7)
- HDR1 pad 9: 5V -> unconnected-(HDR1-Pad9)
