File: x1p-006/x1p-006.kicad_pcb (KiCad board)
At the start: 2 copper layers, 20.8 x 27.4 mm, 11 parts, among them U1 AD24C02, U3 TLP172GM(TPL,E(O, U6 TLP172GM(TPL,E(O

Commit message: 0 drc errors \o/
Parts:
- C1: footprint x1p-005:C0402 -> x1p-006:C0402
- HDR1: footprint x1p-005:HDR-TH_16P-P2.54-H-F-R2-C8-W8.5 -> x1p-006:HDR-TH_16P-P2.54-H-F-R2-C8-W8.5
- R1, R2: footprint x1p-005:R0402 -> x1p-006:R0402
- U1: footprint x1p-005:SOT-23-5_L2.9-W1.6-P0.95-LS2.8-BL -> x1p-006:SOT-23-5_L2.9-W1.6-P0.95-LS2.8-BL
Connections:
- HDR1 pad 7: 5V -> unconnected-(HDR1-Pad7)
- HDR1 pad 9: 5V -> unconnected-(HDR1-Pad9)

Commit message: x1p-006 singlesided
Parts:
- C1, R1, R2, R3, R4, U1, U3, U6: moved to F.Cu
- moved R1 7.89 mm to (72.4, 112.8)
- moved R2 7.39 mm to (77.2, 112.8)
- moved C1 6.61 mm to (76.5, 109.8), turned to 0 degrees
- moved R4 6.28 mm to (70.6, 115.8)
- moved U1 5.95 mm to (74.8, 112.1), turned to 0 degrees
- moved R3 5.55 mm to (64.2, 115.8)
- moved PJ1 5.20 mm to (62.5, 103.5)
- moved PJ2 5.20 mm to (74.5, 103.5)
- moved U6 2.57 mm to (68.0, 112.4)
- moved U3 2.51 mm to (61.6, 112.4)
Routing:
- net LD7: track 3.81 -> 11.1 mm, vias 0 -> 1
- net LD6: track 3.88 -> 10.0 mm
- net Net-(PJ1-Pad3): track 4.24 -> 9.74 mm
- net Net-(PJ1-Pad1): track 3.84 -> 8.08 mm, vias 0 -> 1
- net Net-(PJ2-Pad3): track 10.9 -> 15.1 mm, vias 0 -> 1
- net LD1: track 7.84 -> 9.27 mm
- net LD0: track 4.85 -> 5.85 mm
- net GND: track 5.47 -> 5.93 mm, vias 4 -> 5
- added copper zone on F.Cu, net 3V3
- added copper zone on B.Cu, net GND
- removed copper zone on B.Cu, net 3V3
- removed copper zone on F.Cu, net GND
Other:
- board size 20.8 x 27.4 mm -> 20.8 x 32.6 mm

Commit message: x1p-006-b01
Parts:
- removed U6: TLP172GM(TPL,E(O, x1p-006:SMD-4_L4.6-W3.7-P2.54-LS7.0-BR
- added U2: TLP240A(TP1,F, x1p-006:RELAY-SMD_TLP240A, F.Cu at (62.2, 111.7)
- HDR1: value PM254-2-08-W-8.5 -> 220R-2*10P H=8.5MM Ytype Gold-plated black; footprint x1p-006:HDR-TH_16P-P2.54-H-F-R2-C8-W8.5 -> x1p-006:HDR-TH_20P-P2.54-H-F-R2-C10-S2.54-W10.2
- U3: value TLP172GM(TPL,E(O -> TLP240A(TP1,F; footprint x1p-006:SMD-4_L4.6-W3.7-P2.54-LS7.0-BR -> x1p-006:RELAY-SMD_TLP240A
- moved U3 13.2 mm to (74.8, 111.7)
- moved C1 10.9 mm to (70.0, 101.0)
- moved R1 10.9 mm to (66.0, 104.0)
- moved R2 10.9 mm to (70.8, 104.0)
- moved U1 10.9 mm to (68.5, 103.3)
- moved R3 6.06 mm to (58.2, 115.2), turned to 180 degrees
- moved PJ1 1.65 mm to (60.8, 103.5)
- moved PJ2 1.55 mm to (76.0, 103.5)
- moved R4 0.60 mm to (70.8, 115.2), turned to 180 degrees
Connections:
- HDR1 pad 1: GND -> unconnected-(HDR1-Pad1)
- HDR1 pad 11: 3V3 -> unconnected-(HDR1-Pad11)
- HDR1 pad 13: GND -> LD5
- HDR1 pad 14: LD6 -> 3V3
- HDR1 pad 15: GND -> LD6
- HDR1 pad 16: LD7 -> GND
- HDR1 pad 2: LD0 -> unconnected-(HDR1-Pad2)
- HDR1 pad 3: GND -> unconnected-(HDR1-Pad3)
- HDR1 pad 4: LD1 -> GND
- HDR1 pad 5: 3V3 -> unconnected-(HDR1-Pad5)
- HDR1 pad 6: unconnected-(HDR1-Pad6) -> GND
- HDR1 pad 8: unconnected-(HDR1-Pad8) -> 3V3
- HDR1 pad 9: unconnected-(HDR1-Pad9) -> LD3
- PJ1 pad 2: unconnected-(PJ1-Pad2) -> Net-(PJ1-Pad2)
- PJ1 pad 3: Net-(PJ1-Pad3) -> unconnected-(PJ1-Pad3)
- PJ2 pad 2: unconnected-(PJ2-Pad2) -> Net-(PJ2-Pad2)
- PJ2 pad 3: Net-(PJ2-Pad3) -> unconnected-(PJ2-Pad3)
- R3 pad 2: Net-(R3-Pad2) -> Net-(U2-C)
- R4 pad 2: Net-(R4-Pad2) -> Net-(U3-C)
- U3 pad 1: LD0 -> LD5
- U3 pad 2: Net-(R3-Pad2) -> Net-(U3-C)
- U3 pad 3: Net-(PJ1-Pad1) -> Net-(PJ2-Pad1)
- U3 pad 4: Net-(PJ1-Pad3) -> Net-(PJ2-Pad2)
Routing:
- net Net-(PJ2-Pad3): track 15.1 -> 0.00 mm, vias 1 -> 0
- net LD3: track 0.00 -> 14.8 mm
- net LD5: track 0.00 -> 13.5 mm
- net LD7: track 11.1 -> 22.5 mm
- net LD6: track 10.0 -> 20.0 mm
- net Net-(PJ1-Pad3): track 9.74 -> 0.00 mm
- net Net-(PJ1-Pad2): track 0.00 -> 9.71 mm
- net LD1: track 9.27 -> 0.00 mm
- net Net-(PJ2-Pad2): track 0.00 -> 8.66 mm
- net Net-(PJ1-Pad1): track 8.08 -> 15.5 mm, vias 1 -> 0
- net LD0: track 5.85 -> 0.00 mm
- net Net-(PJ2-Pad1): track 9.50 -> 14.3 mm
- net Net-(U2-C): track 0.00 -> 2.28 mm
- net Net-(U3-C): track 0.00 -> 2.20 mm
- net Net-(R3-Pad2): track 1.45 -> 0.00 mm
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Other:
- board size 20.8 x 32.6 mm -> 26 x 32.6 mm
- board text added: "X1P-006-B01"
- board text removed: "X1P-006-A01"

Commit message: change jack to trrs
Parts:
- removed PJ1, PJ2: PJ-211, x1p-006:AUDIO-TH_PJ-211
- added CAM1: PJ-2013-L6S, x1p-006:AUDIO-TH_PJ-2013-L6S, F.Cu at (60.8, 100.3)
- added CAM2: PJ-2013-L6S, x1p-006:AUDIO-TH_PJ-2013-L6S, F.Cu at (76.0, 100.3)
- added JP1: SolderJumper_2_Bridged, Jumper:SolderJumper-2_P1.3mm_Bridged_RoundedPad1.0x1.5mm, B.Cu at (62.8, 102.4)
- added JP2: SolderJumper_2_Bridged, Jumper:SolderJumper-2_P1.3mm_Bridged_RoundedPad1.0x1.5mm, B.Cu at (78.0, 102.4)
Routing:
- net Net-(CAM2-Pad1): track 14.3 -> 20.8 mm
- net Net-(CAM1-Pad1): track 15.5 -> 21.7 mm
- net Net-(JP2-B): track 0.00 -> 2.59 mm
- net Net-(JP2-A): track 8.66 -> 11.2 mm
- net Net-(JP1-A): track 9.71 -> 12.1 mm
- net Net-(JP1-B): track 0.00 -> 2.39 mm

Commit message: fixes
Parts:
- added H1: MountingHole, MountingHole:MountingHole_2.2mm_M2_ISO7380, F.Cu at (68.4, 107.8)
- added JP3: SolderJumper_2_Bridged, Jumper:SolderJumper-2_P1.3mm_Bridged_RoundedPad1.0x1.5mm, B.Cu at (65.2, 96.2)
- added JP4: SolderJumper_2_Bridged, Jumper:SolderJumper-2_P1.3mm_Bridged_RoundedPad1.0x1.5mm, B.Cu at (71.4, 96.2)
- added JP5: SolderJumper_2_Bridged, Jumper:SolderJumper-2_P1.3mm_Bridged_RoundedPad1.0x1.5mm, B.Cu at (63.8, 104.6)
- added JP6: SolderJumper_2_Bridged, Jumper:SolderJumper-2_P1.3mm_Bridged_RoundedPad1.0x1.5mm, B.Cu at (79.2, 104.6)
- added R5: 3.3k, x1p-006:R0402, F.Cu at (58.0, 110.2)
- added R6: 3.3k, x1p-006:R0402, F.Cu at (70.6, 110.2)
- JP1, JP2: value SolderJumper_2_Bridged -> SolderJumper_2_Open; footprint Jumper:SolderJumper-2_P1.3mm_Bridged_RoundedPad1.0x1.5mm -> Jumper:SolderJumper-2_P1.3mm_Open_RoundedPad1.0x1.5mm
- moved JP1 3.64 mm to (60.2, 99.8)
- moved JP2 3.44 mm to (75.4, 100.2)
- moved R4 1.76 mm to (69.2, 114.5), turned to -90 degrees
- moved R3 1.73 mm to (56.6, 114.5), turned to -90 degrees
- moved U3 1.62 mm to (75.4, 113.2)
- moved U2 1.62 mm to (62.8, 113.2)
- moved C1 1.40 mm to (70.0, 99.6)
- moved R1 1.40 mm to (66.0, 102.6)
- moved R2 1.40 mm to (70.8, 102.6)
- moved U1 1.40 mm to (68.5, 101.9)
Connections:
- CAM1 pad 2: unconnected-(CAM1-Pad2) -> Net-(JP3-B)
- CAM1 pad 4: Net-(JP1-A) -> Net-(JP5-B)
- CAM2 pad 2: unconnected-(CAM2-Pad2) -> Net-(JP4-B)
- CAM2 pad 4: Net-(JP2-A) -> Net-(JP6-B)
Routing:
- net Net-(JP3-A): track 21.7 -> 29.8 mm
- net Net-(JP4-B): track 0.00 -> 7.56 mm
- net Net-(JP4-A): track 20.8 -> 25.0 mm
- net Net-(JP3-B): track 0.00 -> 3.47 mm
- net Net-(JP1-A): track 12.1 -> 14.8 mm, vias 0 -> 1
- net Net-(JP6-B): track 0.00 -> 2.60 mm
- net Net-(JP5-B): track 0.00 -> 2.60 mm
- net LD7: track 22.5 -> 25.1 mm
- net Net-(JP2-A): track 11.2 -> 13.6 mm, vias 0 -> 1
- net GND: track 5.99 -> 7.93 mm, vias 5 -> 7
- net LD6: track 20.0 -> 21.4 mm
- net LD5: track 13.5 -> 12.4 mm
Other:
- board text added: "R"
- board text added: "S"
- board text added: "T"
