File: x1p-006/x1p-006.kicad_pcb (KiCad board)
At the start: 2 copper layers, 26 x 32.6 mm, 20 parts, among them U1 AD24C02, U2 TLP240A(TP1,F, U3 TLP240A(TP1,F

Commit message: change to TRS jack, change ssr to instock part, remove jumpers
Parts:
- removed JP1, JP2: SolderJumper_2_Open, Jumper:SolderJumper-2_P1.3mm_Open_RoundedPad1.0x1.5mm
- removed JP3, JP4, JP5, JP6: SolderJumper_2_Bridged, Jumper:SolderJumper-2_P1.3mm_Bridged_RoundedPad1.0x1.5mm
- CAM1, CAM2: value PJ-2013-L6S -> PJ-211A; footprint x1p-006:AUDIO-TH_PJ-2013-L6S -> x1p-006:AUDIO-TH_PJ-211A
- U2, U3: value TLP240A(TP1,F -> AQY212EHAX; footprint x1p-006:RELAY-SMD_TLP240A -> x1p-006:SOP-4_L6.5-W4.6-P2.54-LS10.2-TR
- moved R4 11.8 mm to (79.8, 109.4)
- moved R6 6.21 mm to (76.8, 109.8)
- moved R3 5.64 mm to (59.8, 109.8), turned to 180 degrees
- moved U1 2.95 mm to (68.4, 99.0)
- moved C1 2.95 mm to (70.0, 96.7)
- moved R1 2.95 mm to (66.0, 99.7)
- moved R2 2.95 mm to (70.8, 99.7)
- moved CAM1 2.90 mm to (60.8, 103.2)
- moved CAM2 2.90 mm to (76.0, 103.2)
- moved R5 1.28 mm to (57.0, 109.4), turned to -90 degrees
- moved U2 0.70 mm to (62.1, 113.1), turned to 90 degrees
- moved U3 0.68 mm to (74.7, 113.1)
Connections:
- CAM1 pad 1: Net-(JP3-A) -> Net-(U2-S)
- CAM1 pad 2: Net-(JP3-B) -> Net-(U2-S1)
- CAM1 pad 3: Net-(JP1-B) -> unconnected-(CAM1-Pad3)
- CAM2 pad 1: Net-(JP4-A) -> Net-(U3-S)
- CAM2 pad 2: Net-(JP4-B) -> Net-(U3-S1)
- CAM2 pad 3: Net-(JP2-B) -> unconnected-(CAM2-Pad3)
- U2 pad 3: Net-(JP3-A) -> Net-(U2-S1)
- U2 pad 4: Net-(JP1-A) -> Net-(U2-S)
- U3 pad 3: Net-(JP4-A) -> Net-(U3-S1)
- U3 pad 4: Net-(JP2-A) -> Net-(U3-S)
Routing:
- net Net-(JP3-A): track 29.8 -> 0.00 mm
- net Net-(JP4-A): track 25.0 -> 0.00 mm
- net Net-(U3-S): track 0.00 -> 16.4 mm, vias 0 -> 1
- net Net-(U2-S): track 0.00 -> 15.3 mm, vias 0 -> 1
- net Net-(JP1-A): track 14.8 -> 0.00 mm, vias 1 -> 0
- net Net-(U2-S1): track 0.00 -> 13.9 mm, vias 0 -> 1
- net Net-(JP2-A): track 13.6 -> 0.00 mm, vias 1 -> 0
- net Net-(U3-S1): track 0.00 -> 11.3 mm, vias 0 -> 1
- net Net-(JP4-B): track 7.56 -> 0.00 mm
- net LD5: track 12.4 -> 18.4 mm, vias 0 -> 2
- net Net-(U2-K): track 1.99 -> 6.98 mm
- net Net-(JP3-B): track 3.47 -> 0.00 mm
- net LD7: track 25.1 -> 28.3 mm
- net LD6: track 21.4 -> 24.4 mm
- net Net-(JP2-B): track 2.62 -> 0.00 mm
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Other:
- board text removed: "R"
- board text removed: "S"
- board text removed: "T"

Commit message: add jumpers
Parts:
- added JP1: SolderJumper_2_Bridged, Jumper:SolderJumper-2_P1.3mm_Bridged_RoundedPad1.0x1.5mm, B.Cu at (64.2, 106.8)
- added JP2: SolderJumper_2_Open, Jumper:SolderJumper-2_P1.3mm_Open_RoundedPad1.0x1.5mm, B.Cu at (64.8, 102.5)
- added JP3: SolderJumper_2_Bridged, Jumper:SolderJumper-2_P1.3mm_Bridged_RoundedPad1.0x1.5mm, B.Cu at (78.8, 106.0)
- added JP4: SolderJumper_2_Open, Jumper:SolderJumper-2_P1.3mm_Open_RoundedPad1.0x1.5mm, B.Cu at (79.8, 102.5)
Connections:
- CAM1 pad 1: Net-(U2-S) -> Net-(JP1-B)
- CAM1 pad 3: unconnected-(CAM1-Pad3) -> Net-(JP2-B)
- CAM2 pad 1: Net-(U3-S) -> Net-(JP3-B)
- CAM2 pad 3: unconnected-(CAM2-Pad3) -> Net-(JP4-B)
- U2 pad 4: Net-(U2-S) -> Net-(JP1-A)
- U3 pad 4: Net-(U3-S) -> Net-(JP3-A)
Routing:
- net Net-(JP3-A): track 0.00 -> 17.6 mm, vias 0 -> 1
- net Net-(U3-S): track 16.4 -> 0.00 mm, vias 1 -> 0
- net Net-(U2-S): track 15.3 -> 0.00 mm, vias 1 -> 0
- net Net-(JP1-A): track 0.00 -> 11.1 mm, vias 0 -> 1
- net Net-(JP1-B): track 0.00 -> 7.68 mm
- net Net-(JP3-B): track 0.00 -> 6.66 mm
- net Net-(JP2-B): track 0.00 -> 2.24 mm
- net Net-(JP4-B): track 0.00 -> 2.04 mm

Commit message: x1p-006: adjust layout to homogenize
Parts:
- C1: footprint x1p-006:C0402 -> Capacitor_SMD:C_0402_1005Metric
- R1, R2, R3, R4, R5, R6: footprint x1p-006:R0402 -> Resistor_SMD:R_0402_1005Metric
- moved R6 86.5 mm to (161.6, 92.8), turned to 90 degrees
- moved U3 85.2 mm to (156.4, 89.0)
- moved U2 85.0 mm to (143.6, 89.0)
- moved JP4 84.9 mm to (161.6, 79.8)
- moved R2 84.7 mm to (152.4, 77.0)
- moved JP2 84.7 mm to (146.4, 79.8)
- moved U1 84.7 mm to (150.0, 76.3)
- moved CAM2 84.7 mm to (157.6, 80.6)
- moved HDR1 84.7 mm to (150.0, 100.0)
- moved CAM1 84.7 mm to (142.4, 80.6)
- moved R1 84.7 mm to (147.5, 77.0)
- moved JP3 84.3 mm to (160.0, 83.4)
- moved R5 84.2 mm to (139.6, 92.8), turned to 90 degrees
- moved JP1 84.0 mm to (144.8, 83.4)
- moved C1 83.1 mm to (150.0, 74.0), turned to 180 degrees
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Routing:
- net Net-(U2-K): track 6.98 -> 2.77 mm
- net Net-(U3-K): track 2.06 -> 5.18 mm
- net GND: track 7.87 -> 9.75 mm, vias 7 -> 3
- net Net-(U2-S1): track 13.9 -> 12.1 mm
- net LD5: track 18.4 -> 16.9 mm, vias 2 -> 0
- net Net-(JP1-B): track 7.68 -> 6.26 mm
- net Net-(U3-S1): track 11.3 -> 9.87 mm
- net Net-(JP1-A): track 11.1 -> 10.0 mm
- net LD3: track 17.4 -> 17.8 mm, vias 1 -> 0
Other:
- board size 26 x 32.6 mm -> 26.4 x 33 mm
- board text added: "X1P-006-B02"
- board text removed: "X1P-006-B01"

Commit message: reduce overall BOM on panels, load manufacturer and MPN in
Parts:
- C1: value 0.1uf -> 0.1uF
- HDR1: value 220R-2*10P H=8.5MM Ytype Gold-plated black -> B-2200R20P-B120
- R1, R2, R5, R6: value 3.3k -> 2.2k

Commit message: add King Credie recommended components, fix panel placement, fix pulldown on x1p-005, fix bridges on x1p-006
Parts:
- JP2, JP4: footprint Jumper:SolderJumper-2_P1.3mm_Open_RoundedPad1.0x1.5mm -> Jumper:SolderJumper-2_P1.3mm_Bridged_RoundedPad1.0x1.5mm
Other:
- board text added: "R"
- board text added: "T"
Changed lines of the file:
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@@
 			)
 		)
-		(property "MPN" ""
+		(property "MPN" "RC0402FR-07220RL"
 			(at 0 0 90)
 			(unlocked yes)
@@
 			)
 		)
-		(property "Manufacturer" ""
+		(property "Manufacturer" "YAGEO"
 			(at 0 0 90)
 			(unlocked yes)
@@
 			)
 		)
-		(property "MPN" ""
+		(property "MPN" "RC0402FR-072K2L"
 			(at 0 0 90)
 			(unlocked yes)
@@
 			)
 		)
-		(property "Manufacturer" ""
+		(property "Manufacturer" "YAGEO"
 			(at 0 0 90)
 			(unlocked yes)
@@
 			)
 		)
-		(property "MPN" ""
+		(property "MPN" "RC0402FR-072K2L"
 			(at 0 0 90)
 			(unlocked yes)
@@
 			)
 		)
-		(property "Manufacturer" ""
+		(property "Manufacturer" "YAGEO"
 			(at 0 0 90)
 			(unlocked yes)
@@
 			)
 		)
-		(property "MPN" ""
+		(property "MPN" "RC0402FR-072K2L"
 			(at 0 0 90)
 			(unlocked yes)
@@
 			)
 		)
-		(property "Manufacturer" ""
+		(property "Manufacturer" "YAGEO"
 			(at 0 0 90)
 			(unlocked yes)
@@
 			)
 		)
-		(property "MPN" ""
+		(property "MPN" "RC0402FR-07220RL"
 			(at 0 0 90)
 			(unlocked yes)
@@
 			)
 		)
-		(property "Manufacturer" ""
+		(property "Manufacturer" "YAGEO"
 			(at 0 0 90)
 			(unlocked yes)
@@
 			)
 		)
-		(property "MPN" ""
+		(property "MPN" "CL05B104KB54PNC"
 			(at 0 0 180)
 			(unlocked yes)
@@
 			)
 		)
-		(property "Manufacturer" ""
+		(property "Manufacturer" "Samsung"
 			(at 0 0 180)
 			(unlocked yes)
@@
 			)
 		)
-		(property "MPN" ""
+		(property "MPN" "RC0402FR-072K2L"
 			(at 0 0 90)
 			(unlocked yes)
@@
 			)
 		)
-		(property "Manufacturer" ""
+		(property "Manufacturer" "YAGEO"
 			(at 0 0 90)
 			(unlocked yes)
@@
 		)
 	)
-	(footprint "Jumper:SolderJumper-2_P1.3mm_Open_RoundedPad1.0x1.5mm"
+	(footprint "Jumper:SolderJumper-2_P1.3mm_Bridged_RoundedPad1.0x1.5mm"
 		(layer "B.Cu")
 		(at 146.39 79.8 90)
-		(descr "SMD Solder Jumper, 1x1.5mm, rounded Pads, 0.3mm gap, open")
-		(tags "solder jumper open")
+		(descr "SMD Solder Jumper, 1x1.5mm, rounded Pads, 0.3mm gap, bridged with 1 copper strip")
+		(tags "net tie solder jumper bridged")
 		(property "Reference" "JP2"
-			(at 0 1.8 90)
+			(at 0 1.8 -90)
 			(layer "B.SilkS")
 			(hide yes)
@@
 		)
 		(property "Value" "SolderJumper_2_Open"
-			(at 0 -1.9 90)
+			(at 0 -1.9 -90)
 			(layer "B.Fab")
-			(hide yes)
 			(effects
 				(font
@@
 			)
 		)
-		(property "Footprint" "Jumper:SolderJumper-2_P1.3mm_Open_RoundedPad1.0x1.5mm"
+		(property "Footprint" "Jumper:SolderJumper-2_P1.3mm_Bridged_RoundedPad1.0x1.5mm"
 			(at 0 0 -90)
 			(unlocked yes)
@@
 			)
 		)
-		(property "Description" "Solder Jumper, 2-pole, open"
+		(property "Description" "Solder Jumper, 2-pole, closed/bridged"
 			(at 0 0 -90)
 			(unlocked yes)
@@
 			)
 		)
-		(property ki_fp_filters "SolderJumper*Open*")
+		(property ki_fp_filters "SolderJumper*Bridged*")
 		(sheetname "Root")
 		(sheetfile "x1p-006.kicad_sch")
 		(zone_connect 1)
 		(attr exclude_from_pos_files exclude_from_bom dnp)
+		(net_tie_pad_groups "1, 2")
+		(fp_poly
+			(pts
+				(xy 0.25 0.3) (xy -0.25 0.3) (xy -0.25 -0.3) (xy 0.25 -0.3)
+			)
+			(stroke
+				(width 0)
+				(type solid)
+			)
+			(fill solid)
+			(layer "B.Cu")
+		)
 		(fp_line
 			(start -0.7 -1)
@@
 		)
 	)
-	(footprint "Jumper:SolderJumper-2_P1.3mm_Open_RoundedPad1.0x1.5mm"
+	(footprint "Jumper:SolderJumper-2_P1.3mm_Bridged_RoundedPad1.0x1.5mm"
 		(layer "B.Cu")
 		(at 161.6 79.8 90)
-		(descr "SMD Solder Jumper, 1x1.5mm, rounded Pads, 0.3mm gap, open")
-		(tags "solder jumper open")
+		(descr "SMD Solder Jumper, 1x1.5mm, rounded Pads, 0.3mm gap, bridged with 1 copper strip")
+		(tags "net tie solder jumper bridged")
 		(property "Reference" "JP4"
-			(at 0 1.8 90)
+			(at 0 1.8 -90)
 			(layer "B.SilkS")
 			(hide yes)
@@
 		)
 		(property "Value" "SolderJumper_2_Open"
-			(at 0 -1.9 90)
+			(at 0 -1.9 -90)
 			(layer "B.Fab")
-			(hide yes)
 			(effects
 				(font
@@
 			)
 		)
-		(property "Footprint" "Jumper:SolderJumper-2_P1.3mm_Open_RoundedPad1.0x1.5mm"
+		(property "Footprint" "Jumper:SolderJumper-2_P1.3mm_Bridged_RoundedPad1.0x1.5mm"
 			(at 0 0 -90)
 			(unlocked yes)
@@
 			)
 		)
-		(property "Description" "Solder Jumper, 2-pole, open"
+		(property "Description" "Solder Jumper, 2-pole, closed/bridged"
 			(at 0 0 -90)
 			(unlocked yes)
@@
 			)
 		)
-		(property ki_fp_filters "SolderJumper*Open*")
+		(property ki_fp_filters "SolderJumper*Bridged*")
 		(sheetname "Root")
 		(sheetfile "x1p-006.kicad_sch")
 		(zone_connect 1)
 		(attr exclude_from_pos_files exclude_from_bom dnp)
+		(net_tie_pad_groups "1, 2")
+		(fp_poly
+			(pts
+				(xy 0.25 0.3) (xy -0.25 0.3) (xy -0.25 -0.3) (xy 0.25 -0.3)
+			)
+			(stroke
+				(width 0)
+				(type solid)
+			)
+			(fill solid)
+			(layer "B.Cu")
+		)
 		(fp_line
 			(start -0.7 -1)
@@
 			)
 			(justify mirror)
+		)
+	)
+	(gr_text "T"
+		(at 142.6 83.6 0)
+		(layer "B.SilkS")
+		(effects
+			(font
+				(size 1 1)
+				(thickness 0.2)
+				(bold yes)
+			)
+			(justify mirror)
+		)
+	)
+	(gr_text "R"
+		(at 161.6 77.6 0)
+		(layer "B.SilkS")
+		(effects
+			(font
+				(size 1 1)
+				(thickness 0.2)
+				(bold yes)
+			)
+			(justify mirror)
+		)
+	)
+	(gr_text "R"
+		(at 146.4 77.6 0)
+		(layer "B.SilkS")
+		(effects
+			(font
+				(size 1 1)
+				(thickness 0.2)
+				(bold yes)
+			)
+			(justify mirror)
+		)
+	)
+	(gr_text "T"
+		(at 157.8 83.6 0)
+		(layer "B.SilkS")
+		(effects
+			(font
+				(size 1 1)
+				(thickness 0.2)
+				(bold yes)
+			)
+			(justify mirror)
