File: x1p-006/x1p-006.kicad_sch (KiCad schematic)
At the start: 18 parts, among them U1 AD24C02, U2 AQY212EHAX, U3 AQY212EHAX

Commit message: add King Credie recommended components, fix panel placement, fix pulldown on x1p-005, fix bridges on x1p-006
Parts:
- C1: MPN (none) -> CL05B104KB54PNC; Manufacturer (none) -> Samsung
- JP2, JP4: footprint Jumper:SolderJumper-2_P1.3mm_Open_RoundedPad1.0x1.5mm -> Jumper:SolderJumper-2_P1.3mm_Bridged_RoundedPad1.0x1.5mm; symbol Jumper:SolderJumper_2_Open -> Jumper:SolderJumper_2_Bridged
- R1, R2, R5, R6: MPN (none) -> RC0402FR-072K2L; Manufacturer (none) -> YAGEO
- R3, R4: MPN (none) -> RC0402FR-07220RL; Manufacturer (none) -> YAGEO
Changed lines of the file:
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@@
 			)
 		)
-		(property "MPN" ""
+		(property "MPN" "RC0402FR-07220RL"
 			(at 113.03 66.04 0)
 			(effects
@@
 			)
 		)
-		(property "Manufacturer" ""
+		(property "Manufacturer" "YAGEO"
 			(at 113.03 66.04 0)
 			(effects
@@
 	)
 	(symbol
-		(lib_id "Jumper:SolderJumper_2_Open")
+		(lib_id "Jumper:SolderJumper_2_Bridged")
 		(at 161.29 30.48 0)
 		(unit 1)
@@
 			)
 		)
-		(property "Footprint" "Jumper:SolderJumper-2_P1.3mm_Open_RoundedPad1.0x1.5mm"
+		(property "Footprint" "Jumper:SolderJumper-2_P1.3mm_Bridged_RoundedPad1.0x1.5mm"
 			(at 161.29 30.48 0)
 			(effects
@@
 			)
 		)
-		(property "Description" "Solder Jumper, 2-pole, open"
+		(property "Description" "Solder Jumper, 2-pole, closed/bridged"
 			(at 161.29 30.48 0)
 			(effects
@@
 			)
 		)
-		(property "MPN" ""
+		(property "MPN" "RC0402FR-072K2L"
 			(at 52.07 72.39 0)
 			(effects
@@
 			)
 		)
-		(property "Manufacturer" ""
+		(property "Manufacturer" "YAGEO"
 			(at 52.07 72.39 0)
 			(effects
@@
 			)
 		)
-		(property "MPN" ""
+		(property "MPN" "CL05B104KB54PNC"
 			(at 68.58 73.66 0)
 			(effects
@@
 			)
 		)
-		(property "Manufacturer" ""
+		(property "Manufacturer" "Samsung"
 			(at 68.58 73.66 0)
 			(effects
@@
 			)
 		)
-		(property "MPN" ""
+		(property "MPN" "RC0402FR-072K2L"
 			(at 102.87 58.42 0)
 			(effects
@@
 			)
 		)
-		(property "Manufacturer" ""
+		(property "Manufacturer" "YAGEO"
 			(at 102.87 58.42 0)
 			(effects
@@
 			)
 		)
-		(property "MPN" ""
+		(property "MPN" "RC0402FR-072K2L"
 			(at 102.87 33.02 0)
 			(effects
@@
 			)
 		)
-		(property "Manufacturer" ""
+		(property "Manufacturer" "YAGEO"
 			(at 102.87 33.02 0)
 			(effects
@@
 			)
 		)
-		(property "MPN" ""
+		(property "MPN" "RC0402FR-07220RL"
 			(at 113.03 40.64 0)
 			(effects
@@
 			)
 		)
-		(property "Manufacturer" ""
+		(property "Manufacturer" "YAGEO"
 			(at 113.03 40.64 0)
 			(effects
@@
 			)
 		)
-		(property "MPN" ""
+		(property "MPN" "RC0402FR-072K2L"
 			(at 44.45 72.39 0)
 			(effects
@@
 			)
 		)
-		(property "Manufacturer" ""
+		(property "Manufacturer" "YAGEO"
 			(at 44.45 72.39 0)
 			(effects
@@
 	)
 	(symbol
-		(lib_id "Jumper:SolderJumper_2_Open")
+		(lib_id "Jumper:SolderJumper_2_Bridged")
 		(at 161.29 55.88 0)
 		(unit 1)
@@
 			)
 		)
-		(property "Footprint" "Jumper:SolderJumper-2_P1.3mm_Open_RoundedPad1.0x1.5mm"
+		(property "Footprint" "Jumper:SolderJumper-2_P1.3mm_Bridged_RoundedPad1.0x1.5mm"
 			(at 161.29 55.88 0)
 			(effects
@@
 			)
 		)
-		(property "Description" "Solder Jumper, 2-pole, open"
+		(property "Description" "Solder Jumper, 2-pole, closed/bridged"
 			(at 161.29 55.88 0)
 			(effects
