File: x1p-005/x1p-005.kicad_pcb (KiCad board)
At the start: 2 copper layers, 26 x 61.8 mm, 72 parts, among them Q1 LMBT3904LT1G, SW1 6.0*6.0*6.0, SW2 6.0*6.0*6.0, U1 AD24C02, U2 SN74LVC1T45DBVR, U4 SN74LVC1G3157DBVR_C3040658, U5 SN74LVC1G3157DBVR_C3040658

Commit message: x1p-005: resistors to 2.2k; remove a weird dangling trace; label beepies and clickies with their pin number (#56)
* x1p-005: resistors to 2.2k; remove a weird dangling trace; label beepies and clickies with their pin number

* x1p-005: rotate r3 to "correct" orientation, add second thermal spoke back to buzzer
Parts:
- R1, R2, R5: value 3.3k -> 2.2k
- R3: value 3.3k -> 2.2k; footprint x1p-004:R0402 -> x1p-005:R0402
- turned R3 to 180 degrees
Connections:
- R3 pad 1: LD1 -> GND
- R3 pad 2: GND -> LD1
Routing:
- net 5V: track 61.2 -> 59.7 mm
Other:
- board text added: "IO3"
