File: x1p-005/x1p-005.kicad_pcb (KiCad board)
At the start: 2 copper layers, 20.8 x 61.8 mm, 40 parts, among them Q1 LMBT3904LT1G, SW1 6.0*6.0*6.0, SW2 6.0*6.0*6.0, U1 AD24C02, U2 SN74LVC1T45DBVR, U4 SN74LVC1G3157DBVR_C3040658, U5 SN74LVC1G3157DBVR_C3040658

Commit message: x1p-005-b01
Parts:
- removed R5: 1k, x1p-005:RES-ADJ-TH_3362P
- added H1: MountingHole, MountingHole:MountingHole_2.2mm_M2_ISO7380, F.Cu at (68.4, 74.0)
- added H2: MountingHole, MountingHole:MountingHole_2.2mm_M2_ISO7380, F.Cu at (75.8, 107.6)
- HDR1: value PM254-2-08-W-8.5 -> 220R-2*10P H=8.5MM Ytype Gold-plated black; footprint x1p-005:HDR-TH_16P-P2.54-H-F-R2-C8-W8.5 -> x1p-005:HDR-TH_20P-P2.54-H-F-R2-C10-S2.54-W10.2
Connections:
- HDR1 pad 1: GND -> unconnected-(HDR1-Pad1)
- HDR1 pad 10: LD4 -> 5V
- HDR1 pad 11: 3V3 -> unconnected-(HDR1-Pad11)
- HDR1 pad 12: LD5 -> 5V
- HDR1 pad 13: GND -> LD5
- HDR1 pad 14: LD6 -> 3V3
- HDR1 pad 15: GND -> LD6
- HDR1 pad 16: LD7 -> GND
- HDR1 pad 3: GND -> unconnected-(HDR1-Pad3)
- HDR1 pad 4: LD1 -> GND
- HDR1 pad 5: 3V3 -> LD1
- HDR1 pad 6: unconnected-(HDR1-Pad6) -> GND
- HDR1 pad 7: 5V -> unconnected-(HDR1-Pad7)
- HDR1 pad 8: unconnected-(HDR1-Pad8) -> 3V3
- HDR1 pad 9: 5V -> LD3
- Q1 pad 3: Net-(Q1-C) -> Net-(BUZZER1--)
- R6 pad 1: LD4 -> LD3
Routing:
- net Net-(BUZZER1--): track 24.0 -> 6.90 mm, vias 3 -> 0
- net LD4: track 12.9 -> 0.00 mm
- net LD3: track 0.00 -> 12.6 mm
- net Net-(R4-Pad2): track 56.9 -> 61.2 mm
- net Net-(Q1-C): track 2.52 -> 0.00 mm
- net 3V3: track 16.1 -> 18.3 mm, vias 5 -> 4
- net SDA: track 12.7 -> 11.1 mm
- net Net-(R7-Pad2): track 49.2 -> 50.2 mm
- net HD1: track 26.7 -> 27.6 mm
Other:
- board size 20.8 x 61.8 mm -> 26 x 61.8 mm
- board text added: "X1P-005-B01"
- board text removed: "X1P-005-A01"

Commit message: x1p-005-b01-fixes-1
Parts:
- removed R8: 10k, x1p-005:R0402
- added C15: 0.1uf, x1p-004:C0402, F.Cu at (58.6, 87.2)
- added C16: 0.1uf, x1p-004:C0402, F.Cu at (63.7, 87.2)
- added C17: 0.1uf, x1p-004:C0402, F.Cu at (68.8, 87.2)
- added C18: 0.1uf, x1p-004:C0402, F.Cu at (73.8, 87.2)
- added C19: 0.1uf, x1p-004:C0402, F.Cu at (78.9, 87.2)
- added C20: 0.1uf, x1p-004:C0402, F.Cu at (58.6, 92.3)
- added C21: 0.1uf, x1p-004:C0402, F.Cu at (63.7, 92.3)
- added C22: 0.1uf, x1p-004:C0402, F.Cu at (68.8, 92.3)
- added C23: 0.1uf, x1p-004:C0402, F.Cu at (73.8, 92.3)
- added C24: 0.1uf, x1p-004:C0402, F.Cu at (78.9, 92.3)
- added C25: 0.1uf, x1p-004:C0402, F.Cu at (58.6, 97.4)
- added C26: 0.1uf, x1p-004:C0402, F.Cu at (63.7, 97.4)
- added C27: 0.1uf, x1p-004:C0402, F.Cu at (68.8, 97.4)
- added C28: 0.1uf, x1p-004:C0402, F.Cu at (73.8, 97.4)
- added C29: 0.1uf, x1p-004:C0402, F.Cu at (78.9, 97.4)
- added LED10: XL-1615RGBC-WS2812B, x1p-005:LED-SMD_4P-L1.6-W1.5_XL-1615RGBC-WS2812B, F.Cu at (78.7, 84.5)
- added LED11: XL-1615RGBC-WS2812B, x1p-005:LED-SMD_4P-L1.6-W1.5_XL-1615RGBC-WS2812B, F.Cu at (58.4, 89.5)
- added LED12: XL-1615RGBC-WS2812B, x1p-005:LED-SMD_4P-L1.6-W1.5_XL-1615RGBC-WS2812B, F.Cu at (63.5, 89.5)
- added LED13: XL-1615RGBC-WS2812B, x1p-005:LED-SMD_4P-L1.6-W1.5_XL-1615RGBC-WS2812B, F.Cu at (68.5, 89.5)
- added LED14: XL-1615RGBC-WS2812B, x1p-005:LED-SMD_4P-L1.6-W1.5_XL-1615RGBC-WS2812B, F.Cu at (73.6, 89.5)
- added LED15: XL-1615RGBC-WS2812B, x1p-005:LED-SMD_4P-L1.6-W1.5_XL-1615RGBC-WS2812B, F.Cu at (78.7, 89.5)
- added LED16: XL-1615RGBC-WS2812B, x1p-005:LED-SMD_4P-L1.6-W1.5_XL-1615RGBC-WS2812B, F.Cu at (58.4, 94.6)
- added LED17: XL-1615RGBC-WS2812B, x1p-005:LED-SMD_4P-L1.6-W1.5_XL-1615RGBC-WS2812B, F.Cu at (63.5, 94.6)
- added LED18: XL-1615RGBC-WS2812B, x1p-005:LED-SMD_4P-L1.6-W1.5_XL-1615RGBC-WS2812B, F.Cu at (68.5, 94.6)
- added LED19: XL-1615RGBC-WS2812B, x1p-005:LED-SMD_4P-L1.6-W1.5_XL-1615RGBC-WS2812B, F.Cu at (73.6, 94.6)
- added LED20: XL-1615RGBC-WS2812B, x1p-005:LED-SMD_4P-L1.6-W1.5_XL-1615RGBC-WS2812B, F.Cu at (78.7, 94.6)
- added LED21: XL-1615RGBC-WS2812B, x1p-005:LED-SMD_4P-L1.6-W1.5_XL-1615RGBC-WS2812B, F.Cu at (58.4, 99.7)
- added LED22: XL-1615RGBC-WS2812B, x1p-005:LED-SMD_4P-L1.6-W1.5_XL-1615RGBC-WS2812B, F.Cu at (63.5, 99.7)
- added LED23: XL-1615RGBC-WS2812B, x1p-005:LED-SMD_4P-L1.6-W1.5_XL-1615RGBC-WS2812B, F.Cu at (68.5, 99.7)
- added LED24: XL-1615RGBC-WS2812B, x1p-005:LED-SMD_4P-L1.6-W1.5_XL-1615RGBC-WS2812B, F.Cu at (73.6, 99.7)
- added LED25: XL-1615RGBC-WS2812B, x1p-005:LED-SMD_4P-L1.6-W1.5_XL-1615RGBC-WS2812B, F.Cu at (78.7, 99.7)
- added R5: 3.3k, x1p-005:R0402, F.Cu at (71.8, 119.6)
- C1, C10, C11, C13, C14, C2, C3, C4, C5, C6, C7, C8, C9, Q1, R1, R2, R3, R4, R6, R7, U1, U2, U4, U5: moved to F.Cu
- C12: value 10uf -> 0.1uf; footprint x1p-005:C1206 -> x1p-004:C0402; moved to F.Cu
- LED1, LED2, LED3, LED4, LED5, LED6, LED7, LED8, LED9: value XL-5050RGBC-WS2812B -> XL-1615RGBC-WS2812B; footprint x1p-005:LED-SMD_4P-L5.0-W5.0-BL_XL-5050RGBC -> x1p-005:LED-SMD_4P-L1.6-W1.5_XL-1615RGBC-WS2812B
- moved R4 38.6 mm to (57.6, 74.6)
- moved R7 37.6 mm to (80.2, 74.2)
- moved C12 27.9 mm to (78.9, 82.1), turned to 180 degrees
- moved C5 20.6 mm to (68.7, 77.0), turned to 180 degrees
- moved C4 20.2 mm to (63.7, 77.0), turned to 180 degrees
- moved C3 19.9 mm to (58.6, 77.0), turned to 180 degrees
- moved LED3 19.6 mm to (68.5, 79.4)
- moved LED2 19.0 mm to (63.5, 79.4)
- moved LED1 18.5 mm to (58.4, 79.4)
- moved C6 18.2 mm to (73.8, 77.0), turned to 180 degrees
- moved LED6 17.8 mm to (58.4, 84.5)
- moved C8 16.9 mm to (58.6, 82.1), turned to 180 degrees
- moved C7 16.6 mm to (78.9, 77.0), turned to 180 degrees
- moved LED4 15.7 mm to (73.6, 79.4)
- moved LED5 14.1 mm to (78.7, 79.4)
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Connections:
- C12 pad 1: GND -> 5V
- C12 pad 2: 5V -> GND
- LED1 pad 1: 5V -> HD1
- LED1 pad 2: Net-(LED1-DOU) -> 5V
- LED1 pad 4: HD1 -> Net-(LED1-DI)
- LED2 pad 1: 5V -> Net-(LED1-DI)
- LED2 pad 2: Net-(LED2-DOU) -> 5V
- LED2 pad 4: Net-(LED1-DOU) -> Net-(LED2-DI)
- LED3 pad 1: 5V -> Net-(LED2-DI)
- LED3 pad 2: Net-(LED3-DOU) -> 5V
- LED3 pad 4: Net-(LED2-DOU) -> Net-(LED3-DI)
- LED4 pad 1: 5V -> Net-(LED3-DI)
- LED4 pad 2: Net-(LED4-DOU) -> 5V
- LED4 pad 4: Net-(LED3-DOU) -> Net-(LED4-DI)
- LED5 pad 1: 5V -> Net-(LED4-DI)
- LED5 pad 2: Net-(LED5-DOU) -> 5V
- LED5 pad 4: Net-(LED4-DOU) -> Net-(LED5-DI)
- LED6 pad 1: 5V -> Net-(LED5-DI)
- LED6 pad 2: Net-(LED6-DOU) -> 5V
- LED6 pad 4: Net-(LED5-DOU) -> Net-(LED6-DI)
- LED7 pad 1: 5V -> Net-(LED6-DI)
- LED7 pad 2: Net-(LED7-DOU) -> 5V
- LED7 pad 4: Net-(LED6-DOU) -> Net-(LED7-DI)
- LED8 pad 1: 5V -> Net-(LED7-DI)
- LED8 pad 2: Net-(LED8-DOU) -> 5V
- LED8 pad 4: Net-(LED7-DOU) -> Net-(LED8-DI)
- LED9 pad 1: 5V -> Net-(LED8-DI)
- LED9 pad 2: unconnected-(LED9-DOU-Pad2) -> 5V
- LED9 pad 4: Net-(LED8-DOU) -> Net-(LED10-DO)
Routing:
- net Net-(R4-Pad2): track 61.2 -> 1.57 mm, vias 3 -> 0
- net BTN1: track 1.48 -> 51.3 mm, vias 0 -> 4
- net Net-(R7-Pad2): track 50.2 -> 8.21 mm, vias 1 -> 0
- net BTN2: track 1.50 -> 37.2 mm, vias 0 -> 2
- net GND: track 33.3 -> 0.00 mm, vias 31 -> 0
- net 5V: track 29.7 -> 61.2 mm, vias 21 -> 26
- net Net-(LED3-DOU): track 28.8 -> 0.00 mm
- net Net-(LED6-DOU): track 28.7 -> 0.00 mm
- net Net-(LED5-DI): track 0.00 -> 24.6 mm, vias 0 -> 2
- net Net-(LED20-DI): track 0.00 -> 24.5 mm, vias 0 -> 2
- net Net-(LED15-DI): track 0.00 -> 24.5 mm, vias 0 -> 2
- net Net-(LED10-DI): track 0.00 -> 24.5 mm, vias 0 -> 2
- net SCL: track 12.9 -> 3.69 mm
- net HD1: track 27.6 -> 35.9 mm, vias 1 -> 0
- net Net-(LED7-DOU): track 6.74 -> 0.00 mm
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- removed copper zone on F.Cu, net 5V
- removed copper zone on B.Cu, net GND

Commit message: fix reversed di/do
Parts:
- moved C7 30.9 mm to (58.1, 100.0), turned to 0 degrees
- moved C3 30.3 mm to (78.5, 100.0), turned to 0 degrees
- moved LED25 30.3 mm to (58.3, 77.3), turned to 180 degrees
- moved LED21 30.2 mm to (78.7, 77.3), turned to 180 degrees
- moved LED5 27.3 mm to (58.3, 97.6), turned to 180 degrees
- moved C29 27.3 mm to (58.1, 79.7), turned to 0 degrees
- moved LED1 27.3 mm to (78.7, 97.6), turned to 180 degrees
- moved C25 26.6 mm to (78.5, 79.7), turned to 0 degrees
- moved C6 25.3 mm to (63.2, 100.0), turned to 0 degrees
- moved C4 24.9 mm to (73.4, 100.0), turned to 0 degrees
- moved LED24 24.6 mm to (63.4, 77.3), turned to 180 degrees
- moved LED22 24.6 mm to (73.6, 77.3), turned to 180 degrees
- moved C12 24.4 mm to (58.1, 94.9), turned to 0 degrees
- moved LED20 23.8 mm to (58.3, 82.4), turned to 180 degrees
- moved LED16 23.7 mm to (78.7, 82.4), turned to 180 degrees
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Connections:
- LED1 pad 1: HD1 -> unconnected-(LED1-DO-Pad1)
- LED25 pad 4: unconnected-(LED25-DI-Pad4) -> HD1
Routing:
- net HD1: track 35.9 -> 38.0 mm

Commit message: x1p-005: resistors to 2.2k; remove a weird dangling trace; label beepies and clickies with their pin number
Parts:
- R1, R2, R5: value 3.3k -> 2.2k
- R3: value 3.3k -> 2.2k; footprint x1p-004:R0402 -> x1p-005:R0402
Connections:
- R3 pad 1: LD1 -> GND
- R3 pad 2: GND -> LD1
Routing:
- net 5V: track 61.2 -> 58.2 mm
Other:
- board text added: "IO3"

Commit message: x1p-005: rotate r3 to "correct" orientation, add second thermal spoke back to buzzer
Parts:
- turned R3 to 180 degrees
Routing:
- net 5V: track 58.2 -> 59.7 mm
Changed lines of the file:
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@@
 			(pinfunction "+")
 			(pintype "unspecified")
+			(thermal_bridge_angle 90)
 		)
 		(pad "2" thru_hole circle
@@
 	(footprint "x1p-005:R0402"
 		(layer "F.Cu")
-		(at 61.17 115)
+		(at 61.17 115 180)
 		(property "Reference" "R3"
-			(at 0 -4 0)
+			(at 0 -4 360)
 			(layer "F.SilkS")
 			(hide yes)
@@
 		)
 		(property "Value" "2.2k"
-			(at 0 4 0)
+			(at 0 4 360)
 			(layer "F.Fab")
 			(hide yes)
@@
 		)
 		(property "Footprint" "x1p-005:R0402"
-			(at 0 0 0)
+			(at 0 0 360)
 			(layer "F.Fab")
 			(hide yes)
@@
 		)
 		(property "Datasheet" "https://lcsc.com/product-detail/Chip-Resistor-Surface-Mount-UniOhm_2-2KR-2201-1_C25879.html"
-			(at 0 0 0)
+			(at 0 0 360)
 			(layer "F.Fab")
 			(hide yes)
@@
 		)
 		(property "Description" ""
-			(at 0 0 0)
+			(at 0 0 360)
 			(layer "F.Fab")
 			(hide yes)
@@
 		)
 		(property "LCSC Part" "C25879"
-			(at 0 0 0)
+			(at 0 0 180)
 			(unlocked yes)
 			(layer "F.Fab")
@@
 		(attr smd)
 		(fp_line
-			(start -0.94 -0.5)
-			(end -0.23 -0.5)
+			(start 0.94 0.5)
+			(end 0.94 -0.5)
 			(stroke
 				(width 0.15)
@@
 		)
 		(fp_line
-			(start -0.94 0.5)
-			(end -0.94 -0.5)
+			(start 0.94 -0.5)
+			(end 0.23 -0.5)
 			(stroke
 				(width 0.15)
@@
 		)
 		(fp_line
-			(start -0.23 0.5)
-			(end -0.94 0.5)
+			(start 0.23 0.5)
+			(end 0.94 0.5)
 			(stroke
 				(width 0.15)
@@
 		)
 		(fp_line
-			(start 0.23 0.5)
-			(end 0.94 0.5)
+			(start -0.23 0.5)
+			(end -0.94 0.5)
 			(stroke
 				(width 0.15)
@@
 		)
 		(fp_line
-			(start 0.94 -0.5)
-			(end 0.23 -0.5)
+			(start -0.94 0.5)
+			(end -0.94 -0.5)
 			(stroke
 				(width 0.15)
@@
 		)
 		(fp_line
-			(start 0.94 0.5)
-			(end 0.94 -0.5)
+			(start -0.94 -0.5)
+			(end -0.23 -0.5)
 			(stroke
 				(width 0.15)
@@
 		)
 		(fp_text user "${REFERENCE}"
-			(at 0 0 0)
+			(at 0 0 360)
 			(layer "F.Fab")
 			(hide yes)
@@
 		)
 		(pad "1" smd rect
-			(at -0.43 0)
+			(at -0.43 0 180)
 			(size 0.57 0.54)
 			(layers "F.Cu" "F.Paste" "F.Mask")
@@
 		)
 		(pad "2" smd rect
-			(at 0.43 0)
+			(at 0.43 0 180)
 			(size 0.57 0.54)
 			(layers "F.Cu" "F.Paste" "F.Mask")
@@
 	(segment
 		(start 57.6 110.4)
-		(end 65.9 110.4)
+		(end 65.8 110.4)
 		(width 0.2)
 		(layer "B.Cu")
@@
 	)
 	(segment
+		(start 65.8 110.4)
+		(end 65.9 110.4)
+		(width 0.2)
+		(layer "B.Cu")
+		(net 1)
+	)
+	(segment
+		(start 65.8 110.4)
+		(end 67.3 110.4)
+		(width 0.2)
+		(layer "B.Cu")
+		(net 1)
+	)
+	(segment
 		(start 72.1 125.9)
 		(end 72.22 125.78)
@@
 		(polygon
 			(pts
-				(xy 65.6 102.6) (xy 71 102.6) (xy 71 126) (xy 65.6 126)
+				(xy 65.6 121.4) (xy 66.4 121.4) (xy 66.4 107.2) (xy 65.6 107.2) (xy 65.6 102.6) (xy 71 102.6) (xy 71 126)
+				(xy 65.6 126)
 			)
 		)

Commit message: add clearance for LEDs from mounting holes, return symmetry to zone fills
Parts:
- moved C10 0.92 mm to (68.3, 95.8)
- moved C11 0.92 mm to (63.2, 95.8)
- moved C12 0.92 mm to (58.1, 95.8)
- moved C15 0.92 mm to (78.5, 90.8)
- moved C16 0.92 mm to (73.4, 90.8)
- moved C17 0.92 mm to (68.3, 90.8)
- moved C18 0.92 mm to (63.2, 90.8)
- moved C19 0.92 mm to (58.1, 90.8)
- moved C20 0.92 mm to (78.5, 85.7)
- moved C21 0.92 mm to (73.4, 85.7)
- moved C22 0.92 mm to (68.3, 85.7)
- moved C23 0.92 mm to (63.2, 85.7)
- moved C24 0.92 mm to (58.1, 85.7)
- moved C25 0.92 mm to (78.5, 80.6)
- moved C26 0.92 mm to (73.4, 80.6)
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Routing:
- net BTN1: track 51.3 -> 53.9 mm
- net HD1: track 38.0 -> 37.0 mm
- net BTN2: track 37.2 -> 38.0 mm
Other:
- board text added: "SW1"
- board text added: "SW2"

Commit message: x1p-005: fix up board layout to align with x1p-004
Parts:
- C1, C13, C14: footprint x1p-005:C0402 -> Capacitor_SMD:C_0402_1005Metric
- C10, C11, C12, C15, C16, C17, C18, C19, C2, C20, C21, C22, C23, C24, C25, C26, C27, C28, C29, C3, C4, C5, C6, C7, C8, C9: footprint x1p-004:C0402 -> Capacitor_SMD:C_0402_1005Metric
- R1, R2, R3, R4, R5, R6, R7: footprint x1p-005:R0402 -> Resistor_SMD:R_0402_1005Metric
- moved H1 85.1 mm to (150.0, 50.0)
- moved SW1 84.7 mm to (143.0, 47.5)
- moved SW2 84.7 mm to (157.0, 47.5)
- moved R2 84.7 mm to (159.4, 97.0)
- moved C1 84.7 mm to (158.8, 81.8)
- moved C2 84.7 mm to (139.6, 86.4)
- moved HDR1 84.7 mm to (150.0, 100.0)
- moved Q1 84.7 mm to (143.2, 86.4)
- moved R4 84.7 mm to (139.2, 52.0)
- moved R6 84.7 mm to (144.2, 89.4)
- moved U1 84.7 mm to (158.4, 84.9)
- moved C14 84.7 mm to (160.8, 93.0)
- moved R1 84.7 mm to (156.8, 97.0)
- moved R3 84.7 mm to (142.8, 92.4)
- moved R5 84.7 mm to (153.4, 97.0)
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Routing:
- net GND: track 0.00 -> 3.10 mm
- net 3V3: track 23.5 -> 25.6 mm
Other:
- board size 26 x 61.8 mm -> 26.4 x 62 mm
- board text added: "X1P-005-B02"
- board text removed: "X1P-005-B01"

Commit message: reduce overall BOM on panels, load manufacturer and MPN in
Parts:
- C1, C10, C11, C12, C13, C14, C15, C16, C17, C18, C19, C2, C20, C21, C22, C23, C24, C25, C26, C27, C28, C29, C3, C4, C5, C6, C7, C8, C9: value 0.1uf -> 0.1uF
- HDR1: value 220R-2*10P H=8.5MM Ytype Gold-plated black -> B-2200R20P-B120
- R4, R7: value 330 -> 220
