File: x1p-005/x1p-005.kicad_sch (KiCad schematic)
At the start: 35 parts, among them Q1 LMBT3904LT1G, SW1 6.0*6.0*6.0, SW2 6.0*6.0*6.0, U1 AD24C02, U2 SN74LVC1T45DBVR

Commit message: pcb layout
Parts:
- removed C12: 10uf, x1p-005:CAP-SMD_BD6.3-L6.6-W6.6-LS7.6-FD, symbol Device:C_Polarized_Small_US
- added C12: 10uf, x1p-005:C1206, symbol x1p-005:CL31A106KBHNNNE
- added JP1: Jumper_2_Bridged, Jumper:SolderJumper-2_P1.3mm_Bridged_RoundedPad1.0x1.5mm, symbol Jumper:Jumper_2_Bridged
- added TP1, TP2: TestPoint, TestPoint:TestPoint_Pad_D2.0mm, symbol Connector:TestPoint
- U2: footprint x1p-004:SOT-23-6_L2.9-W1.6-P0.95-LS2.8-BR -> x1p-005:SOT-23-6_L2.9-W1.6-P0.95-LS2.8-BR
Connections:
- net 5V: now also C12.2
- net GND: now also C12.1
- net LD0: now also JP1.1 (A); no longer R3.1, U2.3 (A)
- net LD1: now also R3.1, U2.3 (A); no longer R6.1
- net LD4: now reaches HDR1.10
- net LD4: now also TP1.1
- net HD0 renamed HD1
- new net: JP1.2 (B), R6.1, TP2.1
- no-connect marks 8 -> 7
Other:
- moved on the sheet: BUZZER1, Q1, R5, R6

Commit message: add eeprom/switch mux, change buzzer
Parts:
- removed BUZZER1: QMB-09B-03, x1p-005:BUZ-TH_BD9.0-P4.00-D0.6-FD, symbol x1p-005:QMB-09B-03
- removed JP1: Jumper_2_Bridged, Jumper:SolderJumper-2_P1.3mm_Bridged_RoundedPad1.0x1.5mm, symbol Jumper:Jumper_2_Bridged
- removed R7, R8: 2.2k, x1p-005:R0402, symbol x1p-005:0402WGF2201TCE
- removed TP1, TP2: TestPoint, TestPoint:TestPoint_Pad_D2.0mm, symbol Connector:TestPoint
- added BUZZER1: HNB09A03, x1p-005:BUZ-TH_BD9.0-P5.00-D0.6-FD, symbol x1p-005:HNB09A03
- added C13, C14: 0.1uf, x1p-005:C0402, symbol lcsc:CL05B104KO5NNNC
- added R4, R7: 330, x1p-005:R0402, symbol x1p-005:0402WGF3300TCE
- added R8: 10k, x1p-005:R0402, symbol x1p-005:0402WGF1002TCE
- added U4, U5: SN74LVC1G3157DBVR_C3040658, x1p-005:SOT-23-6_L2.9-W1.6-P0.95-LS2.8-BL, symbol x1p-005:SN74LVC1G3157DBVR_C3040658
Connections:
- net VCC is gone; now on net 5V: U2.6 (VCCB)
- net 3V3: now also BUZZER1.1 (+), C13.1, C14.1, R8.2
- net 5V: now also U4.5 (VCC), U5.5 (VCC)
- net GND: now also SW1.4, SW2.4, C13.2, C14.2, U4.2 (GND), U5.2 (GND)
- net LD4: now also R6.1
- net LD6: now also U4.4 (A); no longer U1.3 (SDA)
- net LD7: now also U5.4 (A); no longer U1.1 (SCL)
- net at R5.3: now also BUZZER1.2 (-)
- net LD5: now reaches HDR1.12
- net LD5: now also R8.1, U4.6 (SEL), U5.6 (SEL)
- net at SW1.1: now also R4.2
- net at SW2.1: now also R7.2
- net LD0: no longer names the net of HDR1.2
- net LD2: no longer names the net of HDR1.6
- net LD2: no longer SW1.4
- net LD3: no longer names the net of HDR1.8
- net LD3: no longer SW2.4
- new net BTN1: R4.1, U4.1 (B1)
- new net BTN2: R7.1, U5.1 (B1)
- new net SCL: U1.1 (SCL), U5.3 (B0)
- new net SDA: U1.3 (SDA), U4.3 (B0)
- no-connect marks 7 -> 9
Other:
- note added: "EEPROM / Clicky Selector"
- note added: "LD5 hi EEPROM ena SW1/SW2 disa LD5 lo EEPROM disa SW1/SW2 ena"
- note added: "SN74LVC1G3157DBVR C3040658"
- moved on the sheet: Q1, R5, R6, SW1, SW2

Commit message: 0 drc violations \o/
Connections:
- net 3V3: now also U4.5 (VCC), U5.5 (VCC)
- net 5V: no longer U4.5 (VCC), U5.5 (VCC)
Changed lines of the file:
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@@
+		)
+	)
+	(global_label "3V3"
+		(shape input)
+		(at 58.42 111.76 0)
+		(fields_autoplaced yes)
+		(effects
+			(font
+				(size 1.27 1.27)
+			)
+			(justify left)
+		)
+		(property "Intersheetrefs" "${INTERSHEET_REFS}"
+			(at 64.9128 111.76 0)
+			(effects
+				(font
+					(size 1.27 1.27)
+				)
+				(justify left)
+				(hide yes)
+			)
 		)
 	)
@@
 		)
 	)
-	(global_label "5V"
+	(global_label "3V3"
+		(shape input)
+		(at 48.26 97.79 90)
+		(fields_autoplaced yes)
+		(effects
+			(font
+				(size 1.27 1.27)
+			)
+			(justify left)
+		)
+		(property "Intersheetrefs" "${INTERSHEET_REFS}"
+			(at 48.26 91.2972 90)
+			(effects
+				(font
+					(size 1.27 1.27)
+				)
+				(justify left)
+				(hide yes)
+			)
+		)
+	)
+	(global_label "GND"
+		(shape input)
+		(at 129.54 30.48 270)
+		(fields_autoplaced yes)
+		(effects
+			(font
+				(size 1.27 1.27)
+			)
+			(justify right)
+		)
+		(property "Intersheetrefs" "${INTERSHEET_REFS}"
+			(at 129.54 37.3357 90)
+			(effects
+				(font
+					(size 1.27 1.27)
+				)
+				(justify right)
+				(hide yes)
+			)
+		)
+	)
+	(global_label "GND"
+		(shape input)
+		(at 34.29 43.18 180)
+		(fields_autoplaced yes)
+		(effects
+			(font
+				(size 1.27 1.27)
+			)
+			(justify right)
+		)
+		(property "Intersheetrefs" "${INTERSHEET_REFS}"
+			(at 27.4343 43.18 0)
+			(effects
+				(font
+					(size 1.27 1.27)
+				)
+				(justify right)
+				(hide yes)
+			)
+		)
+	)
+	(global_label "3V3"
 		(shape input)
 		(at 58.42 124.46 0)
@@
 		)
 		(property "Intersheetrefs" "${INTERSHEET_REFS}"
-			(at 63.7033 124.46 0)
-			(effects
-				(font
-					(size 1.27 1.27)
-				)
-				(justify left)
-				(hide yes)
-			)
-		)
-	)
-	(global_label "3V3"
-		(shape input)
-		(at 48.26 97.79 90)
-		(fields_autoplaced yes)
-		(effects
-			(font
-				(size 1.27 1.27)
-			)
-			(justify left)
-		)
-		(property "Intersheetrefs" "${INTERSHEET_REFS}"
-			(at 48.26 91.2972 90)
-			(effects
-				(font
-					(size 1.27 1.27)
-				)
-				(justify left)
-				(hide yes)
-			)
-		)
-	)
-	(global_label "GND"
-		(shape input)
-		(at 129.54 30.48 270)
-		(fields_autoplaced yes)
-		(effects
-			(font
-				(size 1.27 1.27)
-			)
-			(justify right)
-		)
-		(property "Intersheetrefs" "${INTERSHEET_REFS}"
-			(at 129.54 37.3357 90)
-			(effects
-				(font
-					(size 1.27 1.27)
-				)
-				(justify right)
-				(hide yes)
-			)
-		)
-	)
-	(global_label "GND"
-		(shape input)
-		(at 34.29 43.18 180)
-		(fields_autoplaced yes)
-		(effects
-			(font
-				(size 1.27 1.27)
-			)
-			(justify right)
-		)
-		(property "Intersheetrefs" "${INTERSHEET_REFS}"
-			(at 27.4343 43.18 0)
-			(effects
-				(font
-					(size 1.27 1.27)
-				)
-				(justify right)
-				(hide yes)
-			)
-		)
-	)
-	(global_label "5V"
-		(shape input)
-		(at 58.42 111.76 0)
-		(fields_autoplaced yes)
-		(effects
-			(font
-				(size 1.27 1.27)
-			)
-			(justify left)
-		)
-		(property "Intersheetrefs" "${INTERSHEET_REFS}"
-			(at 63.7033 111.76 0)
-			(effects
-				(font
+			(at 64.9128 124.46 0)
+			(effects
+				(font

Commit message: x1p-005-b01
Parts:
- removed HDR1: PM254-2-08-W-8.5, x1p-005:HDR-TH_16P-P2.54-H-F-R2-C8-W8.5, symbol lcsc:PM254-2-08-W-8.5
- removed R5: 1k, x1p-005:RES-ADJ-TH_3362P, symbol x1p-005:3362P-1-102
- added H1, H2: MountingHole, MountingHole:MountingHole_2.2mm_M2_ISO7380, symbol Mechanical:MountingHole
- added HDR1: 220R-2*10P H=8.5MM Ytype Gold-plated black, x1p-005:HDR-TH_20P-P2.54-H-F-R2-C10-S2.54-W10.2, symbol x1p-006:220R-2*10PH=8.5MMYtypeGold-platedblack
Connections:
- net 3V3: now also HDR1.14, HDR1.8
- net 5V: now also HDR1.10, HDR1.12
- net GND: now also HDR1.16, HDR1.18, HDR1.4, HDR1.6
- net LD1: now also HDR1.5
- net LD5: now also HDR1.13
- net LD6: now also HDR1.15
- net LD7: now also HDR1.17
- net at Q1.3 (C): now also BUZZER1.2 (-)
- net LD4 renamed LD3
- net LD3: now also HDR1.9
- no-connect marks 9 -> 12
Other:
- note removed: "Volume Control"

Commit message: x1p-005-b01-fixes-1
Parts:
- removed C12: 10uf, x1p-005:C1206, symbol x1p-005:CL31A106KBHNNNE
- removed LED1, LED2, LED3, LED4, LED5, LED6, LED7, LED8, LED9: XL-5050RGBC-WS2812B, x1p-005:LED-SMD_4P-L5.0-W5.0-BL_XL-5050RGBC, symbol x1p-005:XL-5050RGBC-WS2812B
- removed R8: 10k, x1p-005:R0402, symbol x1p-005:0402WGF1002TCE
- added C12, C15, C16, C17, C18, C19, C20, C21, C22, C23, C24, C25, C26, C27, C28, C29: 0.1uf, x1p-004:C0402, symbol lcsc:CL05B104KO5NNNC
- added LED1, LED10, LED11, LED12, LED13, LED14, LED15, LED16, LED17, LED18, LED19, LED2, LED20, LED21, LED22, LED23, LED24, LED25, LED3, LED4, LED5, LED6, LED7, LED8, LED9: XL-1615RGBC-WS2812B, x1p-005:LED-SMD_4P-L1.6-W1.5_XL-1615RGBC-WS2812B, symbol x1p-005:XL-1615RGBC-WS2812B
- added R5: 3.3k, x1p-005:R0402, symbol lcsc:0402WGF3301TCE
Connections:
- net 5V: now also C12.1, C15.1, C16.1, C17.1, C18.1, C19.1, C20.1, C21.1, C22.1, C23.1, C24.1, C25.1, C26.1, C27.1, C28.1, C29.1, LED1.2 (VDD), LED10.2 (VDD), LED11.2 (VDD), LED12.2 (VDD), LED13.2 (VDD), LED14.2 (VDD), LED15.2 (VDD), LED16.2 (VDD), LED17.2 (VDD), LED18.2 (VDD), LED19.2 (VDD), LED2.2 (VDD), LED20.2 (VDD), LED21.2 (VDD), LED22.2 (VDD), LED23.2 (VDD), LED24.2 (VDD), LED25.2 (VDD), LED3.2 (VDD), LED4.2 (VDD), LED5.2 (VDD), LED6.2 (VDD), LED7.2 (VDD), LED8.2 (VDD), LED9.2 (VDD)
- net GND: now also C12.2, C15.2, C16.2, C17.2, C18.2, C19.2, C20.2, C21.2, C22.2, C23.2, C24.2, C25.2, C26.2, C27.2, C28.2, C29.2, LED1.3 (GND), LED10.3 (GND), LED11.3 (GND), LED12.3 (GND), LED13.3 (GND), LED14.3 (GND), LED15.3 (GND), LED16.3 (GND), LED17.3 (GND), LED18.3 (GND), LED19.3 (GND), LED2.3 (GND), LED20.3 (GND), LED21.3 (GND), LED22.3 (GND), LED23.3 (GND), LED24.3 (GND), LED25.3 (GND), LED3.3 (GND), LED4.3 (GND), LED5.3 (GND), LED6.3 (GND), LED7.3 (GND), LED8.3 (GND), LED9.3 (GND), R5.1
- net HD1: now also LED1.1 (DO)
- net LD5: now also R5.2
- new net: LED16.4 (DI), LED17.1 (DO)
- new net: LED17.4 (DI), LED18.1 (DO)
- new net: LED1.4 (DI), LED2.1 (DO)
- new net: LED15.4 (DI), LED16.1 (DO)
- new net: LED24.4 (DI), LED25.1 (DO)
- new net: LED6.4 (DI), LED7.1 (DO)
- new net: LED7.4 (DI), LED8.1 (DO)
- new net: LED4.4 (DI), LED5.1 (DO)
- new net: LED5.4 (DI), LED6.1 (DO)
- new net: LED12.4 (DI), LED13.1 (DO)
- new net: LED13.4 (DI), LED14.1 (DO)
- new net: LED18.4 (DI), LED19.1 (DO)
- new net: LED10.1 (DO), LED9.4 (DI)
- new net: LED10.4 (DI), LED11.1 (DO)
- new net: LED3.4 (DI), LED4.1 (DO)
- new net: LED19.4 (DI), LED20.1 (DO)
- new net: LED14.4 (DI), LED15.1 (DO)
- new net: LED22.4 (DI), LED23.1 (DO)
- new net: LED23.4 (DI), LED24.1 (DO)
- new net: LED20.4 (DI), LED21.1 (DO)
- new net: LED21.4 (DI), LED22.1 (DO)
- new net: LED11.4 (DI), LED12.1 (DO)
- new net: LED8.4 (DI), LED9.1 (DO)
- new net: LED2.4 (DI), LED3.1 (DO)
- no-connect marks 12 -> 11
Other:
- note added: "25 x 20mA = 500mA"
- note added: "LD5 lo EEPROM ena SW1/SW2 disa LD5 hi EEPROM disa SW1/SW2 ena"
- note added: "XL-1615RGBC-WS2812B"
- note removed: "9 x 20mA = 180mA"
- note removed: "LD5 hi EEPROM ena SW1/SW2 disa LD5 lo EEPROM disa SW1/SW2 ena"
- note removed: "SN74LVC1G3157DBVR C3040658"
- note removed: "XL-5050RGBC-WS2812B"
- moved on the sheet: C13, C14, R1, R2, R3, U2, U4, U5

Commit message: fix reversed di/do
Connections:
- net HD1: now also LED25.4 (DI); no longer LED1.1 (DO)
Changed lines of the file:
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@@
-		)
-	)
-	(global_label "HD1"
-		(shape input)
-		(at 168.91 31.75 180)
-		(fields_autoplaced yes)
-		(effects
-			(font
-				(size 1.27 1.27)
-			)
-			(justify right)
-		)
-		(property "Intersheetrefs" "${INTERSHEET_REFS}"
-			(at 162.1148 31.75 0)
-			(effects
-				(font
-					(size 1.27 1.27)
-				)
-				(justify right)
-				(hide yes)
-			)
 		)
 	)
@@
 				(hide yes)
 			)
+		)
+	)
+	(global_label "HD1"
+		(shape input)
+		(at 267.97 120.65 0)
+		(fields_autoplaced yes)
+		(effects
+			(font
+				(size 1.27 1.27)
+			)
+			(justify left)
+		)
+		(property "Intersheetrefs" "${INTERSHEET_REFS}"
+			(at 274.7652 120.65 0)
+			(effects
+				(font
+					(size 1.27 1.27)
+				)
+				(justify left)
+				(hide yes)
+			)

Commit message: x1p-005: resistors to 2.2k; remove a weird dangling trace; label beepies and clickies with their pin number
Parts:
- removed R1, R2, R5: 3.3k, x1p-005:R0402, symbol lcsc:0402WGF3301TCE
- removed R3: 3.3k, x1p-004:R0402, symbol lcsc:0402WGF3301TCE
- added R1, R2, R3, R5: 2.2k, x1p-005:R0402, symbol x1p-005:0402WGF2201TCE
Connections:
- net 3V3: now also R1.2, R2.2
- net GND: now also R3.1, R5.1
- net LD1: now also R3.2
- net LD5: now also R5.2
- net LD6: now also R1.1
- net LD7: now also R2.1

Commit message: x1p-005: fix up board layout to align with x1p-004
Parts:
- C1, C13, C14: footprint x1p-005:C0402 -> Capacitor_SMD:C_0402_1005Metric
- C10, C11, C12, C15, C16, C17, C18, C19, C2, C20, C21, C22, C23, C24, C25, C26, C27, C28, C29, C3, C4, C5, C6, C7, C8, C9: footprint x1p-004:C0402 -> Capacitor_SMD:C_0402_1005Metric
- R1, R2, R3, R4, R5, R6, R7: footprint x1p-005:R0402 -> Resistor_SMD:R_0402_1005Metric
Changed lines of the file:
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@@
 			)
 		)
-		(property "Footprint" "x1p-004:C0402"
+		(property "Footprint" "Capacitor_SMD:C_0402_1005Metric"
 			(at 204.47 137.16 0)
 			(effects
@@
 			)
 		)
-		(property "Footprint" "x1p-005:C0402"
+		(property "Footprint" "Capacitor_SMD:C_0402_1005Metric"
 			(at 19.05 101.6 0)
 			(effects
@@
 			)
 		)
-		(property "Footprint" "x1p-004:C0402"
+		(property "Footprint" "Capacitor_SMD:C_0402_1005Metric"
 			(at 247.65 137.16 0)
 			(effects
@@
 			)
 		)
-		(property "Footprint" "x1p-004:C0402"
+		(property "Footprint" "Capacitor_SMD:C_0402_1005Metric"
 			(at 166.37 137.16 0)
 			(effects
@@
 			)
 		)
-		(property "Footprint" "x1p-004:C0402"
+		(property "Footprint" "Capacitor_SMD:C_0402_1005Metric"
 			(at 166.37 149.86 0)
 			(effects
@@
 			)
 		)
-		(property "Footprint" "x1p-005:R0402"
+		(property "Footprint" "Resistor_SMD:R_0402_1005Metric"
 			(at 82.55 132.08 0)
 			(effects
@@
 			)
 		)
-		(property "Footprint" "x1p-004:C0402"
+		(property "Footprint" "Capacitor_SMD:C_0402_1005Metric"
 			(at 220.98 137.16 0)
 			(effects
@@
 			)
 		)
-		(property "Footprint" "x1p-004:C0402"
+		(property "Footprint" "Capacitor_SMD:C_0402_1005Metric"
 			(at 121.92 26.67 0)
 			(effects
@@
 			)
 		)
-		(property "Footprint" "x1p-004:C0402"
+		(property "Footprint" "Capacitor_SMD:C_0402_1005Metric"
 			(at 247.65 149.86 0)
 			(effects
@@
 			)
 		)
-		(property "Footprint" "x1p-005:R0402"
+		(property "Footprint" "Resistor_SMD:R_0402_1005Metric"
 			(at 92.71 41.91 0)
 			(effects
@@
 			)
 		)
-		(property "Footprint" "x1p-004:C0402"
+		(property "Footprint" "Capacitor_SMD:C_0402_1005Metric"
 			(at 189.23 137.16 0)
 			(effects
@@
 			)
 		)
-		(property "Footprint" "x1p-004:C0402"
+		(property "Footprint" "Capacitor_SMD:C_0402_1005Metric"
 			(at 256.54 149.86 0)
 			(effects
@@
 			)
 		)
-		(property "Footprint" "x1p-005:R0402"
+		(property "Footprint" "Resistor_SMD:R_0402_1005Metric"
 			(at 76.2 101.6 0)
 			(effects
@@
 			)
 		)
-		(property "Footprint" "x1p-004:C0402"
+		(property "Footprint" "Capacitor_SMD:C_0402_1005Metric"
 			(at 181.61 137.16 0)
 			(effects
@@
 			)
 		)
-		(property "Footprint" "x1p-005:R0402"
+		(property "Footprint" "Resistor_SMD:R_0402_1005Metric"
 			(at 107.95 137.16 0)
 			(effects
@@
 			)
 		)
-		(property "Footprint" "x1p-004:C0402"
+		(property "Footprint" "Capacitor_SMD:C_0402_1005Metric"
 			(at 220.98 149.86 0)
 			(effects
@@
 			)
 		)
-		(property "Footprint" "x1p-005:C0402"
+		(property "Footprint" "Capacitor_SMD:C_0402_1005Metric"
 			(at 10.16 101.6 0)
 			(effects
@@
 			)
 		)
-		(property "Footprint" "x1p-004:C0402"
+		(property "Footprint" "Capacitor_SMD:C_0402_1005Metric"
 			(at 158.75 149.86 0)
 			(effects
@@
 			)
 		)
-		(property "Footprint" "x1p-004:C0402"
+		(property "Footprint" "Capacitor_SMD:C_0402_1005Metric"
 			(at 189.23 149.86 0)
 			(effects
@@
 			)
 		)
-		(property "Footprint" "x1p-005:C0402"
+		(property "Footprint" "Capacitor_SMD:C_0402_1005Metric"
 			(at 48.26 68.58 0)
 			(effects
@@
 			)
 		)
-		(property "Footprint" "x1p-004:C0402"
+		(property "Footprint" "Capacitor_SMD:C_0402_1005Metric"
 			(at 204.47 149.86 0)
 			(effects
@@
 			)
 		)
-		(property "Footprint" "x1p-004:C0402"
+		(property "Footprint" "Capacitor_SMD:C_0402_1005Metric"
 			(at 212.09 137.16 0)
 			(effects
@@
 			)
 		)
-		(property "Footprint" "x1p-004:C0402"
+		(property "Footprint" "Capacitor_SMD:C_0402_1005Metric"
 			(at 212.09 149.86 0)
 			(effects
@@
 			)
 		)
-		(property "Footprint" "x1p-004:C0402"
+		(property "Footprint" "Capacitor_SMD:C_0402_1005Metric"
 			(at 238.76 149.86 0)
 			(effects
@@
 			)
 		)
-		(property "Footprint" "x1p-005:R0402"
+		(property "Footprint" "Resistor_SMD:R_0402_1005Metric"
 			(at 105.41 95.25 0)
 			(effects
@@
 			)
 		)
-		(property "Footprint" "x1p-004:C0402"
+		(property "Footprint" "Capacitor_SMD:C_0402_1005Metric"
 			(at 196.85 149.86 0)
 			(effects
@@
 			)
 		)
-		(property "Footprint" "x1p-004:C0402"
+		(property "Footprint" "Capacitor_SMD:C_0402_1005Metric"
 			(at 181.61 149.86 0)
 			(effects
@@
 			)
 		)
-		(property "Footprint" "x1p-005:R0402"
+		(property "Footprint" "Resistor_SMD:R_0402_1005Metric"
 			(at 68.58 101.6 0)
 			(effects
@@
 			)
 		)
-		(property "Footprint" "x1p-004:C0402"
+		(property "Footprint" "Capacitor_SMD:C_0402_1005Metric"
 			(at 229.87 137.16 0)
 			(effects
@@
 			)
 		)
-		(property "Footprint" "x1p-005:R0402"
+		(property "Footprint" "Resistor_SMD:R_0402_1005Metric"
 			(at 107.95 121.92 0)
 			(effects
@@
 			)
 		)
-		(property "Footprint" "x1p-004:C0402"
+		(property "Footprint" "Capacitor_SMD:C_0402_1005Metric"
 			(at 196.85 137.16 0)
 			(effects
@@
 			)
 		)
-		(property "Footprint" "x1p-004:C0402"
+		(property "Footprint" "Capacitor_SMD:C_0402_1005Metric"
 			(at 238.76 137.16 0)
 			(effects
@@
 			)
 		)
-		(property "Footprint" "x1p-004:C0402"
+		(property "Footprint" "Capacitor_SMD:C_0402_1005Metric"
 			(at 173.99 149.86 0)
 			(effects
@@
 			)
 		)
-		(property "Footprint" "x1p-004:C0402"
+		(property "Footprint" "Capacitor_SMD:C_0402_1005Metric"
 			(at 158.75 137.16 0)
 			(effects
@@
 			)
 		)
-		(property "Footprint" "x1p-004:C0402"
+		(property "Footprint" "Capacitor_SMD:C_0402_1005Metric"
 			(at 173.99 137.16 0)
 			(effects
@@
 			)
 		)
-		(property "Footprint" "x1p-004:C0402"
+		(property "Footprint" "Capacitor_SMD:C_0402_1005Metric"
 			(at 229.87 149.86 0)
 			(effects
