File: x1p-005/x1p-005.kicad_sch (KiCad schematic)
At the start: 72 parts, among them Q1 LMBT3904LT1G, SW1 6.0*6.0*6.0, SW2 6.0*6.0*6.0, U1 AD24C02, U2 SN74LVC1T45DBVR, U4 SN74LVC1G3157DBVR_C3040658, U5 SN74LVC1G3157DBVR_C3040658

Commit message: reduce overall BOM on panels, load manufacturer and MPN in
Parts:
- BUZZER1: MPN (none) -> HNB09A03; Manufacturer (none) -> Jiangsu Huaneng Electronics
- C1, C10, C11, C12, C13, C14, C15, C16, C17, C18, C19, C2, C20, C21, C22, C23, C24, C25, C26, C27, C28, C29, C3, C4, C5, C6, C7, C8, C9: value 0.1uf -> 0.1uF
- H1, H2: now not fitted
- HDR1: value 220R-2*10P H=8.5MM Ytype Gold-plated black -> B-2200R20P-B120; MPN (none) -> B-2200R20P-B120; Manufacturer (none) -> CKMTW
- LED1, LED10, LED11, LED12, LED13, LED14, LED15, LED16, LED17, LED18, LED19, LED2, LED20, LED21, LED22, LED23, LED24, LED25, LED3, LED4, LED5, LED6, LED7, LED8, LED9: MPN (none) -> XL-1615RGBC-WS2812B; Manufacturer (none) -> XINGLIGHT
- Q1: MPN (none) -> LMBT3904LT1G; Manufacturer (none) -> LRC
- R4, R7: value 330 -> 220; LCSC Part C25104 -> C25091
- SW1, SW2: MPN (none) -> 6.0*6.0*6.0; Manufacturer (none) -> BOOMELE
- U1: MPN (none) -> AD24C02; Manufacturer (none) -> IDCHIP
- U2: MPN (none) -> SN74LVC1T45DBVR; Manufacturer (none) -> Texas Instruments
- U4, U5: MPN (none) -> SN74LVC1G3157DBVR(UMW); Manufacturer (none) -> UMW

Commit message: add King Credie recommended components, fix panel placement, fix pulldown on x1p-005, fix bridges on x1p-006
Parts:
- added R8: 2.2k, Resistor_SMD:R_0402_1005Metric, symbol x1p-005:0402WGF2201TCE
- C1, C10, C11, C12, C13, C14, C15, C16, C17, C18, C19, C2, C20, C21, C22, C23, C24, C25, C26, C27, C28, C29, C3, C4, C5, C6, C7, C8, C9: MPN (none) -> CL05B104KB54PNC; Manufacturer (none) -> Samsung
- R1, R2, R3, R5, R6: MPN (none) -> RC0402FR-072K2L; Manufacturer (none) -> Yageo
- R4, R7: MPN (none) -> RC0402FR-07220RL; Manufacturer (none) -> Yageo
Connections:
- net GND: now also R8.2
- net LD3: now also R8.1
