File: x1p-003/x1p-003.kicad_pcb (KiCad board)
At the start: 4 copper layers, 180 x 109 mm, 50 parts, among them J10 24.243.1 Red, J11 24.243.2 Black, J9 Amphenol 10103594-0001LF, Q1 AO3400A, U1 INA219AxD, U2 INA219AxD, U3 INA219AxD, U4 PCA9536D,118, U5 TPS7A7002DDAR, U6 TPS7A7002DDAR

Commit message: X1P-003-A01 release
Parts:
- removed the G*** at (197.9, 122.6)
- moved R10 106.0 mm to (171.5, 141.5), turned to -90 degrees
- moved R11 105.5 mm to (246.2, 67.0), turned to 90 degrees
- moved G*** 6.90 mm to (197.0, 122.6)
- moved C11 0.90 mm to (172.8, 136.5), turned to -90 degrees
- moved C10 0.65 mm to (240.5, 63.0)
Connections:
- D1 pad 2: +5V -> /5V_LOAD
Routing:
- net +3.3V: track 0.00 -> 268.2 mm, vias 0 -> 7
- net /SCL: track 0.00 -> 258.8 mm, vias 0 -> 2
- net /SDA: track 0.00 -> 246.1 mm, vias 0 -> 2
- net /3V3_LOAD_EN: track 0.00 -> 98.0 mm
- net /5V_LOAD: track 0.00 -> 94.6 mm, vias 0 -> 2
- net /USB_DP: track 0.00 -> 69.9 mm
- net /USB_DN: track 0.00 -> 68.7 mm
- net /24V_DUT: track 0.00 -> 60.3 mm
- net +5V: track 0.00 -> 36.5 mm
- net /5V_LOAD_EN: track 0.00 -> 33.9 mm
- net +24V: track 0.00 -> 29.8 mm
- net /LED_FAIL: track 0.00 -> 20.7 mm
- net GND: track 0.00 -> 20.6 mm, vias 0 -> 48
- net /3V3_LOAD: track 0.00 -> 20.5 mm
- net /LED_PASS: track 0.00 -> 18.7 mm
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- added copper zone on B.Cu, net GND
- added copper zone on F.Cu, net GND
Other:
- outline, holes or cut-outs redrawn
- copper layers 4 -> 2
- board text removed: "SCL"
- board text removed: "TODO: LONGER GROUND POGO SHORTER 24V POGO"
