File: x1p-003/x1p-003.kicad_sch (KiCad schematic)
At the start: 44 parts, among them J1 24V, J10 24.243.2 Black, J2 5V, J3 3.3V, J4 D+, J5 D-, J6 GND, J7 SCL, J8 SDA, J9 24.243.1 Red, J9 USB_B_Micro, U1 INA219AxD, U2 INA219AxD, U3 INA219AxD, U4 PCA9536D,118, U5 TPS7A7002DDAR, U6 TPS7A7002DDAR

Commit message: fix annotation error
Parts:
- renumbered J9 to J10, J10 to J11
Connections:
- no-connect marks 3 -> 4
Changed lines of the file:
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@@
 		(at 123.19 43.18)
 	)
+	(no_connect
+		(at 123.19 53.34)
+	)
 	(wire
 		(pts
@@
 		(dnp no)
 		(fields_autoplaced yes)
-		(property "Reference" "J10"
+		(property "Reference" "J11"
 			(at 121.92 91.4399 0)
 			(effects
@@
 			(project "x1p-003"
 				(path "/9d65e234-c9ea-4162-90c2-0a323aa2325b"
-					(reference "J10")
+					(reference "J11")
 					(unit 1)
 				)
@@
 		(dnp no)
 		(fields_autoplaced yes)
-		(property "Reference" "J9"
+		(property "Reference" "J10"
 			(at 121.92 77.4699 0)
 			(effects
@@
 			(project "x1p-003"
 				(path "/9d65e234-c9ea-4162-90c2-0a323aa2325b"
-					(reference "J9")
+					(reference "J10")
 					(unit 1)
 				)

Commit message: x1p-003: add pogo pin step file and assign a few footprints
Parts:
- C1, C10, C11, C12, C2, C3, C4, C5, C6, C7, C8, C9: footprint (none) -> Capacitor_SMD:C_0603_1608Metric
- J1, J2, J3, J4, J5, J6, J7, J8: footprint (none) -> x1p-003:Pogo_Drill_0.9mm__Pad_2.0mm
- R10, R11: footprint (none) -> Resistor_SMD:R_1210_3225Metric
- R12, R13, R2, R3, R5, R6, R8, R9: footprint (none) -> Resistor_SMD:R_0603_1608Metric
Changed lines of the file:
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@@
 			)
 		)
-		(property "Footprint" ""
+		(property "Footprint" "Capacitor_SMD:C_0603_1608Metric"
 			(at 238.76 109.22 0)
 			(effects
@@
 			)
 		)
-		(property "Footprint" ""
+		(property "Footprint" "Capacitor_SMD:C_0603_1608Metric"
 			(at 27.94 139.7 0)
 			(effects
@@
 			)
 		)
-		(property "Footprint" ""
+		(property "Footprint" "Resistor_SMD:R_0603_1608Metric"
 			(at 226.06 158.75 0)
 			(effects
@@
 			)
 		)
-		(property "Footprint" ""
+		(property "Footprint" "Capacitor_SMD:C_0603_1608Metric"
 			(at 43.18 177.8 0)
 			(effects
@@
 			)
 		)
-		(property "Footprint" ""
+		(property "Footprint" "Capacitor_SMD:C_0603_1608Metric"
 			(at 245.11 52.07 0)
 			(effects
@@
 			)
 		)
-		(property "Footprint" ""
+		(property "Footprint" "x1p-003:Pogo_Drill_0.9mm__Pad_2.0mm"
 			(at 40.64 74.93 0)
 			(effects
@@
 			)
 		)
-		(property "Footprint" ""
+		(property "Footprint" "Capacitor_SMD:C_0603_1608Metric"
 			(at 48.26 139.7 0)
 			(effects
@@
 			)
 		)
-		(property "Footprint" ""
+		(property "Footprint" "x1p-003:Pogo_Drill_0.9mm__Pad_2.0mm"
 			(at 40.64 44.45 0)
 			(effects
@@
 			)
 		)
-		(property "Footprint" ""
+		(property "Footprint" "x1p-003:Pogo_Drill_0.9mm__Pad_2.0mm"
 			(at 40.64 67.31 0)
 			(effects
@@
 			)
 		)
-		(property "Footprint" ""
+		(property "Footprint" "Capacitor_SMD:C_0603_1608Metric"
 			(at 115.57 177.8 0)
 			(effects
@@
 			)
 		)
-		(property "Footprint" ""
+		(property "Footprint" "Resistor_SMD:R_0603_1608Metric"
 			(at 226.06 146.05 0)
 			(effects
@@
 			)
 		)
-		(property "Footprint" ""
+		(property "Footprint" "Resistor_SMD:R_1210_3225Metric"
 			(at 184.15 109.22 0)
 			(effects
@@
 			)
 		)
-		(property "Footprint" ""
+		(property "Footprint" "Resistor_SMD:R_1210_3225Metric"
 			(at 229.87 109.22 0)
 			(effects
@@
 			)
 		)
-		(property "Footprint" ""
+		(property "Footprint" "Resistor_SMD:R_0603_1608Metric"
 			(at 110.49 135.89 0)
 			(effects
@@
 			)
 		)
-		(property "Footprint" ""
+		(property "Footprint" "Resistor_SMD:R_0603_1608Metric"
 			(at 38.1 180.34 0)
 			(effects
@@
 			)
 		)
-		(property "Footprint" ""
+		(property "Footprint" "Resistor_SMD:R_0603_1608Metric"
 			(at 38.1 175.26 0)
 			(effects
@@
 			)
 		)
-		(property "Footprint" ""
+		(property "Footprint" "Capacitor_SMD:C_0603_1608Metric"
 			(at 38.1 139.7 0)
 			(effects
@@
 			)
 		)
-		(property "Footprint" ""
+		(property "Footprint" "x1p-003:Pogo_Drill_0.9mm__Pad_2.0mm"
 			(at 40.64 82.55 0)
 			(effects
@@
 			)
 		)
-		(property "Footprint" ""
+		(property "Footprint" "x1p-003:Pogo_Drill_0.9mm__Pad_2.0mm"
 			(at 40.64 52.07 0)
 			(effects
@@
 			)
 		)
-		(property "Footprint" ""
+		(property "Footprint" "Capacitor_SMD:C_0603_1608Metric"
 			(at 226.06 76.2 0)
 			(effects
@@
 			)
 		)
-		(property "Footprint" ""
+		(property "Footprint" "Resistor_SMD:R_0603_1608Metric"
 			(at 110.49 175.26 0)
 			(effects
@@
 			)
 		)
-		(property "Footprint" ""
+		(property "Footprint" "Capacitor_SMD:C_0603_1608Metric"
 			(at 193.04 109.22 0)
 			(effects
@@
 			)
 		)
-		(property "Footprint" ""
+		(property "Footprint" "x1p-003:Pogo_Drill_0.9mm__Pad_2.0mm"
 			(at 40.64 90.17 0)
 			(effects
@@
 			)
 		)
-		(property "Footprint" ""
+		(property "Footprint" "x1p-003:Pogo_Drill_0.9mm__Pad_2.0mm"
 			(at 40.64 59.69 0)
 			(effects
@@
 			)
 		)
-		(property "Footprint" ""
+		(property "Footprint" "Resistor_SMD:R_0603_1608Metric"
 			(at 110.49 180.34 0)
 			(effects
@@
 			)
 		)
-		(property "Footprint" ""
+		(property "Footprint" "x1p-003:Pogo_Drill_0.9mm__Pad_2.0mm"
 			(at 40.64 97.79 0)
 			(effects
@@
 			)
 		)
-		(property "Footprint" ""
+		(property "Footprint" "Capacitor_SMD:C_0603_1608Metric"
 			(at 180.34 76.2 0)
 			(effects
@@
 			)
 		)
-		(property "Footprint" ""
+		(property "Footprint" "Resistor_SMD:R_0603_1608Metric"
 			(at 110.49 140.97 0)
 			(effects
@@
 			)
 		)
-		(property "Footprint" ""
+		(property "Footprint" "Capacitor_SMD:C_0603_1608Metric"
 			(at 58.42 139.7 0)
 			(effects
@@
 			)
 		)
-		(property "Footprint" ""
+		(property "Footprint" "Capacitor_SMD:C_0603_1608Metric"
 			(at 115.57 138.43 0)
 			(effects

Commit message: x1p-003: switch to mill-max pogos
Parts:
- added Q1: AO3400A, Package_TO_SOT_SMD:SOT-23, symbol Transistor_FET:AO3400A
- D1: footprint (none) -> LED_SMD:LED_0805_2012Metric; LCSC Part (none) -> C965815
- D2: footprint (none) -> LED_SMD:LED_0805_2012Metric; LCSC Part (none) -> C965812
- J11: footprint x1p-003:AUDIO-TH_24.243.2 -> x1p-003:AUDIO-TH_24.243.1
- J9: value USB_B_Micro -> Amphenol 10103594-0001LF; footprint (none) -> Connector_USB:USB_Micro-B_Amphenol_10103594-0001LF_Horizontal; LCSC Part (none) -> C428495
- R1, R4, R7: footprint (none) -> Resistor_SMD:R_1206_3216Metric; symbol Device:R_Shunt_US -> Device:R_Small_US; LCSC Part (none) -> C601089
- R12: value 220 -> 330
- R13: value 220 -> 120
- TP1: renamed from J1; footprint x1p-003:Pogo_Drill_0.9mm__Pad_2.0mm -> x1p-003:MillMax_0908; LCSC Part C5157487 -> (none); MPN (none) -> 0908-5-15-20-75-14-11-0
- TP2: renamed from J2; footprint x1p-003:Pogo_Drill_0.9mm__Pad_2.0mm -> x1p-003:MillMax_0908; LCSC Part C5157487 -> (none); MPN (none) -> 0908-6-15-20-75-14-11-0
- TP3: renamed from J3; footprint x1p-003:Pogo_Drill_0.9mm__Pad_2.0mm -> x1p-003:MillMax_0908; LCSC Part C5157487 -> (none); MPN (none) -> 0908-6-15-20-75-14-11-0
- TP4: renamed from J4; footprint x1p-003:Pogo_Drill_0.9mm__Pad_2.0mm -> x1p-003:MillMax_0908; LCSC Part C5157487 -> (none); MPN (none) -> 0908-6-15-20-75-14-11-0
- TP5: renamed from J5; footprint x1p-003:Pogo_Drill_0.9mm__Pad_2.0mm -> x1p-003:MillMax_0908; LCSC Part C5157487 -> (none); MPN (none) -> 0908-6-15-20-75-14-11-0
- TP6: renamed from J8; footprint x1p-003:Pogo_Drill_0.9mm__Pad_2.0mm -> x1p-003:MillMax_0908; LCSC Part C5157487 -> (none); MPN (none) -> 0908-6-15-20-75-14-11-0
- TP7: renamed from J7; footprint x1p-003:Pogo_Drill_0.9mm__Pad_2.0mm -> x1p-003:MillMax_0908; LCSC Part C5157487 -> (none); MPN (none) -> 0908-6-15-20-75-14-11-0
- TP8: renamed from J6; footprint x1p-003:Pogo_Drill_0.9mm__Pad_2.0mm -> x1p-003:MillMax_0908; LCSC Part C5157487 -> (none); MPN (none) -> 0908-7-15-20-75-14-11-0
Connections:
- net +24V: now also R2.1
- net +3.3V: now also R8.1
- net +5V: now also D1.2 (A), R5.1
- net 24V_DUT: now also R1.2, R3.2; no longer R1.4
- net 3V3_LOAD: now also R7.2, R9.2; no longer R7.4
- net 5V_LOAD: now also R4.2, R6.2; no longer R4.4
- net GND: now also Q1.2 (S); no longer R12.1
- net LED_PASS: now also Q1.1 (G); no longer D1.2 (A)
- new net: Q1.3 (D), R12.1
Other:
- moved on the sheet: D1, R12

Commit message: X1P-003-A01 release
Parts:
- C1, C2, C3, C4: LCSC (none) -> C15849
- C10, C11, C12, C9: LCSC (none) -> C19666
- C5, C6, C7, C8: LCSC (none) -> C14663
- D1: LCSC (none) -> C965815
- D2: LCSC (none) -> C965812
- J10: LCSC (none) -> C7437321
- J11: LCSC (none) -> C7437322
- J9: LCSC (none) -> C428495
- Q1: LCSC (none) -> C347475
- R1, R4, R7: LCSC (none) -> C601089
- R10: LCSC (none) -> C1409
- R11: LCSC (none) -> C25340
- R12: LCSC (none) -> C23138
- R13: LCSC (none) -> C22787
- R2, R3, R5, R6, R8, R9: LCSC (none) -> C22859
- U1, U2, U3: LCSC (none) -> C138706
- U4: LCSC (none) -> C2688883
- U5, U6: LCSC (none) -> C140311
Connections:
- net +5V: no longer D1.2 (A)
- net 5V_LOAD: now also D1.2 (A)
